Commit message: convex decompose for cr5

File: manipulator/Dobot/cr5_description/xacro/arm.xacro (robot description, xacro)
@@ -16,10 +16,10 @@
       <visual>
         <geometry>
-          <mesh filename="file://$(find cr5_description)/meshes/base_link.obj"/>
-        </geometry>
-      </visual>
-      <collision>
-        <geometry>
-          <mesh filename="file://$(find cr5_description)/meshes/base_link.obj"/>
+          <mesh filename="file://$(find cr5_description)/meshes/visual/base_link.obj"/>
+        </geometry>
+      </visual>
+      <collision>
+        <geometry>
+          <mesh filename="file://$(find cr5_description)/meshes/collision/base_link.obj"/>
         </geometry>
       </collision>
@@ -39,10 +39,15 @@
       <visual>
         <geometry>
-          <mesh filename="file://$(find cr5_description)/meshes/Link1.obj"/>
-        </geometry>
-      </visual>
-      <collision>
-        <geometry>
-          <mesh filename="file://$(find cr5_description)/meshes/Link1.obj"/>
+          <mesh filename="file://$(find cr5_description)/meshes/visual/Link1.obj"/>
+        </geometry>
+      </visual>
+      <collision>
+        <geometry>
+          <mesh filename="file://$(find cr5_description)/meshes/collision/Link1_0.obj"/>
+        </geometry>
+      </collision>
+      <collision>
+        <geometry>
+          <mesh filename="file://$(find cr5_description)/meshes/collision/Link1_1.obj"/>
         </geometry>
       </collision>
@@ -69,10 +74,20 @@
       <visual>
         <geometry>
-          <mesh filename="file://$(find cr5_description)/meshes/Link2.obj"/>
-        </geometry>
-      </visual>
-      <collision>
-        <geometry>
-          <mesh filename="file://$(find cr5_description)/meshes/Link2.obj"/>
+          <mesh filename="file://$(find cr5_description)/meshes/visual/Link2.obj"/>
+        </geometry>
+      </visual>
+      <collision>
+        <geometry>
+          <mesh filename="file://$(find cr5_description)/meshes/collision/Link2_0.obj"/>
+        </geometry>
+      </collision>
+      <collision>
+        <geometry>
+          <mesh filename="file://$(find cr5_description)/meshes/collision/Link2_1.obj"/>
+        </geometry>
+      </collision>
+      <collision>
+        <geometry>
+          <mesh filename="file://$(find cr5_description)/meshes/collision/Link2_2.obj"/>
         </geometry>
       </collision>
@@ -99,10 +114,20 @@
       <visual>
         <geometry>
-          <mesh filename="file://$(find cr5_description)/meshes/Link3.obj"/>
-        </geometry>
-      </visual>
-      <collision>
-        <geometry>
-          <mesh filename="file://$(find cr5_description)/meshes/Link3.obj"/>
+          <mesh filename="file://$(find cr5_description)/meshes/visual/Link3.obj"/>
+        </geometry>
+      </visual>
+      <collision>
+        <geometry>
+          <mesh filename="file://$(find cr5_description)/meshes/collision/Link3_0.obj"/>
+        </geometry>
+      </collision>
+      <collision>
+        <geometry>
+          <mesh filename="file://$(find cr5_description)/meshes/collision/Link3_1.obj"/>
+        </geometry>
+      </collision>
+      <collision>
+        <geometry>
+          <mesh filename="file://$(find cr5_description)/meshes/collision/Link3_2.obj"/>
         </geometry>
       </collision>
@@ -129,10 +154,15 @@
       <visual>
         <geometry>
-          <mesh filename="file://$(find cr5_description)/meshes/Link4.obj"/>
-        </geometry>
-      </visual>
-      <collision>
-        <geometry>
-          <mesh filename="file://$(find cr5_description)/meshes/Link4.obj"/>
+          <mesh filename="file://$(find cr5_description)/meshes/visual/Link4.obj"/>
+        </geometry>
+      </visual>
+      <collision>
+        <geometry>
+          <mesh filename="file://$(find cr5_description)/meshes/collision/Link4_0.obj"/>
+        </geometry>
+      </collision>
+      <collision>
+        <geometry>
+          <mesh filename="file://$(find cr5_description)/meshes/collision/Link4_1.obj"/>
         </geometry>
       </collision>
@@ -159,10 +189,10 @@
       <visual>
         <geometry>
-          <mesh filename="file://$(find cr5_description)/meshes/Link5.obj"/>
-        </geometry>
-      </visual>
-      <collision>
-        <geometry>
-          <mesh filename="file://$(find cr5_description)/meshes/Link5.obj"/>
+          <mesh filename="file://$(find cr5_description)/meshes/visual/Link5.obj"/>
+        </geometry>
+      </visual>
+      <collision>
+        <geometry>
+          <mesh filename="file://$(find cr5_description)/meshes/collision/Link5.obj"/>
         </geometry>
       </collision>
@@ -189,10 +219,10 @@
       <visual>
         <geometry>
-          <mesh filename="file://$(find cr5_description)/meshes/Link6.obj"/>
-        </geometry>
-      </visual>
-      <collision>
-        <geometry>
-          <mesh filename="file://$(find cr5_description)/meshes/Link6.obj"/>
+          <mesh filename="file://$(find cr5_description)/meshes/visual/Link6.obj"/>
+        </geometry>
+      </visual>
+      <collision>
+        <geometry>
+          <mesh filename="file://$(find cr5_description)/meshes/collision/Link6.obj"/>
         </geometry>
       </collision>

File: manipulator/Dobot/cr5_description/xacro/ros2_control/cr5.ros2_control.xacro (robot description, xacro)
@@ -12,6 +12,6 @@
         <xacro:if value="${ros2_control_hardware_type == 'isaac'}">
           <plugin>topic_based_ros2_control/TopicBasedSystem</plugin>
-          <param name="joint_commands_topic">/isaac_joint_commands</param>
-          <param name="joint_states_topic">/isaac_joint_states</param>
+          <param name="joint_commands_topic">/isaac/joint_commands</param>
+          <param name="joint_states_topic">/isaac/joint_states</param>
         </xacro:if>
       </hardware>
