Commit message: add ocs2 demo

File: manipulator/AgileX/piper_description/xacro/slave.xacro (robot description, xacro)
@@ -74,5 +74,5 @@
       <parent link="${prefix}link6"/>
       <child link="${prefix}gripper_center"/>
-      <origin xyz="0 0 0.1358"/>
+      <origin xyz="0 0 0.1358" rpy="0 -1.57 0"/>
     </joint>
     <link name="${prefix}camera"/>

File: manipulator/Dobot/cr5_description/urdf/cr5.urdf (robot description, URDF)
Before this commit: robot cr5_robot, 7 links, 6 joints
Joints:
- joint joint1: limit lower=-3.14 upper=3.14 effort=300 velocity=100 -> lower=-6.28318 upper=6.28318 effort=300 velocity=3.14159; origin xyz=0 0 0.147 rpy=0 0 0 -> xyz=0 0 0.147
- joint joint2: limit lower=-3.14 upper=3.14 effort=300 velocity=100 -> lower=-6.28318 upper=6.28318 effort=300 velocity=3.14159; origin xyz=0 0 0 rpy=1.5708 1.5708 0 -> rpy=1.5708 1.5708 0
- joint joint3: limit lower=-2.86 upper=2.86 effort=300 velocity=100 -> lower=-2.7925 upper=2.7925 effort=300 velocity=3.14159; origin xyz=-0.427 0 0 rpy=0 0 0 -> xyz=-0.427 0 0
- joint joint4: limit lower=-3.14 upper=3.14 effort=300 velocity=100 -> lower=-6.28318 upper=6.28318 effort=300 velocity=3.14159
- joint joint5: limit lower=-3.14 upper=3.14 effort=300 velocity=100 -> lower=-6.28318 upper=6.28318 effort=300 velocity=3.14159
- joint joint6: limit lower=-6.28 upper=6.28 effort=300 velocity=100 -> lower=-6.28318 upper=6.28318 effort=300 velocity=3.14159
