Commit message: add ocs2 demo for galaxea a1xy

File: manipulator/Galaxea/a1xy_description/xacro/gripper.xacro (robot description, xacro)
@@ -2,10 +2,8 @@
 <robot xmlns:xacro="http://www.ros.org/wiki/xacro">
   <xacro:macro name="Gripper">
-    <link
-        name="gripper_link">
+    <link name="gripper_link">
       <inertial>
         <origin xyz="-0.0311072323899603 1.17979991887118E-08 7.93394685505433E-08"/>
-        <mass
-            value="0.604"/>
+        <mass value="0.604"/>
         <inertia
             ixx="0.000175881544189539"
@@ -27,16 +25,9 @@
       </collision>
     </link>
-    <joint
-        name="gripper_joint"
-        type="fixed">
-      <origin
-          xyz="0.08165 0 0"
-          rpy="0 0 0"/>
-      <parent
-          link="arm_link6"/>
-      <child
-          link="gripper_link"/>
-      <axis
-          xyz="0 0 0"/>
+    <joint name="gripper_joint" type="fixed">
+      <origin xyz="0.08165 0 0"/>
+      <parent link="arm_link6"/>
+      <child link="gripper_link"/>
+      <axis xyz="0 0 0"/>
     </joint>
     <link
@@ -67,30 +58,15 @@
       </collision>
     </link>
-    <joint
-        name="gripper_finger_joint1"
-        type="prismatic">
-      <origin
-          xyz="0.03689 0.013453 0.00012059"
-          rpy="0 0 0"/>
-      <parent
-          link="gripper_link"/>
-      <child
-          link="gripper_finger_link1"/>
-      <axis
-          xyz="0 1 0"/>
-      <limit
-          lower="0"
-          upper="0.05"
-          effort="100"
-          velocity="0.25"/>
+    <joint name="gripper_finger_joint1" type="prismatic">
+      <origin xyz="0.03689 0.013453 0.00012059"/>
+      <parent link="gripper_link"/>
+      <child link="gripper_finger_link1"/>
+      <axis xyz="0 1 0"/>
+      <limit lower="0" upper="0.05" effort="100" velocity="0.25"/>
     </joint>
-    <link
-        name="gripper_finger_link2">
+    <link name="gripper_finger_link2">
       <inertial>
-        <origin
-            xyz="-0.0195895857999098 0.0151136893508115 -0.00542254357246619"
-        />
-        <mass
-            value="0.027"/>
+        <origin xyz="-0.0195895857999098 0.0151136893508115 -0.00542254357246619"/>
+        <mass value="0.027"/>
         <inertia
             ixx="2.40569340151687E-06"
@@ -112,21 +88,10 @@
       </collision>
     </link>
-    <joint
-        name="gripper_finger_joint2"
-        type="prismatic">
-      <origin
-          xyz="0.03689 -0.013453 -0.00012059"
-          rpy="0 0 0"/>
-      <parent
-          link="gripper_link"/>
-      <child
-          link="gripper_finger_link2"/>
-      <axis
-          xyz="0 -1 0"/>
-      <limit
-          lower="0"
-          upper="0.05"
-          effort="100"
-          velocity="0.25"/>
+    <joint name="gripper_finger_joint2" type="prismatic">
+      <origin xyz="0.03689 -0.013453 -0.00012059"/>
+      <parent link="gripper_link"/>
+      <child link="gripper_finger_link2"/>
+      <axis xyz="0 -1 0"/>
+      <limit lower="0" upper="0.05" effort="100" velocity="0.25"/>
       <mimic joint="gripper_finger_joint1" multiplier="1" offset="0"/>
     </joint>
