Commit message: add agibot g1

File: manipulator/Galaxea/a1xy_description/xacro/a1_x.xacro (robot description, xacro)
@@ -1,7 +1,10 @@
 <?xml version="1.0" encoding="utf-8"?>
 <robot xmlns:xacro="http://www.ros.org/wiki/xacro">
-  <xacro:macro name="Arm">
+  <xacro:macro name="Arm" params="name">
+    <xacro:include filename="$(find a1xy_description)/xacro/xy_base.xacro"/>
+    <xacro:property name="prefix" value="${name + '_' if name else ''}"/>
+    <xacro:Base name=""/>
     <link
-        name="arm_link3">
+        name="${prefix}link3">
       <inertial>
         <origin
@@ -30,5 +33,5 @@
     </link>
     <joint
-        name="arm_joint3"
+        name="${prefix}joint3"
         type="revolute">
       <origin
@@ -36,7 +39,7 @@
           rpy="0 0 0"/>
       <parent
-          link="arm_link2"/>
+          link="${prefix}link2"/>
       <child
-          link="arm_link3"/>
+          link="${prefix}link3"/>
       <axis
           xyz="0 1 0"/>
@@ -48,5 +51,5 @@
     </joint>
     <link
-        name="arm_link4">
+        name="${prefix}link4">
       <inertial>
         <origin
@@ -75,5 +78,5 @@
     </link>
     <joint
-        name="arm_joint4"
+        name="${prefix}joint4"
         type="revolute">
       <origin
@@ -81,7 +84,7 @@
           rpy="0 0 0"/>
       <parent
-          link="arm_link3"/>
+          link="${prefix}link3"/>
       <child
-          link="arm_link4"/>
+          link="${prefix}link4"/>
       <axis
           xyz="0 1 0"/>
@@ -93,5 +96,5 @@
     </joint>
     <link
-        name="arm_link5">
+        name="${prefix}link5">
       <inertial>
         <origin
@@ -120,5 +123,5 @@
     </link>
     <joint
-        name="arm_joint5"
+        name="${prefix}joint5"
         type="revolute">
       <origin
@@ -126,7 +129,7 @@
           rpy="0 0 0"/>
       <parent
-          link="arm_link4"/>
+          link="${prefix}link4"/>
       <child
-          link="arm_link5"/>
+          link="${prefix}link5"/>
       <axis
           xyz="0 0 1"/>
@@ -138,5 +141,5 @@
     </joint>
     <link
-        name="arm_link6">
+        name="${prefix}link6">
       <inertial>
         <origin
@@ -165,5 +168,5 @@
     </link>
     <joint
-        name="arm_joint6"
+        name="${prefix}joint6"
         type="revolute">
       <origin
@@ -171,7 +174,7 @@
           rpy="0 0 0"/>
       <parent
-          link="arm_link5"/>
+          link="${prefix}link5"/>
       <child
-          link="arm_link6"/>
+          link="${prefix}link6"/>
       <axis
           xyz="1 0 0"/>
@@ -182,4 +185,12 @@
           velocity="32.9867"/>
     </joint>
+    <xacro:include filename="$(find a1xy_description)/xacro/gripper.xacro"/>
+    <xacro:Gripper name="${name}"/>
+    <joint name="${prefix}gripper_joint" type="fixed">
+      <origin xyz="0.08165 0 0"/>
+      <parent link="${prefix}link6"/>
+      <child link="${prefix}gripper_link"/>
+      <axis xyz="0 0 0"/>
+    </joint>
   </xacro:macro>
 </robot>

File: manipulator/Galaxea/a1xy_description/xacro/a1_y.xacro (robot description, xacro)
@@ -1,6 +1,9 @@
 <?xml version="1.0" encoding="utf-8"?>
 <robot xmlns:xacro="http://www.ros.org/wiki/xacro">
-  <xacro:macro name="Arm">
-    <link name="arm_link3">
+  <xacro:macro name="Arm" params="name">
+    <xacro:include filename="$(find a1xy_description)/xacro/xy_base.xacro"/>
+    <xacro:property name="prefix" value="${name + '_' if name else ''}"/>
+    <xacro:Base name=""/>
+    <link name="${prefix}link3">
       <inertial>
         <origin xyz="0.0795681449160072 -0.0327357454565678 0.065177920553168"/>
@@ -26,5 +29,5 @@
     </link>
     <joint
-        name="arm_joint3"
+        name="${prefix}joint3"
         type="revolute">
       <origin
@@ -32,7 +35,7 @@
           rpy="0 0 0" />
       <parent
-          link="arm_link2" />
-      <child
-          link="arm_link3" />
+          link="${prefix}link2" />
+      <child
+          link="${prefix}link3" />
       <axis
           xyz="0 1 0" />
@@ -44,5 +47,5 @@
     </joint>
     <link
-        name="arm_link4">
+        name="${prefix}link4">
       <inertial>
         <origin
@@ -78,5 +81,5 @@
     </link>
     <joint
-        name="arm_joint4"
+        name="${prefix}joint4"
         type="revolute">
       <origin
@@ -84,7 +87,7 @@
           rpy="0 0 0" />
       <parent
-          link="arm_link3" />
-      <child
-          link="arm_link4" />
+          link="${prefix}link3" />
+      <child
+          link="${prefix}link4" />
       <axis
           xyz="1 0 0" />
@@ -96,5 +99,5 @@
     </joint>
     <link
-        name="arm_link5">
+        name="${prefix}link5">
       <inertial>
         <origin
@@ -130,5 +133,5 @@
     </link>
     <joint
-        name="arm_joint5"
+        name="${prefix}joint5"
         type="revolute">
       <origin
@@ -136,7 +139,7 @@
           rpy="0 0 0" />
       <parent
-          link="arm_link4" />
-      <child
-          link="arm_link5" />
+          link="${prefix}link4" />
+      <child
+          link="${prefix}link5" />
       <axis
           xyz="0 1 0" />
@@ -148,5 +151,5 @@
     </joint>
     <link
-        name="arm_link6">
+        name="${prefix}link6">
       <inertial>
         <origin
@@ -182,5 +185,5 @@
     </link>
     <joint
-        name="arm_joint6"
+        name="${prefix}joint6"
         type="revolute">
       <origin
@@ -188,7 +191,7 @@
           rpy="0 0 0" />
       <parent
-          link="arm_link5" />
-      <child
-          link="arm_link6" />
+          link="${prefix}link5" />
+      <child
+          link="${prefix}link6" />
       <axis
           xyz="1 0 0" />
@@ -199,4 +202,12 @@
           velocity="32.9867" />
     </joint>
+    <xacro:include filename="$(find a1xy_description)/xacro/gripper.xacro"/>
+    <xacro:Gripper name="${name}"/>
+    <joint name="${prefix}gripper_joint" type="fixed">
+      <origin xyz="0.08165 0 0"/>
+      <parent link="${prefix}link6"/>
+      <child link="${prefix}gripper_link"/>
+      <axis xyz="0 0 0"/>
+    </joint>
   </xacro:macro>
 </robot>

File: manipulator/Galaxea/a1xy_description/xacro/gripper.xacro (robot description, xacro)
@@ -1,6 +1,7 @@
 <?xml version="1.0" encoding="utf-8"?>
 <robot xmlns:xacro="http://www.ros.org/wiki/xacro">
-  <xacro:macro name="Gripper">
-    <link name="gripper_link">
+  <xacro:macro name="Gripper" params="name">
+    <xacro:property name="prefix" value="${name + '_' if name else ''}"/>
+    <link name="${prefix}gripper_link">
       <inertial>
         <origin xyz="-0.0311072323899603 1.17979991887118E-08 7.93394685505433E-08"/>
@@ -25,18 +26,8 @@
       </collision>
     </link>
-    <joint name="gripper_joint" type="fixed">
-      <origin xyz="0.08165 0 0"/>
-      <parent link="arm_link6"/>
-      <child link="gripper_link"/>
-      <axis xyz="0 0 0"/>
-    </joint>
-    <link
-        name="gripper_finger_link1">
+    <link name="${prefix}gripper_finger_link1">
       <inertial>
-        <origin
-            xyz="-0.0195895895552112 -0.0151136845490034 0.00542254359093075"
-        />
-        <mass
-            value="0.027"/>
+        <origin xyz="-0.0195895895552112 -0.0151136845490034 0.00542254359093075"/>
+        <mass value="0.027"/>
         <inertia
             ixx="2.40569358477209E-06"
@@ -58,12 +49,12 @@
       </collision>
     </link>
-    <joint name="gripper_finger_joint1" type="prismatic">
+    <joint name="${prefix}gripper_finger_joint1" type="prismatic">
       <origin xyz="0.03689 0.013453 0.00012059"/>
-      <parent link="gripper_link"/>
-      <child link="gripper_finger_link1"/>
+      <parent link="${prefix}gripper_link"/>
+      <child link="${prefix}gripper_finger_link1"/>
       <axis xyz="0 1 0"/>
       <limit lower="0" upper="0.05" effort="100" velocity="0.25"/>
     </joint>
-    <link name="gripper_finger_link2">
+    <link name="${prefix}gripper_finger_link2">
       <inertial>
         <origin xyz="-0.0195895857999098 0.0151136893508115 -0.00542254357246619"/>
@@ -88,8 +79,8 @@
       </collision>
     </link>
-    <joint name="gripper_finger_joint2" type="prismatic">
+    <joint name="${prefix}gripper_finger_joint2" type="prismatic">
       <origin xyz="0.03689 -0.013453 -0.00012059"/>
-      <parent link="gripper_link"/>
-      <child link="gripper_finger_link2"/>
+      <parent link="${prefix}gripper_link"/>
+      <child link="${prefix}gripper_finger_link2"/>
       <axis xyz="0 -1 0"/>
       <limit lower="0" upper="0.05" effort="100" velocity="0.25"/>

File: manipulator/Galaxea/a1xy_description/xacro/robot.xacro (robot description, xacro)
@@ -1,15 +1,11 @@
 <?xml version="1.0" encoding="utf-8"?>
 <robot name="a1y" xmlns:xacro="http://www.ros.org/wiki/xacro">
-  <xacro:include filename="$(find a1xy_description)/xacro/xy_base.xacro"/>
-  <xacro:Base name=""/>
-  <xacro:include filename="$(find a1xy_description)/xacro/gripper.xacro"/>
-  <xacro:Gripper/>
   <xacro:arg name="type" default="x"/>
   <xacro:if value="${'$(arg type)' == 'x'}">
-    <xacro:include filename="$(find a1xy_description)/xacro/x_link.xacro"/>
+    <xacro:include filename="$(find a1xy_description)/xacro/a1_x.xacro"/>
   </xacro:if>
   <xacro:unless value="${'$(arg type)' == 'x'}">
-    <xacro:include filename="$(find a1xy_description)/xacro/y_link.xacro"/>
+    <xacro:include filename="$(find a1xy_description)/xacro/a1_y.xacro"/>
   </xacro:unless>
-  <xacro:Arm/>
+  <xacro:Arm name=""/>
 </robot>

File: manipulator/Galaxea/a1xy_description/xacro/xy_base.xacro (robot description, xacro)
@@ -2,5 +2,5 @@
 <robot xmlns:xacro="http://www.ros.org/wiki/xacro">
   <xacro:macro name="Base" params="name">
-    <link name="base_link">
+    <link name="${prefix}base_link">
       <inertial>
         <origin
@@ -29,5 +29,5 @@
     </link>
     <link
-        name="arm_link1">
+        name="${prefix}link1">
       <inertial>
         <origin
@@ -69,5 +69,5 @@
     </link>
     <joint
-        name="arm_joint1"
+        name="${prefix}joint1"
         type="revolute">
       <origin
@@ -77,5 +77,5 @@
           link="base_link"/>
       <child
-          link="arm_link1"/>
+          link="${prefix}link1"/>
       <axis
           xyz="0 0 1"/>
@@ -87,5 +87,5 @@
     </joint>
     <link
-        name="arm_link2">
+        name="${prefix}link2">
       <inertial>
         <origin
@@ -127,5 +127,5 @@
     </link>
     <joint
-        name="arm_joint2"
+        name="${prefix}joint2"
         type="revolute">
       <origin
@@ -133,7 +133,7 @@
           rpy="0 0 0"/>
       <parent
-          link="arm_link1"/>
+          link="${prefix}link1"/>
       <child
-          link="arm_link2"/>
+          link="${prefix}link2"/>
       <axis
           xyz="0 1 0"/>
