Commit message: add SO101 arm

File: humanoid/RobotEra/xbot_description/urdf/robot.urdf (robot description, URDF)
Before this commit: robot xbot_l, 91 links, 90 joints
Links:
- added link base; visual box size=0.001 0.001 0.001
- link base_link: geometry collision box size=0.4 0.4 0.4; visual mesh filename=../meshes/base_link.obj
- link left_leg_pitch_link: geometry collision mesh filename=../meshes/left_leg_pitch_link.obj; visual mesh filename=../meshes/left_leg_pitch_link.obj
- link neck_pitch_link: geometry collision mesh filename=../meshes/head.obj; visual mesh filename=../meshes/head.obj
- link realsense_link: geometry collision mesh filename=../meshes/d455.obj; visual mesh filename=../meshes/d455.obj
- link right_leg_pitch_link: geometry collision mesh filename=../meshes/right_leg_pitch_link.obj; visual mesh filename=../meshes/right_leg_pitch_link.obj
Joints:
- added joint floating_base: type fixed, parent base, child base_link
- joint left_arm_base_joint: axis 0 0 0 -> (none)
- joint left_arm_flange_fixed_joint: origin xyz=0.0 0 0.1135 rpy=0 0 0 -> xyz=0.0 0 0.1135
- joint left_hand_index_joint1: origin xyz=0.03583 0 -0.1067 rpy=0 0 0 -> xyz=0.03583 0 -0.1067
- joint left_hand_index_joint2: origin xyz=0 0 -0.06675 rpy=0 0 0 -> xyz=0 0 -0.06675
- joint left_hand_index_tip_link: origin xyz=0 0 -0.0532473502691896 rpy=0 0 0 -> xyz=0 0 -0.0532473502691896
- joint left_hand_mid_joint1: origin xyz=0.00533 -0.008 -0.1072 rpy=0 0 0 -> xyz=0.00533 -0.008 -0.1072
- joint left_hand_mid_joint2: origin xyz=0 0 -0.06525 rpy=0 0 0 -> xyz=0 0 -0.06525
- joint left_hand_mid_tip_joint: origin xyz=0 0 -0.0532473502691905 rpy=0 0 0 -> xyz=0 0 -0.0532473502691905
- joint left_hand_pinky_joint1: origin xyz=-0.04267 -0.008 -0.0992 rpy=0 0 0 -> xyz=-0.04267 -0.008 -0.0992
- joint left_hand_pinky_joint2: origin xyz=0 0 -0.06525 rpy=0 0 0 -> xyz=0 0 -0.06525
- joint left_hand_pinky_tip_link: origin xyz=0 0 -0.0532473502691902 rpy=0 0 0 -> xyz=0 0 -0.0532473502691902
- joint left_hand_ring_joint1: origin xyz=-0.01867 -0.008 -0.1032 rpy=0 0 0 -> xyz=-0.01867 -0.008 -0.1032
- joint left_hand_ring_joint2: origin xyz=0 0 -0.06525 rpy=0 0 0 -> xyz=0 0 -0.06525
- joint left_hand_ring_tip_link: origin xyz=0 0 -0.0532473502691904 rpy=0 0 0 -> xyz=0 0 -0.0532473502691904
- joint left_hand_thumb_bend_joint: origin xyz=0.02503 -0.013 -0.03275 rpy=0 0 0 -> xyz=0.02503 -0.013 -0.03275
- joint left_hand_thumb_rota_joint1: origin xyz=0.032173 -0.0035045 0.00225 rpy=0 0 0 -> xyz=0.032173 -0.0035045 0.00225
- joint left_hand_thumb_rota_joint2: origin xyz=0.06 0 0 rpy=0 0 0 -> xyz=0.06 0 0
- joint left_hand_thumb_tip_joint: origin xyz=0.051457 0 0 rpy=0 0 0 -> xyz=0.051457 0 0
- joint left_shoulder_pitch_joint: origin xyz=0 0 0.2635 rpy=0 0 0 -> xyz=0 0 0.2635
- joint neck_base_joint: axis 0 0 0 -> (none); origin xyz=0 0 0.4 rpy=0 0 0 -> xyz=0 0 0.4
- joint neck_yaw_joint: origin xyz=0 0 0 rpy=0 0 0 -> (none)
- joint realsense_joint: axis 0 0 0 -> (none); origin xyz=0.066371 -0.12536 0.0475 rpy=0.34907 1.5708 0 -> xyz=0.066371 -0.12536 0.0475 rpy=-0.34907 1.5708 0
- joint right_hand_index_joint1: origin xyz=0.03583 0.006 -0.1067 rpy=0 0 0 -> xyz=0.03583 0.006 -0.1067
- joint right_hand_index_joint2: origin xyz=0 0 -0.06675 rpy=0 0 0 -> xyz=0 0 -0.06675
- joint right_hand_index_tip_joint: origin xyz=0 0 -0.053247 rpy=0 0 0 -> xyz=0 0 -0.053247
- joint right_hand_mid_joint1: origin xyz=0.00533 0.008 -0.1072 rpy=0 0 0 -> xyz=0.00533 0.008 -0.1072
- joint right_hand_mid_joint2: origin xyz=0 0 -0.06525 rpy=0 0 0 -> xyz=0 0 -0.06525
- joint right_hand_mid_tip_link: origin xyz=0 0 -0.053247 rpy=0 0 0 -> xyz=0 0 -0.053247
- joint right_hand_pinky_joint1: origin xyz=-0.04267 0.008 -0.0992 rpy=0 0 0 -> xyz=-0.04267 0.008 -0.0992
- joint right_hand_pinky_joint2: origin xyz=0 0 -0.06525 rpy=0 0 0 -> xyz=0 0 -0.06525
- joint right_hand_pinky_tip_joint: origin xyz=0 0 -0.053247 rpy=0 0 0 -> xyz=0 0 -0.053247
- joint right_hand_ring_joint1: origin xyz=-0.01867 0.008 -0.1032 rpy=0 0 0 -> xyz=-0.01867 0.008 -0.1032
- joint right_hand_ring_joint2: origin xyz=0 0 -0.06525 rpy=0 0 0 -> xyz=0 0 -0.06525
- joint right_hand_ring_tip_joint: origin xyz=0 0 -0.0532473502691896 rpy=0 0 0 -> xyz=0 0 -0.0532473502691896
- joint right_hand_thumb_bend_joint: origin xyz=0.02433 0.011 -0.03275 rpy=0 0 0 -> xyz=0.02433 0.011 -0.03275
- joint right_hand_thumb_rota_joint1: origin xyz=0.032873 0.0055045 0.00225 rpy=0 0 0 -> xyz=0.032873 0.0055045 0.00225
- joint right_hand_thumb_rota_joint2: origin xyz=0.06 0 0 rpy=0 0 0 -> xyz=0.06 0 0
- joint right_hand_thumb_rota_tip_joint: origin xyz=0.051457 0 0 rpy=0 0 0 -> xyz=0.051457 0 0
- joint right_shoulder_pitch_joint: origin xyz=0 0 0.2635 rpy=0 0 0 -> xyz=0 0 0.2635
- joint waist_yaw_joint: origin xyz=0 0 -0.0975 rpy=0 0 0 -> xyz=0 0 -0.0975
