Commit message: add SO101 arm

File: manipulator/TheRobotStudio/so_arm_description/xacro/so101.xacro (robot description, xacro)
@@ -349,4 +349,39 @@
       <child link="${prefix}motor6"/>
     </joint>
+    <link name="${prefix}camera_support">
+      <visual>
+        <geometry>
+          <mesh filename="file://$(find so_arm_description)/meshes/so101/camera_support.stl"/>
+        </geometry>
+        <material name="3d_printed"/>
+      </visual>
+      <collision>
+        <geometry>
+          <mesh filename="file://$(find so_arm_description)/meshes/so101/camera_support.stl"/>
+        </geometry>
+      </collision>
+    </link>
+    <joint name="${prefix}camera_support_joint" type="fixed">
+      <origin xyz="-0.001 0.025 -0.023" rpy="-1.5708 1.5708 0"/>
+      <parent link="${prefix}gripper"/>
+      <child link="${prefix}camera_support"/>
+    </joint>
+    <link name="${prefix}camera">
+      <visual>
+        <geometry>
+          <mesh filename="file://$(find so_arm_description)/meshes/so101/camera.obj"/>
+        </geometry>
+      </visual>
+      <collision>
+        <geometry>
+          <mesh filename="file://$(find so_arm_description)/meshes/so101/camera.obj"/>
+        </geometry>
+      </collision>
+    </link>
+    <joint name="${prefix}camera_joint" type="fixed">
+      <origin xyz="0.024 0 0.0375" rpy="0 0.611 0"/>
+      <parent link="${prefix}camera_support"/>
+      <child link="${prefix}camera"/>
+    </joint>
     <!-- Joint from wrist to gripper -->
     <joint name="${prefix}wrist_roll" type="revolute">

Commit message: add SO101 arm

File: manipulator/TheRobotStudio/so_arm_description/xacro/so101.xacro (robot description, xacro)
@@ -384,4 +384,10 @@
       <child link="${prefix}camera"/>
     </joint>
+    <link name="${prefix}camera_len"/>
+    <joint name="${prefix}camera_len_joint" type="fixed">
+      <origin xyz="0.02 0 0"/>
+      <parent link="${prefix}camera"/>
+      <child link="${prefix}camera_len"/>
+    </joint>
     <!-- Joint from wrist to gripper -->
     <joint name="${prefix}wrist_roll" type="revolute">
@@ -429,6 +435,11 @@
       <parent link="${prefix}gripper"/>
       <child link="${prefix}gripperframe"/>
-      <axis xyz="0 0 0"/>
-    </joint>
+    </joint>
+    <joint name="${prefix}moving_Jaw_tip_joint" type="fixed">
+      <origin rpy="0 0 0" xyz="-0.01 -0.0745 0.019"/>
+      <parent link="${prefix}moving_jaw_so101_v1"/>
+      <child link="${prefix}moving_jaw_tip"/>
+    </joint>
+    <link name="${prefix}moving_jaw_tip"/>
   </xacro:macro>
 </robot>
