Commit message: add SO101 arm

File: manipulator/TheRobotStudio/so_arm_description/urdf/so_arm.urdf (robot description, URDF)
Before this commit: robot Piper single, 15 links, 14 joints
Links:
- added link camera; collision mesh filename=package://so_arm_description/meshes/so101/camera.obj; visual mesh filename=package://so_arm_description/meshes/so101/camera.obj
- added link camera_support; collision mesh filename=package://so_arm_description/meshes/so101/camera_support.stl; visual mesh filename=package://so_arm_description/meshes/so101/camera_support.stl
Joints:
- added joint camera_joint: type fixed, parent camera_support, child camera, origin xyz=0.024 0 0.0375 rpy=0 0.611 0
- added joint camera_support_joint: type fixed, parent gripper, child camera_support, origin xyz=-0.001 0.025 -0.023 rpy=-1.5708 1.5708 0
- joint base_joint: origin xyz=-0.020791 -0.0157608 -0.0324817 rpy=0 0 1.5708 -> xyz=-0.020791 -0.0157608 -0.0324817

Commit message: fix so101 meshes, add so100

File: manipulator/TheRobotStudio/so_arm_description/urdf/so_arm.urdf (robot description, URDF)
Before this commit: robot Piper single, 17 links, 16 joints
Links:
- removed link base
- added link camera_len
- added link moving_jaw_tip
- link base_link: mass None -> 0.147; geometry collision mesh filename=package://so_arm_description/meshes/so101/base.stl; collision mesh filename=package://so_arm_description/meshes/so101/base_motor_holder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
- link gripper: geometry collision mesh filename=package://so_arm_description/meshes/so101/wrist_roll_follow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; collision mesh filename=package://so_arm_description/meshes/so101/wrist_roll_follow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
- link lower_arm: geometry collision mesh filename=package://so_arm_description/meshes/so101/motor_holder_wris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; collision mesh filename=package://so_arm_description/meshes/so101/under_arm.stl
- link motor1: geometry visual mesh filename=package://so_arm_description/meshes/so101/sts3215_03a_v1.stl
- link motor2: geometry visual mesh filename=package://so_arm_description/meshes/so101/sts3215_03a_v1.stl
- link motor3: geometry visual mesh filename=package://so_arm_description/meshes/so101/sts3215_03a_v1.stl
- link motor4: geometry visual mesh filename=package://so_arm_description/meshes/so101/sts3215_03a_v1.stl
- link motor5: geometry visual mesh filename=package://so_arm_description/meshes/so101/sts3215_03a_v1.stl
- link motor6: geometry visual mesh filename=package://so_arm_description/meshes/so101/sts3215_03a_v1.stl
- link moving_jaw_so101_v1: geometry collision mesh filename=package://so_arm_description/meshes/so101/moving_jaw/moving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; collision mesh filename=package://so_arm_description/meshes/so101/moving_jaw/moving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
- link shoulder: geometry collision mesh filename=package://so_arm_description/meshes/so101/motor_holder_base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; collision mesh filename=package://so_arm_description/meshes/so101/rotation_pitch.stl
- link upper_arm: geometry collision mesh filename=package://so_arm_description/meshes/so101/upper_arm.stl; visual mesh filename=package://so_arm_description/meshes/so101/upper_arm.stl
- link wrist: geometry collision mesh filename=package://so_arm_description/meshes/so101/wrist_roll_pitch.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; visual mesh filename=package://so_arm_description/meshes/so101/wrist_roll_pitch.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
Joints:
- removed joint base_joint
- added joint camera_len_joint: type fixed, parent camera, child camera_len, origin xyz=0.02 0 0
- added joint moving_Jaw_tip_joint: type fixed, parent moving_jaw_so101_v1, child moving_jaw_tip, origin xyz=-0.01 -0.0745 0.019
- joint gripperframe_frame: axis 0 0 0 -> (none)
- joint motor1_joint: origin xyz=0.0207909 -0.0105745 0.0761817 rpy=-2.20282e-15 2.77556e-17 -1.5708 -> xyz=0.0263345 0 0.0437; parent base -> base_link
- joint shoulder_pan: origin xyz=0.0207909 -0.0230745 0.0948817 rpy=-3.14159 6.03684e-16 1.5708 -> xyz=0.0388353 0 0.0624 rpy=-3.14159 0 3.14159; parent base -> base_link

File: manipulator/TheRobotStudio/so_arm_description/xacro/robot.xacro (robot description, xacro)
@@ -10,8 +10,11 @@
   </material>
   <xacro:arg name="type" default="so101"/>
-  <xacro:include filename="$(find so_arm_description)/xacro/so101.xacro"/>
   <!-- 根据type参数决定is_master的值 -->
   <xacro:if value="${'$(arg type)' == 'so101'}">
-    <xacro:Arm name=""/>
+    <xacro:include filename="$(find so_arm_description)/xacro/so101.xacro"/>
   </xacro:if>
+  <xacro:if value="${'$(arg type)' == 'so100'}">
+    <xacro:include filename="$(find so_arm_description)/xacro/so100.xacro"/>
+  </xacro:if>
+  <xacro:Arm name=""/>
 </robot>

File: manipulator/TheRobotStudio/so_arm_description/xacro/so101.xacro (robot description, xacro)
@@ -4,58 +4,42 @@
     <xacro:property name="prefix" value="${name + '_' if name else ''}"/>
     <!-- Frame baseframe (dummy link + fixed joint) -->
-    <link name="${prefix}base_link"/>
-    <joint name="${prefix}base_joint" type="fixed">
-      <origin xyz="-0.020791 -0.0157608 -0.0324817"/>
-      <parent link="${prefix}base_link"/>
-      <child link="${prefix}base"/>
-    </joint>
-    <!-- Link base -->
-    <link name="${prefix}base">
-      <inertial>
-        <origin xyz="0.020739 0.00204287 0.065966"/>
+    <link name="${prefix}base_link">
+      <inertial>
+        <origin xyz="-0.01371 0 0.03348"/>
         <mass value="0.147"/>
         <inertia ixx="0.000136117" ixy="4.59787e-07" ixz="9.75275e-08" iyy="0.000114686" iyz="-4.97151e-06"
                  izz="0.000130364"/>
       </inertial>
-      <!-- Part base_motor_holder_so101_v1 -->
-      <visual>
-        <origin xyz="0.0206915 0.0221255 0.0300817" rpy="1.5708 -1.23909e-16 2.33147e-15"/>
-        <geometry>
-          <mesh filename="file://$(find so_arm_description)/meshes/so101/base_motor_holder_so101_v1.stl"/>
-        </geometry>
-        <material name="3d_printed"/>
-      </visual>
-      <collision>
-        <origin xyz="0.0206915 0.0221255 0.0300817" rpy="1.5708 -1.23909e-16 2.33147e-15"/>
-        <geometry>
-          <mesh filename="file://$(find so_arm_description)/meshes/so101/base_motor_holder_so101_v1.stl"/>
-        </geometry>
-      </collision>
-      <!-- Part base_so101_v2 -->
-      <visual>
-        <origin xyz="0.0207909 0.0221255 0.0300817" rpy="1.5708 -0 0"/>
-        <geometry>
-          <mesh filename="file://$(find so_arm_description)/meshes/so101/base_so101_v2.stl"/>
-        </geometry>
-        <!--      <material name="3d_printed"/>-->
-      </visual>
-      <collision>
-        <origin xyz="0.0207909 0.0221255 0.0300817" rpy="1.5708 -0 0"/>
-        <geometry>
-          <mesh filename="file://$(find so_arm_description)/meshes/so101/base_so101_v2.stl"/>
-        </geometry>
-      </collision>
-      <!-- Part waveshare_mounting_plate_so101_v2 -->
-      <visual>
-        <origin xyz="0.0205915 0.0467435 0.0798817" rpy="1.5708 -1.21716e-14 2.33147e-15"/>
-        <geometry>
-          <mesh filename="file://$(find so_arm_description)/meshes/so101/waveshare_mounting_plate_so101_v2.stl"/>
-        </geometry>
-        <material name="3d_printed"/>
-      </visual>
-      <collision>
-        <origin xyz="0.0205915 0.0467435 0.0798817" rpy="1.5708 -1.21716e-14 2.33147e-15"/>
-        <geometry>
-          <mesh filename="file://$(find so_arm_description)/meshes/so101/waveshare_mounting_plate_so101_v2.stl"/>
+      <visual>
+        <geometry>
+          <mesh filename="file://$(find so_arm_description)/meshes/so101/base_motor_holder.stl"/>
+        </geometry>
+        <material name="3d_printed"/>
+      </visual>
+      <collision>
+        <geometry>
+          <mesh filename="file://$(find so_arm_description)/meshes/so101/base_motor_holder.stl"/>
+        </geometry>
+      </collision>
+      <visual>
+        <geometry>
+          <mesh filename="file://$(find so_arm_description)/meshes/so101/base.stl"/>
+        </geometry>
+        <material name="3d_printed"/>
+      </visual>
+      <collision>
+        <geometry>
+          <mesh filename="file://$(find so_arm_description)/meshes/so101/base.stl"/>
+        </geometry>
+      </collision>
+      <visual>
+        <geometry>
+          <mesh filename="file://$(find so_arm_description)/meshes/so101/base_waveshare_mounting_plate.stl"/>
+        </geometry>
+        <material name="3d_printed"/>
+      </visual>
+      <collision>
+        <geometry>
+          <mesh filename="file://$(find so_arm_description)/meshes/so101/base_waveshare_mounting_plate.stl"/>
         </geometry>
       </collision>
@@ -68,13 +52,8 @@
         <material name="sts3215"/>
       </visual>
-      <collision>
-        <geometry>
-          <mesh filename="file://$(find so_arm_description)/meshes/so101/sts3215_03a_v1.stl"/>
-        </geometry>
-      </collision>
     </link>
     <joint name="${prefix}motor1_joint" type="fixed">
-      <origin xyz="0.0207909 -0.0105745 0.0761817" rpy="-2.20282e-15 2.77556e-17 -1.5708"/>
-      <parent link="${prefix}base"/>
+      <origin xyz="0.0263345 0 0.0437"/>
+      <parent link="${prefix}base_link"/>
       <child link="${prefix}motor1"/>
     </joint>
@@ -82,51 +61,41 @@
     <link name="${prefix}shoulder">
       <inertial>
-        <origin xyz="-0.0307604 -1.66727e-05 -0.0252713" rpy="0 0 0"/>
+        <origin xyz="-0.0307604 -1.66727e-05 -0.0252713" />
         <mass value="0.100006"/>
         <inertia ixx="8.3759e-05" ixy="7.55525e-08" ixz="-1.16342e-06" iyy="8.10403e-05" iyz="1.54663e-07"
                  izz="2.39783e-05"/>
       </inertial>
-      <!-- Part motor_holder_so101_base_v1 -->
-      <visual>
-        <origin xyz="-0.0675992 -0.000177759 0.0158499" rpy="1.5708 -1.5708 0"/>
-        <geometry>
-          <mesh filename="file://$(find so_arm_description)/meshes/so101/motor_holder_so101_base_v1.stl"/>
-        </geometry>
-        <material name="3d_printed"/>
-      </visual>
-      <collision>
-        <origin xyz="-0.0675992 -0.000177759 0.0158499" rpy="1.5708 -1.5708 0"/>
-        <geometry>
-          <mesh filename="file://$(find so_arm_description)/meshes/so101/motor_holder_so101_base_v1.stl"/>
+      <!-- Part motor_holder_base_v1 -->
+      <visual>
+        <geometry>
+          <mesh filename="file://$(find so_arm_description)/meshes/so101/motor_holder_base.stl"/>
+        </geometry>
+        <material name="3d_printed"/>
+      </visual>
+      <collision>
+        <geometry>
+          <mesh filename="file://$(find so_arm_description)/meshes/so101/motor_holder_base.stl"/>
         </geometry>
       </collision>
       <!-- Part rotation_pitch_so101_v1 -->
       <visual>
-        <origin xyz="0.0122008 2.22413e-05 0.0464" rpy="-1.5708 -0 0"/>
-        <geometry>
-          <mesh filename="file://$(find so_arm_description)/meshes/so101/rotation_pitch_so101_v1.stl"/>
-        </geometry>
-        <material name="3d_printed"/>
-      </visual>
-      <collision>
-        <origin xyz="0.0122008 2.22413e-05 0.0464" rpy="-1.5708 -0 0"/>
-        <geometry>
-          <mesh filename="file://$(find so_arm_description)/meshes/so101/rotation_pitch_so101_v1.stl"/>
+        <geometry>
+          <mesh filename="file://$(find so_arm_description)/meshes/so101/rotation_pitch.stl"/>
+        </geometry>
+        <material name="3d_printed"/>
+      </visual>
+      <collision>
+        <geometry>
+          <mesh filename="file://$(find so_arm_description)/meshes/so101/rotation_pitch.stl"/>
         </geometry>
       </collision>
     </link>
     <link name="${prefix}motor2">
-      <!-- Part sts3215_03a_v1_2 -->
-      <visual>
-        <geometry>
-          <mesh filename="file://$(find so_arm_description)/meshes/so101/sts3215_03a_v1.stl"/>
-        </geometry>
-        <material name="sts3215"/>
-      </visual>
-      <collision>
-        <geometry>
-          <mesh filename="file://$(find so_arm_description)/meshes/so101/sts3215_03a_v1.stl"/>
-        </geometry>
-      </collision>
+      <visual>
+        <geometry>
+          <mesh filename="file://$(find so_arm_description)/meshes/so101/sts3215_03a_v1.stl"/>
+        </geometry>
+        <material name="sts3215"/>
+      </visual>
     </link>
     <joint name="${prefix}motor2_joint" type="fixed">
@@ -137,6 +106,6 @@
     <!-- Joint from base to shoulder -->
     <joint name="${prefix}shoulder_pan" type="revolute">
-      <origin xyz="0.0207909 -0.0230745 0.0948817" rpy="-3.14159 6.03684e-16 1.5708"/>
-      <parent link="${prefix}base"/>
+      <origin xyz="0.0388353 0 0.0624" rpy="-3.14159 0 3.14159"/>
+      <parent link="${prefix}base_link"/>
       <child link="${prefix}shoulder"/>
       <axis xyz="0 0 1"/>
@@ -146,37 +115,28 @@
     <link name="${prefix}upper_arm">
       <inertial>
-        <origin xyz="-0.0898471 -0.00838224 0.0184089" rpy="0 0 0"/>
+        <origin xyz="-0.0898471 -0.00838224 0.0184089" />
         <mass value="0.103"/>
         <inertia ixx="4.08002e-05" ixy="-1.97819e-05" ixz="-4.03016e-08" iyy="0.000147318" iyz="8.97326e-09"
                  izz="0.000142487"/>
       </inertial>
-      <!-- Part upper_arm_so101_v1 -->
-      <visual>
-        <origin xyz="-0.065085 0.012 0.0182" rpy="3.14159 -9.35612e-32 0"/>
-        <geometry>
-          <mesh filename="file://$(find so_arm_description)/meshes/so101/upper_arm_so101_v1.stl"/>
-        </geometry>
-        <material name="3d_printed"/>
-      </visual>
-      <collision>
-        <origin xyz="-0.065085 0.012 0.0182" rpy="3.14159 -9.35612e-32 0"/>
-        <geometry>
-          <mesh filename="file://$(find so_arm_description)/meshes/so101/upper_arm_so101_v1.stl"/>
+      <visual>
+        <geometry>
+          <mesh filename="file://$(find so_arm_description)/meshes/so101/upper_arm.stl"/>
+        </geometry>
+        <material name="3d_printed"/>
+      </visual>
+      <collision>
+        <geometry>
+          <mesh filename="file://$(find so_arm_description)/meshes/so101/upper_arm.stl"/>
         </geometry>
       </collision>
     </link>
     <link name="${prefix}motor3">
-      <!-- Part sts3215_03a_v1_3 -->
-      <visual>
-        <geometry>
-          <mesh filename="file://$(find so_arm_description)/meshes/so101/sts3215_03a_v1.stl"/>
-        </geometry>
-        <material name="sts3215"/>
-      </visual>
-      <collision>
-        <geometry>
-          <mesh filename="file://$(find so_arm_description)/meshes/so101/sts3215_03a_v1.stl"/>
-        </geometry>
-      </collision>
+      <visual>
+        <geometry>
+          <mesh filename="file://$(find so_arm_description)/meshes/so101/sts3215_03a_v1.stl"/>
+        </geometry>
+        <material name="sts3215"/>
+      </visual>
     </link>
     <joint name="${prefix}motor3_joint" type="fixed">
@@ -196,5 +156,5 @@
     <link name="${prefix}lower_arm">
       <inertial>
-        <origin xyz="-0.0980701 0.00324376 0.0182831" rpy="0 0 0"/>
+        <origin xyz="-0.0980701 0.00324376 0.0182831"/>
         <mass value="0.104"/>
         <inertia ixx="2.87438e-05" ixy="7.41152e-06" ixz="1.26409e-06" iyy="0.000159844" iyz="-4.90188e-08"
@@ -203,44 +163,34 @@
       <!-- Part under_arm_so101_v1 -->
       <visual>
-        <origin xyz="-0.0648499 -0.032 0.0182" rpy="-3.14159 -0 3.9443e-31"/>
-        <geometry>
-          <mesh filename="file://$(find so_arm_description)/meshes/so101/under_arm_so101_v1.stl"/>
-        </geometry>
-        <material name="3d_printed"/>
-      </visual>
-      <collision>
-        <origin xyz="-0.0648499 -0.032 0.0182" rpy="-3.14159 -0 3.9443e-31"/>
-        <geometry>
-          <mesh filename="file://$(find so_arm_description)/meshes/so101/under_arm_so101_v1.stl"/>
-        </geometry>
-      </collision>
-      <!-- Part motor_holder_so101_wrist_v1 -->
-      <visual>
-        <origin xyz="-0.0648499 -0.032 0.018" rpy="-3.14159 4.73317e-30 7.88861e-31"/>
-        <geometry>
-          <mesh filename="file://$(find so_arm_description)/meshes/so101/motor_holder_so101_wrist_v1.stl"/>
-        </geometry>
-        <material name="3d_printed"/>
-      </visual>
-      <collision>
-        <origin xyz="-0.0648499 -0.032 0.018" rpy="-3.14159 4.73317e-30 7.88861e-31"/>
-        <geometry>
-          <mesh filename="file://$(find so_arm_description)/meshes/so101/motor_holder_so101_wrist_v1.stl"/>
+        <geometry>
+          <mesh filename="file://$(find so_arm_description)/meshes/so101/under_arm.stl"/>
+        </geometry>
+        <material name="3d_printed"/>
+      </visual>
+      <collision>
+        <geometry>
+          <mesh filename="file://$(find so_arm_description)/meshes/so101/under_arm.stl"/>
+        </geometry>
+      </collision>
+      <!-- Part motor_holder_wrist_v1 -->
+      <visual>
+        <geometry>
+          <mesh filename="file://$(find so_arm_description)/meshes/so101/motor_holder_wrist.stl"/>
+        </geometry>
+        <material name="3d_printed"/>
+      </visual>
+      <collision>
+        <geometry>
+          <mesh filename="file://$(find so_arm_description)/meshes/so101/motor_holder_wrist.stl"/>
         </geometry>
       </collision>
     </link>
     <link name="${prefix}motor4">
-      <!-- Part sts3215_03a_v1_4 -->
-      <visual>
-        <geometry>
-          <mesh filename="file://$(find so_arm_description)/meshes/so101/sts3215_03a_v1.stl"/>
-        </geometry>
-        <material name="sts3215"/>
-      </visual>
-      <collision>
-        <geometry>
-          <mesh filename="file://$(find so_arm_description)/meshes/so101/sts3215_03a_v1.stl"/>
-        </geometry>
-      </collision>
+      <visual>
+        <geometry>
+          <mesh filename="file://$(find so_arm_description)/meshes/so101/sts3215_03a_v1.stl"/>
+        </geometry>
+        <material name="sts3215"/>
+      </visual>
     </link>
     <joint name="${prefix}motor4_joint" type="fixed">
@@ -261,5 +211,5 @@
     <link name="${prefix}wrist">
       <inertial>
-        <origin xyz="-0.000103312 -0.0386143 0.0281156" rpy="0 0 0"/>
+        <origin xyz="-0.000103312 -0.0386143 0.0281156" />
         <mass value="0.079"/>
         <inertia ixx="3.68263e-05" ixy="1.7893e-08" ixz="-5.28128e-08" iyy="2.5391e-05" iyz="3.6412e-06" izz="2.1e-05"/>
@@ -267,30 +217,22 @@
       <!-- Part wrist_roll_pitch_so101_v2 -->
       <visual>
-        <origin xyz="0 -0.028 0.0181" rpy="-1.5708 -1.5708 0"/>
-        <geometry>
-          <mesh filename="file://$(find so_arm_description)/meshes/so101/wrist_roll_pitch_so101_v2.stl"/>
-        </geometry>
-        <material name="3d_printed"/>
-      </visual>
-      <collision>
-        <origin xyz="0 -0.028 0.0181" rpy="-1.5708 -1.5708 0"/>
-        <geometry>
-          <mesh filename="file://$(find so_arm_description)/meshes/so101/wrist_roll_pitch_so101_v2.stl"/>
+        <geometry>
+          <mesh filename="file://$(find so_arm_description)/meshes/so101/wrist_roll_pitch.stl"/>
+        </geometry>
+        <material name="3d_printed"/>
+      </visual>
+      <collision>
+        <geometry>
+          <mesh filename="file://$(find so_arm_description)/meshes/so101/wrist_roll_pitch.stl"/>
         </geometry>
       </collision>
     </link>
     <link name="${prefix}motor5">
-      <!-- Part sts3215_03a_v1_6 -->
-      <visual>
-        <geometry>
-          <mesh filename="file://$(find so_arm_description)/meshes/so101/sts3215_03a_v1.stl"/>
-        </geometry>
-        <material name="sts3215"/>
-      </visual>
-      <collision>
-        <geometry>
-          <mesh filename="file://$(find so_arm_description)/meshes/so101/sts3215_03a_v1.stl"/>
-        </geometry>
-      </collision>
+      <visual>
+        <geometry>
+          <mesh filename="file://$(find so_arm_description)/meshes/so101/sts3215_03a_v1.stl"/>
+        </geometry>
+        <material name="sts3215"/>
+      </visual>
     </link>
     <joint name="${prefix}motor5_joint" type="fixed">
@@ -310,5 +252,5 @@
     <link name="${prefix}gripper">
       <inertial>
-        <origin xyz="0.000213627 0.000245138 -0.025187" rpy="0 0 0"/>
+        <origin xyz="0.000213627 0.000245138 -0.025187" />
         <mass value="0.087"/>
         <inertia ixx="2.75087e-05" ixy="-3.35241e-07" ixz="-5.7352e-06" iyy="4.33657e-05" iyz="-5.17847e-08"
@@ -317,30 +259,32 @@
       <!-- Part wrist_roll_follower_so101_v1 -->
       <visual>
-        <origin xyz="5.55112e-17 -0.000218214 0.000949706" rpy="-3.14159 -5.55112e-17 -9.17912e-24"/>
-        <geometry>
-          <mesh filename="file://$(find so_arm_description)/meshes/so101/wrist_roll_follower_so101_v1.stl"/>
-        </geometry>
-        <material name="3d_printed"/>
-      </visual>
-      <collision>
-        <origin xyz="5.55112e-17 -0.000218214 0.000949706" rpy="-3.14159 -5.55112e-17 -9.17912e-24"/>
-        <geometry>
-          <mesh filename="file://$(find so_arm_description)/meshes/so101/wrist_roll_follower_so101_v1.stl"/>
+        <geometry>
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