Commit message: modified mesh

File: manipulator/AgileX/mobile_aloha2_description/xacro/robot.xacro (robot description, xacro)
@@ -282,14 +282,11 @@
       <origin xyz="0 0 0.168" rpy="0 0 3.14"/>
       <geometry>
-        <mesh filename="package://mobile_aloha2_description/meshes/body.dae"/>
-      </geometry>
-      <material name="">
-        <color rgba="0.79216 0.81961 0.93333 1"/>
-      </material>
+        <mesh filename="package://mobile_aloha2_description/meshes/body.obj"/>
+      </geometry>
     </visual>
     <collision>
       <origin xyz="0 0 0.168" rpy="0 0 3.14"/>
       <geometry>
-        <mesh filename="package://mobile_aloha2_description/meshes/body.dae"/>
+        <mesh filename="package://mobile_aloha2_description/meshes/body.obj"/>
       </geometry>
     </collision>

Commit message: modified mesh

File: manipulator/AgileX/mobile_aloha2_description/xacro/robot.xacro (robot description, xacro)
@@ -9,16 +9,12 @@
     <visual>
       <origin xyz="0 0 0" rpy="1.57 0 0"/>
-      <!--<origin xyz="0 0 0" rpy="0 0 0"/>-->
-      <geometry>
-        <mesh filename="package://mobile_aloha2_description/meshes/tracer_base_link_no_wheel.dae"/>
-      </geometry>
-    </visual>
-    <collision>
-      <!--origin
-        xyz="-0.0145261552504705 0.0231316650320557 0.00586280190939592"
-        rpy="0 0 0" /-->
+      <geometry>
+        <mesh filename="package://mobile_aloha2_description/meshes/tracer_base_link.obj"/>
+      </geometry>
+    </visual>
+    <collision>
       <origin xyz="0 0 0" rpy="1.57 0 0"/>
       <geometry>
-        <mesh filename="package://mobile_aloha2_description/meshes/tracer_base_link_no_wheel.dae"/>
+        <mesh filename="package://mobile_aloha2_description/meshes/tracer_base_link.obj"/>
       </geometry>
     </collision>
@@ -52,16 +48,14 @@
     <inertial>
       <mass value="6"/>
-      <origin xyz="0 0 0"/>
-      <inertia ixx="0.7171" ixy="0" ixz="0" iyy="0.1361" iyz="0" izz="0.7171"/>
-    </inertial>
-    <visual>
-      <origin xyz="0 0 0" rpy="0 0 0"/>
-      <geometry>
-        <mesh filename="package://mobile_aloha2_description/meshes/tracer_wheel.dae"/>
-      </geometry>
-    </visual>
-    <collision>
-      <geometry>
-        <mesh filename="package://mobile_aloha2_description/meshes/tracer_wheel.dae"/>
+      <inertia ixx="0.7171" ixy="0" ixz="0" iyy="0.1361" iyz="0" izz="0.7171"/>
+    </inertial>
+    <visual>
+      <geometry>
+        <mesh filename="package://mobile_aloha2_description/meshes/tracer_wheel.obj"/>
+      </geometry>
+    </visual>
+    <collision>
+      <geometry>
+        <mesh filename="package://mobile_aloha2_description/meshes/tracer_wheel.obj"/>
       </geometry>
     </collision>
@@ -76,16 +70,14 @@
     <inertial>
       <mass value="6"/>
-      <origin xyz="0 0 0"/>
-      <inertia ixx="0.7171" ixy="0" ixz="0" iyy="0.1361" iyz="0" izz="0.7171"/>
-    </inertial>
-    <visual>
-      <origin xyz="0 0 0" rpy="0 0 0"/>
-      <geometry>
-        <mesh filename="package://mobile_aloha2_description/meshes/tracer_wheel.dae"/>
-      </geometry>
-    </visual>
-    <collision>
-      <geometry>
-        <mesh filename="package://mobile_aloha2_description/meshes/tracer_wheel.dae"/>
+      <inertia ixx="0.7171" ixy="0" ixz="0" iyy="0.1361" iyz="0" izz="0.7171"/>
+    </inertial>
+    <visual>
+      <geometry>
+        <mesh filename="package://mobile_aloha2_description/meshes/tracer_wheel.obj"/>
+      </geometry>
+    </visual>
+    <collision>
+      <geometry>
+        <mesh filename="package://mobile_aloha2_description/meshes/tracer_wheel.obj"/>
       </geometry>
     </collision>
@@ -100,10 +92,9 @@
     <inertial>
       <mass value="1"/>
-      <origin xyz="0 0 0"/>
-      <inertia ixx="0.7171" ixy="0" ixz="0" iyy="0.1361" iyz="0" izz="0.7171"/>
-    </inertial>
-    <visual>
-      <geometry>
-        <mesh filename="package://mobile_aloha2_description/meshes/castor_joint.dae"/>
+      <inertia ixx="0.7171" ixy="0" ixz="0" iyy="0.1361" iyz="0" izz="0.7171"/>
+    </inertial>
+    <visual>
+      <geometry>
+        <mesh filename="package://mobile_aloha2_description/meshes/castor_joint.obj"/>
       </geometry>
     </visual>
@@ -118,10 +109,9 @@
     <inertial>
       <mass value="1"/>
-      <origin xyz="0 0 0"/>
-      <inertia ixx="0.7171" ixy="0" ixz="0" iyy="0.1361" iyz="0" izz="0.7171"/>
-    </inertial>
-    <visual>
-      <geometry>
-        <mesh filename="package://mobile_aloha2_description/meshes/castor_joint.dae"/>
+      <inertia ixx="0.7171" ixy="0" ixz="0" iyy="0.1361" iyz="0" izz="0.7171"/>
+    </inertial>
+    <visual>
+      <geometry>
+        <mesh filename="package://mobile_aloha2_description/meshes/castor_joint.obj"/>
       </geometry>
     </visual>
@@ -136,10 +126,9 @@
     <inertial>
       <mass value="1"/>
-      <origin xyz="0 0 0"/>
-      <inertia ixx="0.7171" ixy="0" ixz="0" iyy="0.1361" iyz="0" izz="0.7171"/>
-    </inertial>
-    <visual>
-      <geometry>
-        <mesh filename="package://mobile_aloha2_description/meshes/castor_joint.dae"/>
+      <inertia ixx="0.7171" ixy="0" ixz="0" iyy="0.1361" iyz="0" izz="0.7171"/>
+    </inertial>
+    <visual>
+      <geometry>
+        <mesh filename="package://mobile_aloha2_description/meshes/castor_joint.obj"/>
       </geometry>
     </visual>
@@ -154,10 +143,9 @@
     <inertial>
       <mass value="1"/>
-      <origin xyz="0 0 0"/>
-      <inertia ixx="0.7171" ixy="0" ixz="0" iyy="0.1361" iyz="0" izz="0.7171"/>
-    </inertial>
-    <visual>
-      <geometry>
-        <mesh filename="package://mobile_aloha2_description/meshes/castor_joint.dae"/>
+      <inertia ixx="0.7171" ixy="0" ixz="0" iyy="0.1361" iyz="0" izz="0.7171"/>
+    </inertial>
+    <visual>
+      <geometry>
+        <mesh filename="package://mobile_aloha2_description/meshes/castor_joint.obj"/>
       </geometry>
     </visual>
@@ -172,15 +160,14 @@
     <inertial>
       <mass value="1"/>
-      <origin xyz="0 0 0"/>
       <inertia ixx="0.3131" ixy="0" ixz="0" iyy="0.3131" iyz="0" izz="0.1361"/>
     </inertial>
     <visual>
       <geometry>
-        <mesh filename="package://mobile_aloha2_description/meshes/castor.dae"/>
+        <mesh filename="package://mobile_aloha2_description/meshes/castor.obj"/>
       </geometry>
     </visual>
     <collision>
       <geometry>-->
-        <mesh filename="package://mobile_aloha2_description/meshes/castor.dae"/>
+        <mesh filename="package://mobile_aloha2_description/meshes/castor.obj"/>
       </geometry>
     </collision>
@@ -196,15 +183,14 @@
     <inertial>
       <mass value="1"/>
-      <origin xyz="0 0 0"/>
       <inertia ixx="0.3131" ixy="0" ixz="0" iyy="0.3131" iyz="0" izz="0.1361"/>
     </inertial>
     <visual>
       <geometry>
-        <mesh filename="package://mobile_aloha2_description/meshes/castor.dae"/>
+        <mesh filename="package://mobile_aloha2_description/meshes/castor.obj"/>
       </geometry>
     </visual>
     <collision>
       <geometry>-->
-        <mesh filename="package://mobile_aloha2_description/meshes/castor.dae"/>
+        <mesh filename="package://mobile_aloha2_description/meshes/castor.obj"/>
       </geometry>
     </collision>
@@ -220,16 +206,14 @@
     <inertial>
       <mass value="1"/>
-      <origin xyz="0 0 0"/>
       <inertia ixx="0.3131" ixy="0" ixz="0" iyy="0.3131" iyz="0" izz="0.1361"/>
-      <!--<inertia ixx="0" ixy="0" ixz="0" iyy="0" iyz="0" izz="0" />-->
-    </inertial>
-    <visual>
-      <geometry>
-        <mesh filename="package://mobile_aloha2_description/meshes/castor.dae"/>
-      </geometry>
-    </visual>
-    <collision>
-      <geometry>
-        <mesh filename="package://mobile_aloha2_description/meshes/castor.dae"/>
+    </inertial>
+    <visual>
+      <geometry>
+        <mesh filename="package://mobile_aloha2_description/meshes/castor.obj"/>
+      </geometry>
+    </visual>
+    <collision>
+      <geometry>
+        <mesh filename="package://mobile_aloha2_description/meshes/castor.obj"/>
       </geometry>
     </collision>
@@ -245,15 +229,14 @@
     <inertial>
       <mass value="1"/>
-      <origin xyz="0 0 0"/>
       <inertia ixx="0.3131" ixy="0" ixz="0" iyy="0.3131" iyz="0" izz="0.1361"/>
     </inertial>
     <visual>
       <geometry>
-        <mesh filename="package://mobile_aloha2_description/meshes/castor.dae"/>
-      </geometry>
-    </visual>
-    <collision>
-      <geometry>
-        <mesh filename="package://mobile_aloha2_description/meshes/castor.dae"/>
+        <mesh filename="package://mobile_aloha2_description/meshes/castor.obj"/>
+      </geometry>
+    </visual>
+    <collision>
+      <geometry>
+        <mesh filename="package://mobile_aloha2_description/meshes/castor.obj"/>
       </geometry>
     </collision>
