Commit message: remove undesired meshes

File: manipulator/LeRobot/lekiwi_description/xacro/base.xacro (robot description, xacro)
@@ -18,8 +18,8 @@
       <color rgba="0.4 0.8196 0.945 1.0"/>
     </material>
-    <link name="base_link"/>
-    <joint name="base_joint" type="fixed">
+    <link name="${prefix}base_link"/>
+    <joint name="${prefix}base_joint" type="fixed">
       <origin rpy="0 0 -1.5708"/>
-      <parent link="base_link"/>
+      <parent link="${prefix}base_link"/>
       <child link="base_plate_layer1-v5"/>
     </joint>

File: manipulator/LeRobot/lekiwi_description/xacro/robot.xacro (robot description, xacro)
@@ -4,5 +4,4 @@
   <xacro:include filename="$(find lekiwi_description)/xacro/base.xacro"/>
   <xacro:mobile_base name=""/>
-  <!-- 根据type参数决定is_master的值 -->
   <xacro:if value="${'$(arg type)' == 'so101'}">
     <xacro:include filename="$(find so_arm_description)/xacro/so101.xacro"/>

File: manipulator/LeRobot/so_arm_description/xacro/robot.xacro (robot description, xacro)
@@ -1,7 +1,6 @@
 <?xml version="1.0"?>
-<robot name="Piper single" xmlns:xacro="http://www.ros.org/wiki/xacro">
+<robot name="SO-Arm" xmlns:xacro="http://www.ros.org/wiki/xacro">
   <!-- Materials -->
   <material name="3d_printed">
-<!--    <color rgba="1.0 0.82 0.12 1.0"/>-->
     <color rgba="0.4 0.8196 0.945 1.0"/>
   </material>
