Commit message: add galaxea R1 robot

File: manipulator/Galaxea/galaxea_a1_description/xacro/a1_x.xacro (robot description, xacro)
@@ -2,5 +2,5 @@
 <robot xmlns:xacro="http://www.ros.org/wiki/xacro">
   <xacro:macro name="Arm" params="name">
-    <xacro:include filename="$(find a1xy_description)/xacro/xy_base.xacro"/>
+    <xacro:include filename="(find galaxea_a1_description)/xacro/a1xy_base.xacro"/>
     <xacro:property name="prefix" value="${name + '_' if name else ''}"/>
     <xacro:Base name=""/>
@@ -23,10 +23,10 @@
       <visual>
         <geometry>
-          <mesh filename="file://$(find a1xy_description)/meshes/x_link/link3.obj"/>
+          <mesh filename="file://$(find galaxea_a1_description)/meshes/a1_xy/a1_x/link3.obj"/>
         </geometry>
       </visual>
       <collision>
         <geometry>
-          <mesh filename="file://$(find a1xy_description)/meshes/x_link/link3.obj"/>
+          <mesh filename="file://$(find galaxea_a1_description)/meshes/a1_xy/a1_x/link3.obj"/>
         </geometry>
       </collision>
@@ -68,10 +68,10 @@
       <visual>
         <geometry>
-          <mesh filename="file://$(find a1xy_description)/meshes/x_link/link4.obj"/>
+          <mesh filename="file://$(find galaxea_a1_description)/meshes/a1_xy/a1_x/link4.obj"/>
         </geometry>
       </visual>
       <collision>
         <geometry>
-          <mesh filename="file://$(find a1xy_description)/meshes/x_link/link4.obj"/>
+          <mesh filename="file://$(find galaxea_a1_description)/meshes/a1_xy/a1_x/link4.obj"/>
         </geometry>
       </collision>
@@ -113,10 +113,10 @@
       <visual>
         <geometry>
-          <mesh filename="file://$(find a1xy_description)/meshes/x_link/link5.obj"/>
+          <mesh filename="file://$(find galaxea_a1_description)/meshes/a1_xy/a1_x/link5.obj"/>
         </geometry>
       </visual>
       <collision>
         <geometry>
-          <mesh filename="file://$(find a1xy_description)/meshes/x_link/link5.obj"/>
+          <mesh filename="file://$(find galaxea_a1_description)/meshes/a1_xy/a1_x/link5.obj"/>
         </geometry>
       </collision>
@@ -158,10 +158,10 @@
       <visual>
         <geometry>
-          <mesh filename="file://$(find a1xy_description)/meshes/link6.obj"/>
+          <mesh filename="file://$(find galaxea_a1_description)/meshes/a1_xy/link6.obj"/>
         </geometry>
       </visual>
       <collision>
         <geometry>
-          <mesh filename="file://$(find a1xy_description)/meshes/link6.obj"/>
+          <mesh filename="file://$(find galaxea_a1_description)/meshes/a1_xy/link6.obj"/>
         </geometry>
       </collision>
@@ -185,5 +185,5 @@
           velocity="32.9867"/>
     </joint>
-    <xacro:include filename="$(find a1xy_description)/xacro/gripper.xacro"/>
+    <xacro:include filename="(find galaxea_a1_description)/xacro/gripper.xacro"/>
     <xacro:Gripper name="${name}"/>
     <joint name="${prefix}gripper_joint" type="fixed">

File: manipulator/Galaxea/galaxea_a1_description/xacro/a1_y.xacro (robot description, xacro)
@@ -2,5 +2,5 @@
 <robot xmlns:xacro="http://www.ros.org/wiki/xacro">
   <xacro:macro name="Arm" params="name">
-    <xacro:include filename="$(find a1xy_description)/xacro/xy_base.xacro"/>
+    <xacro:include filename="(find galaxea_a1_description)/xacro/a1xy_base.xacro"/>
     <xacro:property name="prefix" value="${name + '_' if name else ''}"/>
     <xacro:Base name=""/>
@@ -19,10 +19,10 @@
       <visual>
         <geometry>
-          <mesh filename="file://$(find a1xy_description)/meshes/y_link/link3.obj" />
-        </geometry>
-      </visual>
-      <collision>
-        <geometry>
-          <mesh filename="file://$(find a1xy_description)/meshes/y_link/link3.obj" />
+          <mesh filename="file://$(find galaxea_a1_description)/meshes/a1_xy/a1_y/link3.obj" />
+        </geometry>
+      </visual>
+      <collision>
+        <geometry>
+          <mesh filename="file://$(find galaxea_a1_description)/meshes/a1_xy/a1_y/link3.obj" />
         </geometry>
       </collision>
@@ -65,5 +65,5 @@
         <geometry>
           <mesh
-              filename="file://$(find a1xy_description)/meshes/y_link/link4.obj" />
+              filename="file://$(find galaxea_a1_description)/meshes/a1_xy/a1_y/link4.obj" />
         </geometry>
         <material
@@ -76,5 +76,5 @@
         <geometry>
           <mesh
-              filename="file://$(find a1xy_description)/meshes/y_link/link4.obj" />
+              filename="file://$(find galaxea_a1_description)/meshes/a1_xy/a1_y/link4.obj" />
         </geometry>
       </collision>
@@ -117,5 +117,5 @@
         <geometry>
           <mesh
-              filename="file://$(find a1xy_description)/meshes/y_link/link5.obj" />
+              filename="file://$(find galaxea_a1_description)/meshes/a1_xy/a1_y/link5.obj" />
         </geometry>
         <material
@@ -128,5 +128,5 @@
         <geometry>
           <mesh
-              filename="file://$(find a1xy_description)/meshes/y_link/link5.obj" />
+              filename="file://$(find galaxea_a1_description)/meshes/a1_xy/a1_y/link5.obj" />
         </geometry>
       </collision>
@@ -169,5 +169,5 @@
         <geometry>
           <mesh
-              filename="file://$(find a1xy_description)/meshes/link6.obj" />
+              filename="file://$(find a1xy_description)/meshes/a1_xy/link6.obj" />
         </geometry>
         <material
@@ -180,5 +180,5 @@
         <geometry>
           <mesh
-              filename="file://$(find a1xy_description)/meshes/link6.obj" />
+              filename="file://$(find a1xy_description)/meshes/a1_xy/link6.obj" />
         </geometry>
       </collision>
@@ -202,5 +202,5 @@
           velocity="32.9867" />
     </joint>
-    <xacro:include filename="$(find a1xy_description)/xacro/gripper.xacro"/>
+    <xacro:include filename="(find galaxea_a1_description)/xacro/gripper.xacro"/>
     <xacro:Gripper name="${name}"/>
     <joint name="${prefix}gripper_joint" type="fixed">

File: manipulator/Galaxea/galaxea_a1_description/xacro/a1xy_base.xacro (robot description, xacro)
@@ -19,10 +19,10 @@
       <visual>
         <geometry>
-          <mesh filename="file://$(find a1xy_description)/meshes/xy_base/base_link.obj"/>
+          <mesh filename="file://$(find galaxea_a1_description)/meshes/a1_xy/base_link.obj"/>
         </geometry>
       </visual>
       <collision>
         <geometry>
-          <mesh filename="file://$(find a1xy_description)/meshes/xy_base/base_link.obj"/>
+          <mesh filename="file://$(find galaxea_a1_description)/meshes/a1_xy/base_link.obj"/>
         </geometry>
       </collision>
@@ -50,5 +50,5 @@
         <geometry>
           <mesh
-              filename="file://$(find a1xy_description)/meshes/xy_base/link1.obj"/>
+              filename="file://$(find galaxea_a1_description)/meshes/a1_xy/link1.obj"/>
         </geometry>
         <material
@@ -64,5 +64,5 @@
         <geometry>
           <mesh
-              filename="file://$(find a1xy_description)/meshes/xy_base/link1.obj"/>
+              filename="file://$(find galaxea_a1_description)/meshes/a1_xy/link1.obj"/>
         </geometry>
       </collision>
@@ -108,5 +108,5 @@
         <geometry>
           <mesh
-              filename="file://$(find a1xy_description)/meshes/xy_base/link2.obj"/>
+              filename="file://$(find galaxea_a1_description)/meshes/a1_xy/link2.obj"/>
         </geometry>
         <material
@@ -122,5 +122,5 @@
         <geometry>
           <mesh
-              filename="file://$(find a1xy_description)/meshes/xy_base/link2.obj"/>
+              filename="file://$(find galaxea_a1_description)/meshes/a1_xy/link2.obj"/>
         </geometry>
       </collision>

File: manipulator/Galaxea/galaxea_a1_description/xacro/gripper.xacro (robot description, xacro)
@@ -17,10 +17,10 @@
       <visual>
         <geometry>
-          <mesh filename="file://$(find a1xy_description)/meshes/gripper/gripper_link.obj"/>
+          <mesh filename="file://$(find galaxea_a1_description)/meshes/gripper/gripper_link.obj"/>
         </geometry>
       </visual>
       <collision>
         <geometry>
-          <mesh filename="file://$(find a1xy_description)/meshes/gripper/gripper_link.obj"/>
+          <mesh filename="file://$(find galaxea_a1_description)/meshes/gripper/gripper_link.obj"/>
         </geometry>
       </collision>
@@ -40,10 +40,10 @@
       <visual>
         <geometry>
-          <mesh filename="file://$(find a1xy_description)/meshes/gripper/gripper_finger1.obj"/>
+          <mesh filename="file://$(find galaxea_a1_description)/meshes/gripper/gripper_finger1.obj"/>
         </geometry>
       </visual>
       <collision>
         <geometry>
-          <mesh filename="file://$(find a1xy_description)/meshes/gripper/gripper_finger1.obj"/>
+          <mesh filename="file://$(find galaxea_a1_description)/meshes/gripper/gripper_finger1.obj"/>
         </geometry>
       </collision>
@@ -70,10 +70,10 @@
       <visual>
         <geometry>
-          <mesh filename="file://$(find a1xy_description)/meshes/gripper/gripper_finger2.obj"/>
+          <mesh filename="file://$(find galaxea_a1_description)/meshes/gripper/gripper_finger2.obj"/>
         </geometry>
       </visual>
       <collision>
         <geometry>
-          <mesh filename="file://$(find a1xy_description)/meshes/gripper/gripper_finger2.obj"/>
+          <mesh filename="file://$(find galaxea_a1_description)/meshes/gripper/gripper_finger2.obj"/>
         </geometry>
       </collision>
@@ -85,5 +85,5 @@
       <axis xyz="0 -1 0"/>
       <limit lower="0" upper="0.05" effort="100" velocity="0.25"/>
-      <mimic joint="gripper_finger_joint1" multiplier="1" offset="0"/>
+      <mimic joint="${prefix}gripper_finger_joint1" multiplier="1" offset="0"/>
     </joint>
   </xacro:macro>
