Commit message: add realman rm65, inspire eg2, realman aidal, galaxea g1

File: gripper/galaxea_g1_description/xacro/gripper.xacro (robot description, xacro)
@@ -3,5 +3,5 @@
   <xacro:macro name="Gripper" params="name">
     <xacro:property name="prefix" value="${name + '_' if name else ''}"/>
-    <link name="${prefix}gripper_link">
+    <link name="${prefix}base_link">
       <inertial>
         <origin xyz="-0.0311072323899603 1.17979991887118E-08 7.93394685505433E-08"/>
@@ -17,14 +17,14 @@
       <visual>
         <geometry>
-          <mesh filename="file://$(find galaxea_a1_description)/meshes/gripper/gripper_link.obj"/>
+          <mesh filename="file://$(find galaxea_g1_description)/meshes/gripper_link.obj"/>
         </geometry>
       </visual>
       <collision>
         <geometry>
-          <mesh filename="file://$(find galaxea_a1_description)/meshes/gripper/gripper_link.obj"/>
+          <mesh filename="file://$(find galaxea_g1_description)/meshes/gripper_link.obj"/>
         </geometry>
       </collision>
     </link>
-    <link name="${prefix}gripper_finger_link1">
+    <link name="${prefix}link1">
       <inertial>
         <origin xyz="-0.0195895895552112 -0.0151136845490034 0.00542254359093075"/>
@@ -40,21 +40,21 @@
       <visual>
         <geometry>
-          <mesh filename="file://$(find galaxea_a1_description)/meshes/gripper/gripper_finger1.obj"/>
+          <mesh filename="file://$(find galaxea_g1_description)/meshes/gripper_finger1.obj"/>
         </geometry>
       </visual>
       <collision>
         <geometry>
-          <mesh filename="file://$(find galaxea_a1_description)/meshes/gripper/gripper_finger1.obj"/>
+          <mesh filename="file://$(find galaxea_g1_description)/meshes/gripper_finger1.obj"/>
         </geometry>
       </collision>
     </link>
-    <joint name="${prefix}gripper_finger_joint1" type="prismatic">
+    <joint name="${prefix}joint1" type="prismatic">
       <origin xyz="0.03689 0.013453 0.00012059"/>
-      <parent link="${prefix}gripper_link"/>
-      <child link="${prefix}gripper_finger_link1"/>
+      <parent link="${prefix}base_link"/>
+      <child link="${prefix}link1"/>
       <axis xyz="0 1 0"/>
       <limit lower="0" upper="0.05" effort="100" velocity="0.25"/>
     </joint>
-    <link name="${prefix}gripper_finger_link2">
+    <link name="${prefix}link2">
       <inertial>
         <origin xyz="-0.0195895857999098 0.0151136893508115 -0.00542254357246619"/>
@@ -70,20 +70,20 @@
       <visual>
         <geometry>
-          <mesh filename="file://$(find galaxea_a1_description)/meshes/gripper/gripper_finger2.obj"/>
+          <mesh filename="file://$(find galaxea_g1_description)/meshes/gripper_finger2.obj"/>
         </geometry>
       </visual>
       <collision>
         <geometry>
-          <mesh filename="file://$(find galaxea_a1_description)/meshes/gripper/gripper_finger2.obj"/>
+          <mesh filename="file://$(find galaxea_g1_description)/meshes/gripper_finger2.obj"/>
         </geometry>
       </collision>
     </link>
-    <joint name="${prefix}gripper_finger_joint2" type="prismatic">
+    <joint name="${prefix}joint2" type="prismatic">
       <origin xyz="0.03689 -0.013453 -0.00012059"/>
-      <parent link="${prefix}gripper_link"/>
-      <child link="${prefix}gripper_finger_link2"/>
+      <parent link="${prefix}base_link"/>
+      <child link="${prefix}link2"/>
       <axis xyz="0 -1 0"/>
       <limit lower="0" upper="0.05" effort="100" velocity="0.25"/>
-      <mimic joint="${prefix}gripper_finger_joint1" multiplier="1" offset="0"/>
+      <mimic joint="${prefix}joint1" multiplier="1" offset="0"/>
     </joint>
   </xacro:macro>

File: manipulator/ARX/r5_description/xacro/R5.xacro (robot description, xacro)
@@ -1,5 +1,5 @@
 <?xml version="1.0"?>
 <robot xmlns:xacro="http://www.ros.org/wiki/xacro">
-  <xacro:macro name="R5" params="name">
+  <xacro:macro name="RM65" params="name">
     <xacro:property name="prefix" value="${name + '_' if name else ''}"/>
     <link name="${prefix}base_link">

File: manipulator/Galaxea/galaxea_a1_description/urdf/galaxea_a1.urdf (robot description, URDF)
Before this commit: robot A1 Single, 10 links, 9 joints
Links:
- removed link gripper_finger_link1
- removed link gripper_finger_link2
- removed link gripper_link
- added link gripper_base_link, mass 0.604; collision mesh filename=package://galaxea_g1_description/meshes/gripper_link.obj; visual mesh filename=package://galaxea_g1_description/meshes/gripper_link.obj
- added link gripper_link1, mass 0.027; collision mesh filename=package://galaxea_g1_description/meshes/gripper_finger1.obj; visual mesh filename=package://galaxea_g1_description/meshes/gripper_finger1.obj
- added link gripper_link2, mass 0.027; collision mesh filename=package://galaxea_g1_description/meshes/gripper_finger2.obj; visual mesh filename=package://galaxea_g1_description/meshes/gripper_finger2.obj
Joints:
- removed joint gripper_finger_joint1
- removed joint gripper_finger_joint2
- added joint gripper_joint1: type prismatic, parent gripper_base_link, child gripper_link1, origin xyz=0.03689 0.013453 0.00012059, axis 0 1 0, limit lower=0 upper=0.05 effort=100 velocity=0.25
- added joint gripper_joint2: type prismatic, parent gripper_base_link, child gripper_link2, origin xyz=0.03689 -0.013453 -0.00012059, axis 0 -1 0, limit lower=0 upper=0.05 effort=100 velocity=0.25, mimic joint=gripper_joint1 multiplier=1 offset=0
- joint gripper_joint: child gripper_link -> gripper_base_link; origin xyz=0.1039 0 0 rpy=-1.57 0 0 -> xyz=0.1039 0 0 rpy=-1.5708 0 0

File: manipulator/Galaxea/galaxea_a1_description/urdf/galaxea_a1_x.urdf (robot description, URDF)
Before this commit: robot A1 Single, 10 links, 9 joints
Links:
- removed link gripper_finger_link1
- removed link gripper_finger_link2
- removed link gripper_link
- added link gripper_base_link, mass 0.604; collision mesh filename=package://galaxea_g1_description/meshes/gripper_link.obj; visual mesh filename=package://galaxea_g1_description/meshes/gripper_link.obj
- added link gripper_link1, mass 0.027; collision mesh filename=package://galaxea_g1_description/meshes/gripper_finger1.obj; visual mesh filename=package://galaxea_g1_description/meshes/gripper_finger1.obj
- added link gripper_link2, mass 0.027; collision mesh filename=package://galaxea_g1_description/meshes/gripper_finger2.obj; visual mesh filename=package://galaxea_g1_description/meshes/gripper_finger2.obj
Joints:
- removed joint gripper_finger_joint1
- removed joint gripper_finger_joint2
- added joint gripper_joint1: type prismatic, parent gripper_base_link, child gripper_link1, origin xyz=0.03689 0.013453 0.00012059, axis 0 1 0, limit lower=0 upper=0.05 effort=100 velocity=0.25
- added joint gripper_joint2: type prismatic, parent gripper_base_link, child gripper_link2, origin xyz=0.03689 -0.013453 -0.00012059, axis 0 -1 0, limit lower=0 upper=0.05 effort=100 velocity=0.25, mimic joint=gripper_joint1 multiplier=1 offset=0
- joint gripper_joint: axis 0 0 0 -> (none); child gripper_link -> gripper_base_link

File: manipulator/Galaxea/galaxea_a1_description/urdf/galaxea_a1_y.urdf (robot description, URDF)
Before this commit: robot A1 Single, 10 links, 9 joints
Links:
- removed link gripper_finger_link1
- removed link gripper_finger_link2
- removed link gripper_link
- added link gripper_base_link, mass 0.604; collision mesh filename=package://galaxea_g1_description/meshes/gripper_link.obj; visual mesh filename=package://galaxea_g1_description/meshes/gripper_link.obj
- added link gripper_link1, mass 0.027; collision mesh filename=package://galaxea_g1_description/meshes/gripper_finger1.obj; visual mesh filename=package://galaxea_g1_description/meshes/gripper_finger1.obj
- added link gripper_link2, mass 0.027; collision mesh filename=package://galaxea_g1_description/meshes/gripper_finger2.obj; visual mesh filename=package://galaxea_g1_description/meshes/gripper_finger2.obj
- link link6: geometry collision mesh filename=package://galaxea_a1_description/meshes/a1_xy/link6.obj; visual mesh filename=package://galaxea_a1_description/meshes/a1_xy/link6.obj
Joints:
- removed joint gripper_finger_joint1
- removed joint gripper_finger_joint2
- added joint gripper_joint1: type prismatic, parent gripper_base_link, child gripper_link1, origin xyz=0.03689 0.013453 0.00012059, axis 0 1 0, limit lower=0 upper=0.05 effort=100 velocity=0.25
- added joint gripper_joint2: type prismatic, parent gripper_base_link, child gripper_link2, origin xyz=0.03689 -0.013453 -0.00012059, axis 0 -1 0, limit lower=0 upper=0.05 effort=100 velocity=0.25, mimic joint=gripper_joint1 multiplier=1 offset=0
- joint gripper_joint: axis 0 0 0 -> (none); child gripper_link -> gripper_base_link

File: manipulator/Galaxea/galaxea_a1_description/xacro/a1.xacro (robot description, xacro)
@@ -324,6 +324,6 @@
       <limit lower="-2.8798" upper="2.8798" effort="7" velocity="25.133" />
     </joint>
-    <xacro:include filename="$(find galaxea_a1_description)/xacro/gripper.xacro"/>
-    <xacro:Gripper name="${name}"/>
+    <xacro:include filename="$(find galaxea_g1_description)/xacro/gripper.xacro"/>
+    <xacro:Gripper name="${prefix}gripper"/>
     <xacro:property name="gripper_origin_xyz" value="${'0.1039 0 0'}"/>
     <xacro:property name="gripper_origin_rpy" value="${'-1.5708 0 0' if direction == 'normal' else '3.14159 0 0' if direction == 'right' else '0 0 0'}"/>
@@ -332,5 +332,5 @@
       <origin xyz="${gripper_origin_xyz}" rpy="${gripper_origin_rpy}"/>
       <parent link="${prefix}link6" />
-      <child link="${prefix}gripper_link" />
+      <child link="${prefix}gripper_base_link"/>
     </joint>
   </xacro:macro>

File: manipulator/Galaxea/galaxea_a1_description/xacro/a1_x.xacro (robot description, xacro)
@@ -2,5 +2,5 @@
 <robot xmlns:xacro="http://www.ros.org/wiki/xacro">
   <xacro:macro name="Arm" params="name">
-    <xacro:include filename="(find galaxea_a1_description)/xacro/a1xy_base.xacro"/>
+    <xacro:include filename="$(find galaxea_a1_description)/xacro/a1xy_base.xacro"/>
     <xacro:property name="prefix" value="${name + '_' if name else ''}"/>
     <xacro:Base name=""/>
@@ -185,11 +185,10 @@
           velocity="32.9867"/>
     </joint>
-    <xacro:include filename="(find galaxea_a1_description)/xacro/gripper.xacro"/>
-    <xacro:Gripper name="${name}"/>
+    <xacro:include filename="$(find galaxea_g1_description)/xacro/gripper.xacro"/>
+    <xacro:Gripper name="${prefix}gripper"/>
     <joint name="${prefix}gripper_joint" type="fixed">
       <origin xyz="0.08165 0 0"/>
       <parent link="${prefix}link6"/>
-      <child link="${prefix}gripper_link"/>
-      <axis xyz="0 0 0"/>
+      <child link="${prefix}gripper_base_link"/>
     </joint>
   </xacro:macro>

File: manipulator/Galaxea/galaxea_a1_description/xacro/a1_y.xacro (robot description, xacro)
@@ -2,5 +2,5 @@
 <robot xmlns:xacro="http://www.ros.org/wiki/xacro">
   <xacro:macro name="Arm" params="name">
-    <xacro:include filename="(find galaxea_a1_description)/xacro/a1xy_base.xacro"/>
+    <xacro:include filename="$(find galaxea_a1_description)/xacro/a1xy_base.xacro"/>
     <xacro:property name="prefix" value="${name + '_' if name else ''}"/>
     <xacro:Base name=""/>
@@ -169,5 +169,5 @@
         <geometry>
           <mesh
-              filename="file://$(find a1xy_description)/meshes/a1_xy/link6.obj" />
+              filename="file://$(find galaxea_a1_description)/meshes/a1_xy/link6.obj" />
         </geometry>
         <material
@@ -180,5 +180,5 @@
         <geometry>
           <mesh
-              filename="file://$(find a1xy_description)/meshes/a1_xy/link6.obj" />
+              filename="file://$(find galaxea_a1_description)/meshes/a1_xy/link6.obj" />
         </geometry>
       </collision>
@@ -202,11 +202,10 @@
           velocity="32.9867" />
     </joint>
-    <xacro:include filename="(find galaxea_a1_description)/xacro/gripper.xacro"/>
-    <xacro:Gripper name="${name}"/>
+    <xacro:include filename="$(find galaxea_g1_description)/xacro/gripper.xacro"/>
+    <xacro:Gripper name="${prefix}gripper"/>
     <joint name="${prefix}gripper_joint" type="fixed">
       <origin xyz="0.08165 0 0"/>
       <parent link="${prefix}link6"/>
-      <child link="${prefix}gripper_link"/>
-      <axis xyz="0 0 0"/>
+      <child link="${prefix}gripper_base_link"/>
     </joint>
   </xacro:macro>

File: manipulator/Realman/rm65_description/xacro/arm.xacro (robot description, xacro)
@@ -1,5 +1,5 @@
 <?xml version="1.0"?>
 <robot name="rm65" xmlns:xacro="http://www.ros.org/wiki/xacro">
-  <xacro:macro name="rm65" params="name">
+  <xacro:macro name="rm65" params="name direction:=''" >
     <xacro:property name="prefix" value="${name + '_' if name else ''}"/>
     <!-- Define constants -->
@@ -23,15 +23,50 @@
     <link name="${prefix}base_link">
       <inertial>
-        <origin xyz="-0.00049840293879996 -5.19350047653785E-05 0.0600202841321701"/>
-        <mass value="0.838885281114303"/>
-        <inertia
-            ixx="0.00172321229549441"
-            ixy="3.09076898315635E-06"
-            ixz="-3.7922126488402E-05"
-            iyy="0.00170514762495823"
-            iyz="1.38793642017112E-06"
-            izz="0.000901589030906685"/>
-      </inertial>
-      <xacro:visual_collision mesh="base_link.obj"/>
+        <!-- Default configuration -->
+        <xacro:if value="${direction != 'l' and direction != 'r'}">
+          <origin xyz="-0.00049840293879996 -5.19350047653785E-05 0.0600202841321701"/>
+          <mass value="0.838885281114303"/>
+          <inertia
+              ixx="0.00172321229549441"
+              ixy="3.09076898315635E-06"
+              ixz="-3.7922126488402E-05"
+              iyy="0.00170514762495823"
+              iyz="1.38793642017112E-06"
+              izz="0.000901589030906685"/>
+        </xacro:if>
+        <!-- Left arm configuration -->
+        <xacro:if value="${direction == 'l'}">
+          <origin xyz="-3.58E-05 -0.0056915 0.024464"/>
+          <mass value="0.23441"/>
+          <inertia
+              ixx="0.00027369"
+              ixy="6.5702E-08"
+              ixz="2.7812E-09"
+              iyy="0.000264"
+              iyz="-1.6355E-06"
+              izz="0.00036679"/>
+        </xacro:if>
+        <!-- Right arm configuration -->
+        <xacro:if value="${direction == 'r'}">
+          <origin xyz="-4.8022E-05 0.0056915 0.024715"/>
+          <mass value="0.23441"/>
+          <inertia
+              ixx="0.00027369"
+              ixy="6.5702E-08"
+              ixz="-3.2599E-09"
+              iyy="0.000264"
+              iyz="1.6355E-06"
+              izz="0.00036679"/>
+        </xacro:if>
+      </inertial>
+      <xacro:if value="${direction == 'l'}">
+        <xacro:visual_collision mesh="base_link_aidal.obj"/>
+      </xacro:if>
+      <xacro:if value="${direction == 'r'}">
+        <xacro:visual_collision mesh="base_link_aidal.obj"/>
+      </xacro:if>
+      <xacro:if value="${direction != 'l' and direction != 'r'}">
+        <xacro:visual_collision mesh="base_link.obj"/>
+      </xacro:if>
     </link>
     <link name="${prefix}link1">
@@ -120,5 +155,16 @@
     </link>
     <joint name="${prefix}joint1" type="revolute">
-      <origin xyz="0 0 0.2405"/>
+      <!-- Default configuration -->
+      <xacro:if value="${direction != 'l' and direction != 'r'}">
+        <origin xyz="0 0 0.2405"/>
+      </xacro:if>
+      <!-- Left arm configuration -->
+      <xacro:if value="${direction == 'l'}">
+        <origin xyz="0 0 0.187" rpy="0 0 3.1415"/>
+      </xacro:if>
+      <!-- Right arm configuration -->
+      <xacro:if value="${direction == 'r'}">
+        <origin xyz="0 0 0.187" rpy="0 0 0"/>
+      </xacro:if>
       <parent link="${prefix}base_link"/>
       <child link="${prefix}link1"/>
@@ -155,5 +201,10 @@
     </joint>
     <joint name="${prefix}joint6" type="revolute">
-      <origin xyz="0 -0.115 -0.00029971" rpy="-1.5708 0 0"/>
+      <xacro:if value="${direction == 'r'}">
+        <origin xyz="0 -0.115 0" rpy="-1.5708 3.14159 0"/>
+      </xacro:if>
+      <xacro:unless value="${direction == 'r'}">
+        <origin xyz="0 -0.115 0" rpy="-1.5708 0 0"/>
+      </xacro:unless>
       <parent link="${prefix}link5"/>
       <child link="${prefix}link6"/>
@@ -161,4 +212,19 @@
       <limit lower="-6.28" upper="6.28" effort="10" velocity="3.925"/>
     </joint>
+    <link name="${prefix}gripper_plate">
+      <xacro:visual_collision mesh="gripper_plate.obj"/>
+    </link>
+    <joint name="${prefix}ee_joint" type="fixed">
+      <origin xyz="0 0 -0.043" rpy="3.14159 0 1.5708"/>
+      <parent link="${prefix}link6"/>
+      <child link="${prefix}gripper_plate"/>
+    </joint>
+    <xacro:include filename="$(find inspire_eg2_description)/xacro/eg2_4c2.xacro"/>
+    <xacro:Gripper name="${prefix}gripper"/>
+    <joint name="${prefix}gripper_joint" type="fixed">
+      <origin xyz="0 0 0.0043" rpy="0 0 0"/>
+      <parent link="${prefix}gripper_plate" />
+      <child link="${prefix}gripper_base_link" />
+    </joint>
   </xacro:macro>
 </robot>
