Commit message: add license files

File: manipulator/LeRobot/so_arm_description/urdf/so_arm.urdf (robot description, URDF)
Before this commit: robot Piper single, 18 links, 17 joints
Links:
- removed link gripperframe
- removed link moving_jaw_so101_v1
- added link base, mass 0.147; collision mesh filename=package://so_arm_description/meshes/so101/base.stl; collision mesh filename=package://so_arm_description/meshes/so101/base_motor_holder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
- added link fixed_jaw_tip
- added link moving_jaw, mass 0.012; collision mesh filename=package://so_arm_description/meshes/so101/moving_jaw/moving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; collision mesh filename=package://so_arm_description/meshes/so101/moving_jaw/moving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
- link base_link: mass 0.147 -> None; geometry 
Joints:
- removed joint gripperframe_frame
- added joint base_joint: type fixed, parent base_link, child base, origin xyz=0 0 0.0025
- added joint fixed_jaw_tip_joint: type fixed, parent gripper, child fixed_jaw_tip, origin xyz=-0.0079 -0.000218121 -0.0981274 rpy=0 1.5708 0
- joint gripper: child moving_jaw_so101_v1 -> moving_jaw
- joint motor1_joint: parent base_link -> base
- joint moving_Jaw_tip_joint: parent moving_jaw_so101_v1 -> moving_jaw
- joint shoulder_pan: parent base_link -> base

File: manipulator/LeRobot/so_arm_description/xacro/so101.xacro (robot description, xacro)
@@ -3,6 +3,11 @@
   <xacro:macro name="Arm" params="name ">
     <xacro:property name="prefix" value="${name + '_' if name else ''}"/>
-    <!-- Frame baseframe (dummy link + fixed joint) -->
-    <link name="${prefix}base_link">
+    <joint name="${prefix}base_joint" type="fixed">
+      <origin  xyz="0 0 0.0025"/>
+      <parent link="${prefix}base_link"/>
+      <child link="${prefix}base"/>
+    </joint>
+    <link name="${prefix}base_link"/>
+    <link name="${prefix}base">
       <inertial>
         <origin xyz="-0.01371 0 0.03348"/>
@@ -55,5 +60,5 @@
     <joint name="${prefix}motor1_joint" type="fixed">
       <origin xyz="0.0263345 0 0.0437"/>
-      <parent link="${prefix}base_link"/>
+      <parent link="${prefix}base"/>
       <child link="${prefix}motor1"/>
     </joint>
@@ -107,5 +112,5 @@
     <joint name="${prefix}shoulder_pan" type="revolute">
       <origin xyz="0.0388353 0 0.0624" rpy="-3.14159 0 3.14159"/>
-      <parent link="${prefix}base_link"/>
+      <parent link="${prefix}base"/>
       <child link="${prefix}shoulder"/>
       <axis xyz="0 0 1"/>

File: quadruped/deep_robotics/x30_description/xacro/body.xacro (robot description, xacro)
@@ -4,5 +4,4 @@
   <link name="base">
     <visual>
-      <origin rpy="0 0 0" xyz="0 0 0"/>
       <geometry>
         <box size="0.001 0.001 0.001"/>
@@ -11,5 +10,4 @@
   </link>
   <joint name="floating_base" type="fixed">
-    <origin rpy="0 0 0" xyz="0 0 0"/>
     <parent link="base"/>
     <child link="TORSO"/>
@@ -27,5 +25,4 @@
     </visual>
     <collision>
-      <origin xyz="0 0 0" rpy="0 0 0"/>
       <geometry>
         <box size="0.44 0.26 0.15"/>

File: quadruped/deep_robotics/x30_description/xacro/materials.xacro (robot description, xacro)
@@ -20,5 +20,5 @@
     </material>
     <material name="silver">
-        <color rgba="${233/255} ${233/255} ${216/255} 1.0"/>
+        <color rgba="0.9 0.9 0.9 1.0"/>
     </material>
     <material name="white">
