Commit message: simplified deeprobotics mesh

File: quadruped/deep_robotics/lite3_description/urdf/robot.urdf (robot description, URDF)
Before this commit: robot lite3, 19 links, 18 joints
Links:
- link FL_HIP: geometry visual mesh filename=package://lite3_description/meshes/hip.obj scale=1 1 1
- link FL_THIGH: geometry collision box size=0.02 0.02 0.16; visual mesh filename=package://lite3_description/meshes/thigh.obj scale=1 1 1
- link FR_HIP: geometry visual mesh filename=package://lite3_description/meshes/hip.obj scale=1 -1 1
- link FR_THIGH: geometry collision box size=0.02 0.02 0.16; visual mesh filename=package://lite3_description/meshes/thigh.obj scale=1 -1 1
- link HL_HIP: geometry visual mesh filename=package://lite3_description/meshes/hip.obj scale=-1 1 1
- link HL_THIGH: geometry collision box size=0.02 0.02 0.16; visual mesh filename=package://lite3_description/meshes/thigh.obj scale=1 1 1
- link HR_HIP: geometry visual mesh filename=package://lite3_description/meshes/hip.obj scale=-1 -1 1
- link HR_THIGH: geometry collision box size=0.02 0.02 0.16; visual mesh filename=package://lite3_description/meshes/thigh.obj scale=1 -1 1

File: quadruped/deep_robotics/lite3_description/xacro/const.xacro (robot description, xacro)
@@ -1,7 +1,4 @@
 <?xml version="1.0"?>
 <robot xmlns:xacro="http://www.ros.org/wiki/xacro">
-  <material name="silver">
-    <color rgba="${233/255} ${233/255} ${233/255} 1.0"/>
-  </material>
   <xacro:property name="damping" value="0.0"/>
   <xacro:property name="friction" value="0.1"/>

File: quadruped/deep_robotics/lite3_description/xacro/leg.xacro (robot description, xacro)
@@ -2,16 +2,16 @@
 <robot xmlns:xacro="http://www.ros.org/wiki/xacro">
   <xacro:include filename="$(find lite3_description)/xacro/transmission.xacro"/>
-  <xacro:macro name="leg" params="name mirror mirror_dae front_hind front_hind_dae">
+  <xacro:macro name="leg" params="name mirror mirror_dae front_hind">
     <joint name="${name}_HipX" type="revolute">
-      <xacro:if value="${(mirror_dae == False) and (front_hind_dae == True)}">
+      <xacro:if value="${(mirror_dae == False) and (front_hind == 1)}">
         <origin rpy="0 0 0" xyz="${leg_offset_x} ${-leg_offset_y} 0"/>
       </xacro:if>
-      <xacro:if value="${(mirror_dae == True) and (front_hind_dae == True)}">
+      <xacro:if value="${(mirror_dae == True) and (front_hind == 1)}">
         <origin rpy="0 0 0" xyz="${leg_offset_x} ${leg_offset_y} 0"/>
       </xacro:if>
-      <xacro:if value="${(mirror_dae == False) and (front_hind_dae == False)}">
+      <xacro:if value="${(mirror_dae == False) and (front_hind == -1)}">
         <origin rpy="0 0 0" xyz="${-leg_offset_x} ${-leg_offset_y} 0"/>
       </xacro:if>
-      <xacro:if value="${(mirror_dae == True) and (front_hind_dae == False)}">
+      <xacro:if value="${(mirror_dae == True) and (front_hind == -1)}">
         <origin rpy="0 0 0" xyz="${-leg_offset_x} ${leg_offset_y} 0"/>
       </xacro:if>
@@ -34,7 +34,6 @@
       <visual>
         <geometry>
-          <mesh filename="file://$(find lite3_description)/meshes/${name}_hip.STL"/>
+          <mesh filename="file://$(find lite3_description)/meshes/hip.obj" scale="${front_hind} ${mirror} 1"/>
         </geometry>
-        <material name="silver"/>
       </visual>
     </link>
@@ -59,10 +58,5 @@
       <visual>
         <geometry>
-          <xacro:if value="${mirror_dae == True}">
-            <mesh filename="file://$(find lite3_description)/meshes/l_thigh.obj"/>
-          </xacro:if>
-          <xacro:if value="${mirror_dae == False}">
-            <mesh filename="file://$(find lite3_description)/meshes/r_thigh.obj"/>
-          </xacro:if>
+          <mesh filename="file://$(find lite3_description)/meshes/thigh.obj" scale="1 ${mirror} 1"/>
         </geometry>
       </visual>

File: quadruped/deep_robotics/lite3_description/xacro/robot.xacro (robot description, xacro)
@@ -18,5 +18,4 @@
   <link name="base">
     <visual>
-      <origin rpy="0 0 0" xyz="0 0 0"/>
       <geometry>
         <box size="0.001 0.001 0.001"/>
@@ -55,9 +54,7 @@
     <inertial>
       <mass value="0.001"/>
-      <origin rpy="0 0 0" xyz="0 0 0"/>
       <inertia ixx="0.0001" ixy="0" ixz="0" iyy="0.0001" iyz="0" izz="0.0001"/>
     </inertial>
     <visual>
-      <origin rpy="0 0 0" xyz="0 0 0"/>
       <geometry>
         <box size="0.001 0.001 0.001"/>
@@ -65,5 +62,4 @@
     </visual>
     <collision>
-      <origin rpy="0 0 0" xyz="0 0 0"/>
       <geometry>
         <box size=".001 .001 .001"/>
@@ -71,7 +67,7 @@
     </collision>
   </link>
-  <xacro:leg name="FR" mirror="-1" mirror_dae="False" front_hind="1" front_hind_dae="True"/>
-  <xacro:leg name="FL" mirror="1" mirror_dae="True" front_hind="1" front_hind_dae="True"/>
-  <xacro:leg name="HR" mirror="-1" mirror_dae="False" front_hind="-1" front_hind_dae="False"/>
-  <xacro:leg name="HL" mirror="1" mirror_dae="True" front_hind="-1" front_hind_dae="False"/>
+  <xacro:leg name="FR" mirror="-1" mirror_dae="False" front_hind="1"/>
+  <xacro:leg name="FL" mirror="1" mirror_dae="True" front_hind="1"/>
+  <xacro:leg name="HR" mirror="-1" mirror_dae="False" front_hind="-1"/>
+  <xacro:leg name="HL" mirror="1" mirror_dae="True" front_hind="-1"/>
 </robot>

File: quadruped/deep_robotics/x30_description/xacro/body.xacro (robot description, xacro)
@@ -38,7 +38,6 @@
     <visual>
       <geometry>
-        <mesh filename="file://$(find x30_description)/meshes/fl_hip.STL"/>
-      </geometry>
-      <material name="silver"/>
+        <mesh filename="file://$(find x30_description)/meshes/hip.obj"/>
+      </geometry>
     </visual>
   </link>
@@ -58,5 +57,5 @@
     <visual>
       <geometry>
-        <mesh filename="file://$(find x30_description)/meshes/l_thigh.obj"/>
+        <mesh filename="file://$(find x30_description)/meshes/thigh.obj"/>
       </geometry>
     </visual>
@@ -136,7 +135,6 @@
     <visual>
       <geometry>
-        <mesh filename="file://$(find x30_description)/meshes/fr_hip.STL"/>
-      </geometry>
-      <material name="silver"/>
+        <mesh filename="file://$(find x30_description)/meshes/hip.obj" scale="1 -1 1"/>
+      </geometry>
     </visual>
   </link>
@@ -156,5 +154,5 @@
     <visual>
       <geometry>
-        <mesh filename="file://$(find x30_description)/meshes/r_thigh.obj"/>
+        <mesh filename="file://$(find x30_description)/meshes/thigh.obj" scale="1 -1 1"/>
       </geometry>
     </visual>
@@ -234,7 +232,6 @@
     <visual>
       <geometry>
-        <mesh filename="file://$(find x30_description)/meshes/hl_hip.STL"/>
-      </geometry>
-      <material name="silver"/>
+        <mesh filename="file://$(find x30_description)/meshes/hip.obj" scale="-1 1 1"/>
+      </geometry>
     </visual>
   </link>
@@ -254,5 +251,5 @@
     <visual>
       <geometry>
-        <mesh filename="file://$(find x30_description)/meshes/l_thigh.obj"/>
+        <mesh filename="file://$(find x30_description)/meshes/thigh.obj"/>
       </geometry>
     </visual>
@@ -332,7 +329,6 @@
     <visual>
       <geometry>
-        <mesh filename="file://$(find x30_description)/meshes/hr_hip.STL"/>
-      </geometry>
-      <material name="silver"/>
+        <mesh filename="file://$(find x30_description)/meshes/hip.obj" scale="-1 -1 1"/>
+      </geometry>
     </visual>
   </link>
@@ -352,5 +348,5 @@
     <visual>
       <geometry>
-        <mesh filename="file://$(find x30_description)/meshes/r_thigh.obj"/>
+        <mesh filename="file://$(find x30_description)/meshes/thigh.obj" scale="1 -1 1"/>
       </geometry>
     </visual>

File: quadruped/deep_robotics/x30_description/xacro/gazebo.xacro (robot description, xacro)
@@ -102,11 +102,4 @@
     <mu2>0.6</mu2>
     <self_collide>1</self_collide>
-    <visual>
-      <material>
-        <ambient>.05 .05 .05 1.0</ambient>
-        <diffuse>.05 .05 .05 1.0</diffuse>
-        <specular>.05 .05 .05 1.0</specular>
-      </material>
-    </visual>
   </gazebo>
   <gazebo reference="imu_link">

File: quadruped/deep_robotics/x30_description/xacro/robot.xacro (robot description, xacro)
@@ -2,5 +2,4 @@
 <robot name="x30" xmlns:xacro="http://www.ros.org/wiki/xacro">
   <xacro:include filename="$(find x30_description)/xacro/body.xacro"/>
-  <xacro:include filename="$(find x30_description)/xacro/materials.xacro"/>
   <xacro:include filename="$(find x30_description)/xacro/transmission.xacro"/>
   <xacro:arg name="GAZEBO" default="false"/>
