Commit message: add agile split aloha

File: manipulator/AgileX/agilex_aloha_description/xacro/aloha_v2.xacro (robot description, xacro)
@@ -10,5 +10,5 @@
       <origin xyz="0 0 0" rpy="1.57 0 0"/>
       <geometry>
-        <mesh filename="package://mobile_aloha2_description/meshes/tracer_base_link.obj"/>
+        <mesh filename="file://$(find agilex_aloha_description)/meshes/aloha_v2/tracer_base_link.obj"/>
       </geometry>
     </visual>
@@ -16,5 +16,5 @@
       <origin xyz="0 0 0" rpy="1.57 0 0"/>
       <geometry>
-        <mesh filename="package://mobile_aloha2_description/meshes/tracer_base_link.obj"/>
+        <mesh filename="file://$(find agilex_aloha_description)/meshes/aloha_v2/tracer_base_link.obj"/>
       </geometry>
     </collision>
@@ -30,5 +30,5 @@
       <!--<origin
         xyz="-0.0145261552504705 0.0231316650320557 0.00586280190939592"
-        rpy="0 0 0" />-->
+        />-->
       <inertia ixx="0.185196122711036"
                ixy="4.30144213829512E-08"
@@ -41,5 +41,5 @@
   </link>
   <joint name="inertial_joint" type="fixed">
-    <origin xyz="0 0 0" rpy="0 0 0"/>
+    <origin xyz="0 0 0"/>
     <parent link="base_link"/>
     <child link="inertial_link"/>
@@ -52,10 +52,10 @@
     <visual>
       <geometry>
-        <mesh filename="package://mobile_aloha2_description/meshes/tracer_wheel.obj"/>
-      </geometry>
-    </visual>
-    <collision>
-      <geometry>
-        <mesh filename="package://mobile_aloha2_description/meshes/tracer_wheel.obj"/>
+        <mesh filename="file://$(find agilex_aloha_description)/meshes/aloha_v2/tracer_wheel.obj"/>
+      </geometry>
+    </visual>
+    <collision>
+      <geometry>
+        <mesh filename="file://$(find agilex_aloha_description)/meshes/aloha_v2/tracer_wheel.obj"/>
       </geometry>
     </collision>
@@ -64,6 +64,6 @@
     <parent link="base_link"/>
     <child link="right_wheel_link"/>
-    <origin xyz="0 -0.17 -0.082" rpy="0 0 0"/>
-    <axis xyz="0 1 0" rpy="0 0 0"/>
+    <origin xyz="0 -0.17 -0.082"/>
+    <axis xyz="0 1 0"/>
   </joint>
   <link name="left_wheel_link">
@@ -74,10 +74,10 @@
     <visual>
       <geometry>
-        <mesh filename="package://mobile_aloha2_description/meshes/tracer_wheel.obj"/>
-      </geometry>
-    </visual>
-    <collision>
-      <geometry>
-        <mesh filename="package://mobile_aloha2_description/meshes/tracer_wheel.obj"/>
+        <mesh filename="file://$(find agilex_aloha_description)/meshes/aloha_v2/tracer_wheel.obj"/>
+      </geometry>
+    </visual>
+    <collision>
+      <geometry>
+        <mesh filename="file://$(find agilex_aloha_description)/meshes/aloha_v2/tracer_wheel.obj"/>
       </geometry>
     </collision>
@@ -86,6 +86,6 @@
     <parent link="base_link"/>
     <child link="left_wheel_link"/>
-    <origin xyz="0 0.17 -0.082" rpy="0 0 0"/>
-    <axis xyz="0 1 0" rpy="0 0 0"/>
+    <origin xyz="0 0.17 -0.082"/>
+    <axis xyz="0 1 0"/>
   </joint>
   <link name="fl_castor_link">
@@ -96,5 +96,5 @@
     <visual>
       <geometry>
-        <mesh filename="package://mobile_aloha2_description/meshes/castor_joint.obj"/>
+        <mesh filename="file://$(find agilex_aloha_description)/meshes/aloha_v2/castor_joint.obj"/>
       </geometry>
     </visual>
@@ -104,5 +104,5 @@
     <child link="fl_castor_link"/>
     <origin xyz="0.19 0.17 -0.038" rpy="-1.57 0 0"/>
-    <axis xyz="0 1 0" rpy="0 0 0"/>
+    <axis xyz="0 1 0"/>
   </joint>
   <link name="fr_castor_link">
@@ -113,5 +113,5 @@
     <visual>
       <geometry>
-        <mesh filename="package://mobile_aloha2_description/meshes/castor_joint.obj"/>
+        <mesh filename="file://$(find agilex_aloha_description)/meshes/aloha_v2/castor_joint.obj"/>
       </geometry>
     </visual>
@@ -121,5 +121,5 @@
     <parent link="base_link"/>
     <child link="fr_castor_link"/>
-    <axis xyz="0 1 0" rpy="0 0 0"/>
+    <axis xyz="0 1 0"/>
   </joint>
   <link name="rr_castor_link">
@@ -130,5 +130,5 @@
     <visual>
       <geometry>
-        <mesh filename="package://mobile_aloha2_description/meshes/castor_joint.obj"/>
+        <mesh filename="file://$(find agilex_aloha_description)/meshes/aloha_v2/castor_joint.obj"/>
       </geometry>
     </visual>
@@ -138,5 +138,5 @@
     <parent link="base_link"/>
     <child link="rr_castor_link"/>
-    <axis xyz="0 1 0" rpy="0 0 0"/>
+    <axis xyz="0 1 0"/>
   </joint>
   <link name="rl_castor_link">
@@ -147,5 +147,5 @@
     <visual>
       <geometry>
-        <mesh filename="package://mobile_aloha2_description/meshes/castor_joint.obj"/>
+        <mesh filename="file://$(find agilex_aloha_description)/meshes/aloha_v2/castor_joint.obj"/>
       </geometry>
     </visual>
@@ -155,5 +155,5 @@
     <parent link="base_link"/>
     <child link="rl_castor_link"/>
-    <axis xyz="0 1 0" rpy="0 0 0"/>
+    <axis xyz="0 1 0"/>
   </joint>
   <link name="fl_wheel_link">
@@ -164,10 +164,10 @@
     <visual>
       <geometry>
-        <mesh filename="package://mobile_aloha2_description/meshes/castor.obj"/>
+        <mesh filename="file://$(find agilex_aloha_description)/meshes/aloha_v2/castor.obj"/>
       </geometry>
     </visual>
     <collision>
       <geometry>-->
-        <mesh filename="package://mobile_aloha2_description/meshes/castor.obj"/>
+        <mesh filename="file://$(find agilex_aloha_description)/meshes/aloha_v2/castor.obj"/>
       </geometry>
     </collision>
@@ -177,6 +177,6 @@
     <child link="fl_wheel_link"/>
     <dynamics damping="0.0" friction="0.0"/>
-    <origin xyz="-0.0218084 0.077 0" rpy="0 0 0"/>
-    <axis xyz="0 0 1" rpy="0 0 0"/>
+    <origin xyz="-0.0218084 0.077 0"/>
+    <axis xyz="0 0 1"/>
   </joint>
   <link name="fr_wheel_link">
@@ -187,10 +187,10 @@
     <visual>
       <geometry>
-        <mesh filename="package://mobile_aloha2_description/meshes/castor.obj"/>
+        <mesh filename="file://$(find agilex_aloha_description)/meshes/aloha_v2/castor.obj"/>
       </geometry>
     </visual>
     <collision>
       <geometry>-->
-        <mesh filename="package://mobile_aloha2_description/meshes/castor.obj"/>
+        <mesh filename="file://$(find agilex_aloha_description)/meshes/aloha_v2/castor.obj"/>
       </geometry>
     </collision>
@@ -200,6 +200,6 @@
     <child link="fr_wheel_link"/>
     <dynamics damping="0.0" friction="0.0"/>
-    <origin xyz="-0.0218084 0.077 0" rpy="0 0 0"/>
-    <axis xyz="0 0 1" rpy="0 0 0"/>
+    <origin xyz="-0.0218084 0.077 0"/>
+    <axis xyz="0 0 1"/>
   </joint>
   <link name="rr_wheel_link">
@@ -210,10 +210,10 @@
     <visual>
       <geometry>
-        <mesh filename="package://mobile_aloha2_description/meshes/castor.obj"/>
-      </geometry>
-    </visual>
-    <collision>
-      <geometry>
-        <mesh filename="package://mobile_aloha2_description/meshes/castor.obj"/>
+        <mesh filename="file://$(find agilex_aloha_description)/meshes/aloha_v2/castor.obj"/>
+      </geometry>
+    </visual>
+    <collision>
+      <geometry>
+        <mesh filename="file://$(find agilex_aloha_description)/meshes/aloha_v2/castor.obj"/>
       </geometry>
     </collision>
@@ -223,6 +223,6 @@
     <child link="rr_wheel_link"/>
     <dynamics damping="0.0" friction="0.0"/>
-    <origin xyz="-0.0218084 0.077 0" rpy="0 0 0"/>
-    <axis xyz="0 0 1" rpy="0 0 0"/>
+    <origin xyz="-0.0218084 0.077 0"/>
+    <axis xyz="0 0 1"/>
   </joint>
   <link name="rl_wheel_link">
@@ -233,10 +233,10 @@
     <visual>
       <geometry>
-        <mesh filename="package://mobile_aloha2_description/meshes/castor.obj"/>
-      </geometry>
-    </visual>
-    <collision>
-      <geometry>
-        <mesh filename="package://mobile_aloha2_description/meshes/castor.obj"/>
+        <mesh filename="file://$(find agilex_aloha_description)/meshes/aloha_v2/castor.obj"/>
+      </geometry>
+    </visual>
+    <collision>
+      <geometry>
+        <mesh filename="file://$(find agilex_aloha_description)/meshes/aloha_v2/castor.obj"/>
       </geometry>
     </collision>
@@ -246,10 +246,10 @@
     <child link="rl_wheel_link"/>
     <dynamics damping="0.0" friction="0.0"/>
-    <origin xyz="-0.0218084 0.077 0" rpy="0 0 0"/>
-    <axis xyz="0 0 1" rpy="0 0 0"/>
+    <origin xyz="-0.0218084 0.077 0"/>
+    <axis xyz="0 0 1"/>
   </joint>
   <!-- aloha base -->
   <joint name="base_joint" type="fixed">
-    <origin xyz="0 0 0.15" rpy="0 0 0"/>
+    <origin xyz="0 0 0.15"/>
     <parent link="footprint"/>
     <child link="base_link"/>
@@ -258,5 +258,5 @@
   <link name="body_Link">
     <inertial>
-      <origin xyz="0.015107 -0.027922 0.00013672" rpy="0 0 0"/>
+      <origin xyz="0.015107 -0.027922 0.00013672"/>
       <mass value="3.736"/>
       <inertia ixx="0.097545" ixy="-9.2609E-06" ixz="0.00015366" iyy="0.045841" iyz="-0.0020459" izz="0.084773"/>
@@ -265,5 +265,5 @@
       <origin xyz="0 0 0.168" rpy="0 0 3.14"/>
       <geometry>
-        <mesh filename="package://mobile_aloha2_description/meshes/body.obj"/>
+        <mesh filename="file://$(find agilex_aloha_description)/meshes/aloha_v2/body.obj"/>
       </geometry>
     </visual>
@@ -271,10 +271,10 @@
       <origin xyz="0 0 0.168" rpy="0 0 3.14"/>
       <geometry>
-        <mesh filename="package://mobile_aloha2_description/meshes/body.obj"/>
+        <mesh filename="file://$(find agilex_aloha_description)/meshes/aloha_v2/body.obj"/>
       </geometry>
     </collision>
   </link>
   <joint name="body_joint" type="fixed">
-    <origin xyz="0 0 0" rpy="0 0 0"/>
+    <origin xyz="0 0 0"/>
     <parent link="footprint"/>
     <child link="body_Link"/>

File: manipulator/AgileX/piper_description/xacro/slave.xacro (robot description, xacro)
@@ -67,4 +67,5 @@
       <parent link="${prefix}link6"/>
       <child link="${prefix}link8"/>
+      <mimic joint="${prefix}joint7" multiplier="1" offset="0"/>
       <axis xyz="0 1 0"/>
       <limit lower="0" upper="0.035" effort="10" velocity="1"/>
