Commit message: add arx x7s

File: humanoid/ARX/lift_description/urdf/lift_r5.urdf (robot description, URDF)
Before this commit: robot lift, 37 links, 36 joints
Links:
- link left_base_link: mass 0.43995 -> 0.42272; geometry collision mesh filename=package://arx5_description/meshes/r5/base_link.obj; visual mesh filename=package://arx5_description/meshes/r5/base_link.obj
- link left_link1: mass 0.066982 -> 0.096804; geometry collision mesh filename=package://arx5_description/meshes/r5/link1.obj; visual mesh filename=package://arx5_description/meshes/r5/link1.obj
- link left_link2: mass 1.0795 -> 1.1988; geometry collision mesh filename=package://arx5_description/meshes/r5/link2.obj; visual mesh filename=package://arx5_description/meshes/r5/link2.obj
- link left_link3: mass 0.54534 -> 0.84082; geometry collision mesh filename=package://arx5_description/meshes/r5/link3.obj; visual mesh filename=package://arx5_description/meshes/r5/link3.obj
- link left_link4: mass 0.11714 -> 0.12432; geometry collision mesh filename=package://arx5_description/meshes/r5/link4.obj; visual mesh filename=package://arx5_description/meshes/r5/link4.obj
- link left_link5: mass 0.63488 -> 0.63601; geometry collision mesh filename=package://arx5_description/meshes/r5/link5.obj; visual mesh filename=package://arx5_description/meshes/r5/link5.obj
- link left_link6: geometry collision mesh filename=package://arx5_description/meshes/r5/link6.obj; visual mesh filename=package://arx5_description/meshes/r5/link6.obj
- link left_link7: geometry collision mesh filename=package://arx5_description/meshes/r5/link7.obj; visual mesh filename=package://arx5_description/meshes/r5/link7.obj
- link left_link8: mass 0.064798 -> 0.0647981725781684; geometry collision mesh filename=package://arx5_description/meshes/r5/link8.obj; visual mesh filename=package://arx5_description/meshes/r5/link8.obj
- link right_base_link: mass 0.43995 -> 0.42272; geometry collision mesh filename=package://arx5_description/meshes/r5/base_link.obj; visual mesh filename=package://arx5_description/meshes/r5/base_link.obj
- link right_link1: mass 0.066982 -> 0.096804; geometry collision mesh filename=package://arx5_description/meshes/r5/link1.obj; visual mesh filename=package://arx5_description/meshes/r5/link1.obj
- link right_link2: mass 1.0795 -> 1.1988; geometry collision mesh filename=package://arx5_description/meshes/r5/link2.obj; visual mesh filename=package://arx5_description/meshes/r5/link2.obj
- link right_link3: mass 0.54534 -> 0.84082; geometry collision mesh filename=package://arx5_description/meshes/r5/link3.obj; visual mesh filename=package://arx5_description/meshes/r5/link3.obj
- link right_link4: mass 0.11714 -> 0.12432; geometry collision mesh filename=package://arx5_description/meshes/r5/link4.obj; visual mesh filename=package://arx5_description/meshes/r5/link4.obj
- link right_link5: mass 0.63488 -> 0.63601; geometry collision mesh filename=package://arx5_description/meshes/r5/link5.obj; visual mesh filename=package://arx5_description/meshes/r5/link5.obj
- link right_link6: geometry collision mesh filename=package://arx5_description/meshes/r5/link6.obj; visual mesh filename=package://arx5_description/meshes/r5/link6.obj
- link right_link7: geometry collision mesh filename=package://arx5_description/meshes/r5/link7.obj; visual mesh filename=package://arx5_description/meshes/r5/link7.obj
- link right_link8: mass 0.064798 -> 0.0647981725781684; geometry collision mesh filename=package://arx5_description/meshes/r5/link8.obj; visual mesh filename=package://arx5_description/meshes/r5/link8.obj
Joints:
- joint left_gripper_center_fixed: origin xyz=0.145 0 0 -> xyz=0.08657 0 0
- joint left_joint1: limit lower=-2.87 upper=3.14 effort=100 velocity=5 -> lower=-2.618 upper=2.168 effort=100 velocity=5; origin xyz=0 0 0.0605 -> xyz=0 0 0.0565
- joint left_joint2: origin xyz=0.02 0 0.04 -> xyz=0.02 0 0.047
- joint left_joint3: origin xyz=-0.264 0 0 rpy=3.1416 0 0 -> xyz=-0.264 0 0 rpy=-3.1416 0 0
- joint left_joint4: origin xyz=0.245 0 -0.056 -> xyz=0.245 -5E-05 -0.06
- joint left_joint5: origin xyz=0.06775 0.0005 -0.0865 -> xyz=0.0702 5E-05 -0.083391
- joint left_joint6: origin xyz=0.02895 0 0.0865 rpy=-3.1416 0 0 -> xyz=0.025286 0 0.083391 rpy=3.1416 0 0
- joint right_gripper_center_fixed: origin xyz=0.145 0 0 -> xyz=0.08657 0 0
- joint right_joint1: limit lower=-2.87 upper=3.14 effort=100 velocity=5 -> lower=-2.618 upper=2.168 effort=100 velocity=5; origin xyz=0 0 0.0605 -> xyz=0 0 0.0565
- joint right_joint2: origin xyz=0.02 0 0.04 -> xyz=0.02 0 0.047
- joint right_joint3: origin xyz=-0.264 0 0 rpy=3.1416 0 0 -> xyz=-0.264 0 0 rpy=-3.1416 0 0
- joint right_joint4: origin xyz=0.245 0 -0.056 -> xyz=0.245 -5E-05 -0.06
- joint right_joint5: origin xyz=0.06775 0.0005 -0.0865 -> xyz=0.0702 5E-05 -0.083391
- joint right_joint6: origin xyz=0.02895 0 0.0865 rpy=-3.1416 0 0 -> xyz=0.025286 0 0.083391 rpy=3.1416 0 0

File: humanoid/ARX/lift_description/xacro/body.xacro (robot description, xacro)
@@ -21,5 +21,5 @@
     <joint name="joint_lift" type="prismatic">
       <origin xyz="0.022199 0 0.233"/>
-      <parent link="base_link"/>
+      <parent link="base"/>
       <child link="lift_1"/>
       <axis xyz="0.0 0.0 1.0"/>

File: humanoid/ARX/lift_description/xacro/mobile_base.xacro (robot description, xacro)
@@ -2,5 +2,11 @@
 <robot xmlns:xacro="http://www.ros.org/wiki/xacro">
   <xacro:macro name="MobileBase">
-    <link name="base_link">
+    <link name="base_link"/>
+    <joint name="base_joint" type="fixed">
+      <origin rpy="0 0 3.14159"/>
+      <parent link="base_link"/>
+      <child link="base"/>
+    </joint>
+    <link name="base">
       <inertial>
         <origin xyz="0.015300075250394498 -0.0039712791148939055 0.21685783167580347"/>
@@ -42,10 +48,10 @@
     <joint name="joint_wheel1" type="fixed">
       <origin xyz="-0.182349 0.315838 0.03"/>
-      <parent link="base_link"/>
+      <parent link="base"/>
       <child link="wheel_1"/>
     </joint>
     <joint name="joint_wheel2" type="fixed">
       <origin xyz="-0.182349 -0.315838 0.03"/>
-      <parent link="base_link"/>
+      <parent link="base"/>
       <child link="wheel_2"/>
       <axis xyz="-0.5 -0.866025 0.0"/>
@@ -53,5 +59,5 @@
     <joint name="joint_wheel3" type="fixed">
       <origin xyz="0.364699 0.0 0.03"/>
-      <parent link="base_link"/>
+      <parent link="base"/>
       <child link="wheel_3"/>
       <axis xyz="1.0 0.0 -0.0"/>

File: humanoid/ARX/lift_description/xacro/robot.xacro (robot description, xacro)
@@ -1,18 +1,18 @@
 <?xml version="1.0" ?>
 <robot name="lift" xmlns:xacro="http://www.ros.org/wiki/xacro">
-  <xacro:arg name="type" default="r5"/>
+  <xacro:arg name="type" default="x5"/>
   <!-- 根据type参数包含不同的机械臂描述文件 -->
   <xacro:if value="${'$(arg type)' == 'x5'}">
-    <xacro:include filename="$(find x5_description)/xacro/X5.xacro"/>
+    <xacro:include filename="$(find arx5_description)/xacro/X5.xacro"/>
     <!-- 使用R5宏来创建两个机械臂 -->
-    <xacro:X5 name="left_arm"/>
-    <xacro:X5 name="right_arm"/>
+    <xacro:X5 name="left"/>
+    <xacro:X5 name="right"/>
   </xacro:if>
-  <xacro:unless value="${'$(arg type)' == 'x5'}">
-    <xacro:include filename="$(find r5_description)/xacro/R5.xacro"/>
+  <xacro:if value="${'$(arg type)' == 'r5'}">
+    <xacro:include filename="$(find arx5_description)/xacro/R5.xacro"/>
     <!-- 使用R5宏来创建两个机械臂 -->
-    <xacro:R5 name="left_arm"/>
-    <xacro:R5 name="right_arm"/>
-  </xacro:unless>
+    <xacro:R5 name="left"/>
+    <xacro:R5 name="right"/>
+  </xacro:if>
   <xacro:include filename="$(find lift_description)/xacro/mobile_base.xacro"/>
   <xacro:include filename="$(find lift_description)/xacro/body.xacro"/>
@@ -21,10 +21,10 @@
   <joint name="arm_left_fixed" type="fixed">
     <parent link="lift_1"/>
-    <child link="left_arm_base_link"/>
+    <child link="left_base_link"/>
     <origin rpy="0 0 3.1415926" xyz="-0.208 -0.25000 0.092"/>
   </joint>
   <joint name="arm_right_fixed" type="fixed">
     <parent link="lift_1"/>
-    <child link="right_arm_base_link"/>
+    <child link="right_base_link"/>
     <origin rpy="0 0 3.1415926" xyz="-0.208 0.25000 0.092"/>
   </joint>

File: humanoid/ARX/x7s_description/urdf/x7s.urdf (robot description, URDF)
Before this commit: robot X7S, 26 links, 25 joints
Links:
- link base_link: geometry collision mesh filename=package://x7s_description/meshes/base_link.obj; visual mesh filename=package://x7s_description/meshes/base_link.obj
- link body: geometry collision mesh filename=package://x7s_description/meshes/body.obj; visual mesh filename=package://x7s_description/meshes/body.obj
- link head: geometry collision mesh filename=package://x7s_description/meshes/head.obj; visual mesh filename=package://x7s_description/meshes/head.obj
- link head_camera: geometry visual mesh filename=package://arx5_description/meshes/d405.obj
- link left_elbow: geometry collision mesh filename=package://x7s_description/meshes/elbow.obj; visual mesh filename=package://x7s_description/meshes/elbow.obj
- link left_forearm: geometry collision mesh filename=package://x7s_description/meshes/forearm.obj; visual mesh filename=package://x7s_description/meshes/forearm.obj
- link left_gripper_base: geometry collision mesh filename=package://x7s_description/meshes/gripper_base.obj; visual mesh filename=package://x7s_description/meshes/gripper_base.obj
- link left_gripper_left: geometry collision mesh filename=package://x7s_description/meshes/gripper_left.obj; visual mesh filename=package://x7s_description/meshes/gripper_left.obj
- link left_gripper_right: geometry collision mesh filename=package://x7s_description/meshes/gripper_right.obj; visual mesh filename=package://x7s_description/meshes/gripper_right.obj
- link left_mount: geometry collision mesh filename=package://x7s_description/meshes/mount.obj; visual mesh filename=package://x7s_description/meshes/mount.obj
- link left_shoulder: geometry collision mesh filename=package://x7s_description/meshes/shoulder.obj; visual mesh filename=package://x7s_description/meshes/shoulder.obj
- link left_upper_arm: geometry collision mesh filename=package://x7s_description/meshes/upper_arm.obj; visual mesh filename=package://x7s_description/meshes/upper_arm.obj
- link left_wrist: geometry collision mesh filename=package://x7s_description/meshes/wrist.obj; visual mesh filename=package://x7s_description/meshes/wrist.obj
- link lift: geometry collision mesh filename=package://x7s_description/meshes/lift.obj; visual mesh filename=package://x7s_description/meshes/lift.obj
- link neck: geometry collision mesh filename=package://x7s_description/meshes/neck.obj; visual mesh filename=package://x7s_description/meshes/neck.obj
- link right_elbow: geometry collision mesh filename=package://x7s_description/meshes/elbow.obj scale=1 -1 1; visual mesh filename=package://x7s_description/meshes/elbow.obj scale=1 -1 1
- link right_forearm: geometry collision mesh filename=package://x7s_description/meshes/forearm.obj scale=1 -1 1; visual mesh filename=package://x7s_description/meshes/forearm.obj scale=1 -1 1
- link right_gripper_base: geometry collision mesh filename=package://x7s_description/meshes/gripper_base.obj; visual mesh filename=package://x7s_description/meshes/gripper_base.obj
- link right_gripper_left: geometry collision mesh filename=package://x7s_description/meshes/gripper_left.obj; visual mesh filename=package://x7s_description/meshes/gripper_left.obj
- link right_gripper_right: geometry collision mesh filename=package://x7s_description/meshes/gripper_right.obj; visual mesh filename=package://x7s_description/meshes/gripper_right.obj
- link right_mount: geometry collision mesh filename=package://x7s_description/meshes/mount.obj scale=1 -1 1; visual mesh filename=package://x7s_description/meshes/mount.obj scale=1 -1 1
- link right_shoulder: geometry collision mesh filename=package://x7s_description/meshes/shoulder.obj scale=1 -1 1; visual mesh filename=package://x7s_description/meshes/shoulder.obj scale=1 -1 1
- link right_upper_arm: geometry collision mesh filename=package://x7s_description/meshes/upper_arm.obj scale=1 -1 1; visual mesh filename=package://x7s_description/meshes/upper_arm.obj scale=1 -1 1
- link right_wrist: geometry collision mesh filename=package://x7s_description/meshes/wrist.obj scale=1 -1 1; visual mesh filename=package://x7s_description/meshes/wrist.obj scale=1 -1 1
Joints:
- joint head_joint: limit lower=-0.785398 upper=0.785398 effort=100 velocity=5 -> lower=-0.785398 upper=0.785398 effort=100 velocity=1000
- joint left_arm_yaw: limit lower=-1.570796 upper=1.570796 effort=100 velocity=5 -> lower=-1.570796 upper=1.570796 effort=100 velocity=1000
- joint left_elbow_pitch: limit lower=-0.785398 upper=1.570796 effort=100 velocity=5 -> lower=-0.785398 upper=1.570796 effort=100 velocity=1000
- joint left_elbow_roll: limit lower=-2.792527 upper=2.792527 effort=100 velocity=5 -> lower=-2.792527 upper=2.792527 effort=100 velocity=1000
- joint left_shoulder_pitch: limit lower=-0.523599 upper=3.141593 effort=100 velocity=5 -> lower=-0.523599 upper=3.141593 effort=100 velocity=1000
- joint left_shoulder_roll: limit lower=-0.436332 upper=1.570796 effort=100 velocity=5 -> lower=-0.436332 upper=1.570796 effort=100 velocity=1000
- joint left_wrist_pitch: limit lower=-0.785398 upper=1.570796 effort=100 velocity=5 -> lower=-0.785398 upper=1.570796 effort=100 velocity=1000
- joint lift_joint: limit lower=0 upper=0.54 effort=100 velocity=5 -> lower=0 upper=0.54 effort=100 velocity=1000
- joint right_arm_yaw: limit lower=-1.570796 upper=1.570796 effort=100 velocity=5 -> lower=-1.570796 upper=1.570796 effort=100 velocity=1000
- joint right_elbow_pitch: limit lower=-0.785398 upper=1.570796 effort=100 velocity=5 -> lower=-0.785398 upper=1.570796 effort=100 velocity=1000
- joint right_elbow_roll: limit lower=-2.792527 upper=2.792527 effort=100 velocity=5 -> lower=-2.792527 upper=2.792527 effort=100 velocity=1000
- joint right_gripper_0: limit lower=0 upper=0.044 effort=100 velocity=5 -> lower=0 upper=0.044 effort=100 velocity=1000
- joint right_gripper_1: limit lower=0 upper=0.044 effort=100 velocity=5 -> lower=0 upper=0.044 effort=100 velocity=1000
- joint right_shoulder_pitch: limit lower=-0.523599 upper=3.141593 effort=100 velocity=5 -> lower=-0.523599 upper=3.141593 effort=100 velocity=1000
- joint right_shoulder_roll: limit lower=-0.436332 upper=1.570796 effort=100 velocity=5 -> lower=-0.436332 upper=1.570796 effort=100 velocity=1000
- joint right_wrist_pitch: limit lower=-0.785398 upper=1.570796 effort=100 velocity=5 -> lower=-0.785398 upper=1.570796 effort=100 velocity=1000
- joint right_wrist_yaw: limit lower=-1.570796 upper=1.570796 effort=100 velocity=5 -> lower=-1.570796 upper=1.570796 effort=100 velocity=1000
