Commit message: add ros2 control xacro for arx5 and cr5

File: manipulator/ARX/arx5_description/xacro/X5.xacro (robot description, xacro)
@@ -264,5 +264,9 @@
       <parent link="${prefix}link6"/>
       <child link="${prefix}link8"/>
-      <axis xyz="0 -1 0"/>
+      <axis xyz="0 -1 0">
+        <mimic joint="${prefix}joint7">
+          <multiplier>1</multiplier>
+        </mimic>
+      </axis>
       <limit lower="0" upper="0.044" effort="100" velocity="5"/>
       <mimic joint="${prefix}joint7" multiplier="1" offset="0"/>
