Commit message: To avoid confusion, arx5 camera stand name, add prefix 'stand'

File: manipulator/ARX/arx5_description/xacro/R5.xacro (robot description, xacro)
@@ -299,5 +299,5 @@
 				<visual>
 					<geometry>
-						<mesh filename="file://$(find arx5_description)/meshes/camera_stand/d405.obj"/>
+						<mesh filename="file://$(find arx5_description)/meshes/camera_stand/stand_d405.obj"/>
 					</geometry>
 				</visual>
@@ -325,5 +325,5 @@
 				<visual>
 					<geometry>
-						<mesh filename="file://$(find arx5_description)/meshes/camera_stand/d435.obj"/>
+						<mesh filename="file://$(find arx5_description)/meshes/camera_stand/stand_d435.obj"/>
 					</geometry>
 				</visual>

File: manipulator/ARX/arx5_description/xacro/X5.xacro (robot description, xacro)
@@ -290,5 +290,5 @@
         <visual>
           <geometry>
-            <mesh filename="file://$(find arx5_description)/meshes/camera_stand/d405.obj"/>
+            <mesh filename="file://$(find arx5_description)/meshes/camera_stand/stand_d405.obj"/>
           </geometry>
         </visual>
@@ -316,5 +316,5 @@
         <visual>
           <geometry>
-            <mesh filename="file://$(find arx5_description)/meshes/camera_stand/d435.obj"/>
+            <mesh filename="file://$(find arx5_description)/meshes/camera_stand/stand_d435.obj"/>
           </geometry>
         </visual>
