Commit message: add panthera manipulator

File: gripper/robotiq_description/xacro/robotiq85.xacro (robot description, xacro)
@@ -199,5 +199,5 @@
     </link>
     <!-- Main actuated joint - left outer knuckle -->
-    <joint name="left_outer_knuckle_joint" type="revolute">
+    <joint name="finger_joint" type="revolute">
       <origin rpy="0 0 3.14159265359" xyz="0 -0.0306011 0.054904"/>
       <parent link="${prefix}base_link"/>
@@ -219,5 +219,5 @@
       <axis xyz="1 0 0"/>
       <limit effort="1000" lower="0" upper="0.8757" velocity="2.0"/>
-      <mimic joint="left_outer_knuckle_joint" multiplier="1" offset="0"/>
+      <mimic joint="finger_joint" multiplier="1" offset="0"/>
     </joint>
     <!-- Left inner finger has opposite motion to simulate the mechanical linkage -->
@@ -228,5 +228,5 @@
       <axis xyz="1 0 0"/>
       <limit effort="1000" lower="-0.8757" upper="0" velocity="2.0"/>
-      <mimic joint="left_outer_knuckle_joint" multiplier="-1" offset="0"/>
+      <mimic joint="finger_joint" multiplier="-1" offset="0"/>
     </joint>
     <joint name="left_inner_finger_pad_joint" type="fixed">
@@ -243,5 +243,5 @@
       <axis xyz="1 0 0"/>
       <limit effort="1000" lower="0" upper="0.81" velocity="2.0"/>
-      <mimic joint="left_outer_knuckle_joint" multiplier="1" offset="0"/>
+      <mimic joint="finger_joint" multiplier="1" offset="0"/>
     </joint>
     <joint name="right_outer_finger_joint" type="fixed">
@@ -257,5 +257,5 @@
       <axis xyz="1 0 0"/>
       <limit effort="1000" lower="0" upper="0.8757" velocity="2.0"/>
-      <mimic joint="left_outer_knuckle_joint" multiplier="1" offset="0"/>
+      <mimic joint="finger_joint" multiplier="1" offset="0"/>
     </joint>
     <joint name="right_inner_finger_joint" type="revolute">
@@ -265,5 +265,5 @@
       <axis xyz="1 0 0"/>
       <limit effort="1000" lower="-0.8757" upper="0" velocity="2.0"/>
-      <mimic joint="left_outer_knuckle_joint" multiplier="-1" offset="0"/>
+      <mimic joint="finger_joint" multiplier="-1" offset="0"/>
     </joint>
     <joint name="right_inner_finger_pad_joint" type="fixed">

File: gripper/robotiq_description/xacro/ros2_control/robotiq85.ros2_control.xacro (robot description, xacro)
@@ -17,5 +17,5 @@
       </hardware>
       <!-- 关节接口定义 -->
-      <joint name="left_outer_knuckle_joint">
+      <joint name="finger_joint">
         <command_interface name="position"/>
         <state_interface name="position">
@@ -24,24 +24,4 @@
         <state_interface name="velocity"/>
       </joint>
-<!--      <joint name="left_inner_knuckle_joint">-->
-<!--        <state_interface name="position"/>-->
-<!--        <state_interface name="velocity"/>-->
-<!--      </joint>-->
-<!--      <joint name="left_inner_finger_joint">-->
-<!--        <state_interface name="position"/>-->
-<!--        <state_interface name="velocity"/>-->
-<!--      </joint>-->
-<!--      <joint name="right_outer_knuckle_joint">-->
-<!--        <state_interface name="position"/>-->
-<!--        <state_interface name="velocity"/>-->
-<!--      </joint>-->
-<!--      <joint name="right_inner_knuckle_joint">-->
-<!--        <state_interface name="position"/>-->
-<!--        <state_interface name="velocity"/>-->
-<!--      </joint>-->
-<!--      <joint name="right_inner_finger_joint">-->
-<!--        <state_interface name="position"/>-->
-<!--        <state_interface name="velocity"/>-->
-<!--      </joint>-->
     </ros2_control>
   </xacro:macro>

File: manipulator/Ragtime-Lab/panthera_description/xacro/ros2_control/panthera.ros2_control.xacro (robot description, xacro)
@@ -1,5 +1,5 @@
 <?xml version="1.0"?>
 <robot xmlns:xacro="http://www.ros.org/wiki/xacro">
-  <xacro:macro name="cr5_system" params="name ros2_control_hardware_type">
+  <xacro:macro name="panthera_system" params="name ros2_control_hardware_type">
     <ros2_control name="${name}" type="system">
       <hardware>
@@ -19,7 +19,5 @@
       <joint name="joint1">
         <command_interface name="position"/>
-        <state_interface name="position">
-          <param name="initial_value">0</param>
-        </state_interface>
+        <state_interface name="position"/>
         <state_interface name="velocity"/>
         <state_interface name="effort"/>
@@ -28,5 +26,5 @@
         <command_interface name="position"/>
         <state_interface name="position">
-          <param name="initial_value">0</param>
+          <param name="initial_value">0.526</param>
         </state_interface>
         <state_interface name="velocity"/>
@@ -36,5 +34,5 @@
         <command_interface name="position"/>
         <state_interface name="position">
-          <param name="initial_value">-1.5708</param>
+          <param name="initial_value">0.119</param>
         </state_interface>
         <state_interface name="velocity"/>
@@ -44,5 +42,5 @@
         <command_interface name="position"/>
         <state_interface name="position">
-          <param name="initial_value">0</param>
+          <param name="initial_value">-0.391</param>
         </state_interface>
         <state_interface name="velocity"/>
@@ -51,7 +49,5 @@
       <joint name="joint5">
         <command_interface name="position"/>
-        <state_interface name="position">
-          <param name="initial_value">1.5708</param>
-        </state_interface>
+        <state_interface name="position"/>
         <state_interface name="velocity"/>
         <state_interface name="effort"/>
@@ -63,4 +59,13 @@
         <state_interface name="effort"/>
       </joint>
+      <joint name="gripper_joint">
+        <command_interface name="position"/>
+        <state_interface name="position">
+          <param name="initial_value">0.0</param>
+        </state_interface>
+        <state_interface name="velocity">
+          <param name="initial_value">0.0</param>
+        </state_interface>
+      </joint>
     </ros2_control>
   </xacro:macro>
