Commit message: simple collision and anti-self-collision planning for cr5

File: gripper/robotiq_description/xacro/robot.xacro (robot description, xacro)
@@ -1,4 +1,4 @@
 <?xml version="1.0"?>
-<robot name="Robotiq 85 single" xmlns:xacro="http://www.ros.org/wiki/xacro">
+<robot name="Robotiq85" xmlns:xacro="http://www.ros.org/wiki/xacro">
   <xacro:arg name="type" default="85"/>
   <!-- 根据type参数决定使用哪种夹爪 -->

File: gripper/robotiq_description/xacro/ros2_control/robotiq85.ros2_control.xacro (robot description, xacro)
@@ -12,6 +12,6 @@
         <xacro:if value="${ros2_control_hardware_type == 'isaac'}">
           <plugin>topic_based_ros2_control/TopicBasedSystem</plugin>
-          <param name="joint_commands_topic">/isaac_joint_commands</param>
-          <param name="joint_states_topic">/isaac_joint_states</param>
+          <param name="joint_commands_topic">/isaac/joint_command</param>
+          <param name="joint_states_topic">/isaac/joint_states</param>
         </xacro:if>
       </hardware>

File: manipulator/Dobot/cr5_description/urdf/cr5.urdf (robot description, URDF)
Before this commit: robot DobotCR5, 7 links, 6 joints
Links:
- link Link1: geometry collision cylinder length=0.17 radius=0.08; visual mesh filename=package://cr5_description/meshes/visual/Link1.obj
- link Link2: geometry collision cylinder length=0.18 radius=0.07; collision cylinder length=0.18 radius=0.07
- link Link3: geometry collision cylinder length=0.15 radius=0.05; collision cylinder length=0.15 radius=0.07
- link Link4: geometry collision cylinder length=0.155 radius=0.055; visual mesh filename=package://cr5_description/meshes/visual/Link4.obj
- link Link5: geometry collision cylinder length=0.18 radius=0.055; visual mesh filename=package://cr5_description/meshes/visual/Link5.obj
- link Link6: geometry collision box size=0.05 0.15 0.2; visual mesh filename=package://cr5_description/meshes/visual/Link6.obj
- link base_link: geometry collision box size=1.5 1.5 0.05; collision cylinder length=0.1 radius=0.1

File: manipulator/Dobot/cr5_description/xacro/arm.xacro (robot description, xacro)
@@ -1,5 +1,6 @@
 <?xml version="1.0"?>
 <robot name="cr5_robot" xmlns:xacro="http://ros.org/wiki/xacro">
-  <xacro:macro name="CR5" params="name">
+  <xacro:macro name="CR5" params="name collider:=convex">
+    <xacro:property name="prefix" value="${name + '_' if name else ''}"/>
     <link name="base_link">
       <inertial>
@@ -19,9 +20,24 @@
         </geometry>
       </visual>
-      <collision>
-        <geometry>
-          <mesh filename="file://$(find cr5_description)/meshes/collision/base_link.obj"/>
-        </geometry>
-      </collision>
+      <xacro:if value="${collider == 'convex'}">
+        <collision>
+          <geometry>
+            <mesh filename="file://$(find cr5_description)/meshes/collision/base_link.obj"/>
+          </geometry>
+        </collision>
+      </xacro:if>
+      <xacro:if value="${collider == 'simple'}">
+        <collision>
+          <origin xyz="0 0 0.05"/>
+          <geometry>
+            <cylinder length="0.1" radius="0.1"/>
+          </geometry>
+        </collision>
+        <collision>
+          <geometry>
+            <box size="1.5 1.5 0.05"/>
+          </geometry>
+        </collision>
+      </xacro:if>
     </link>
     <link name="Link1">
@@ -42,14 +58,23 @@
         </geometry>
       </visual>
-      <collision>
-        <geometry>
-          <mesh filename="file://$(find cr5_description)/meshes/collision/Link1_0.obj"/>
-        </geometry>
-      </collision>
-      <collision>
-        <geometry>
-          <mesh filename="file://$(find cr5_description)/meshes/collision/Link1_1.obj"/>
-        </geometry>
-      </collision>
+      <xacro:if value="${collider == 'convex'}">
+        <collision>
+          <geometry>
+            <mesh filename="file://$(find cr5_description)/meshes/collision/Link1_0.obj"/>
+          </geometry>
+        </collision>
+        <collision>
+          <geometry>
+            <mesh filename="file://$(find cr5_description)/meshes/collision/Link1_1.obj"/>
+          </geometry>
+        </collision>
+      </xacro:if>
+      <xacro:if value="${collider == 'simple'}">
+        <collision>
+          <geometry>
+            <cylinder length="0.17" radius="0.08"/>
+          </geometry>
+        </collision>
+      </xacro:if>
     </link>
     <joint name="joint1" type="revolute">
@@ -77,19 +102,41 @@
         </geometry>
       </visual>
-      <collision>
-        <geometry>
-          <mesh filename="file://$(find cr5_description)/meshes/collision/Link2_0.obj"/>
-        </geometry>
-      </collision>
-      <collision>
-        <geometry>
-          <mesh filename="file://$(find cr5_description)/meshes/collision/Link2_1.obj"/>
-        </geometry>
-      </collision>
-      <collision>
-        <geometry>
-          <mesh filename="file://$(find cr5_description)/meshes/collision/Link2_2.obj"/>
-        </geometry>
-      </collision>
+      <xacro:if value="${collider == 'convex'}">
+        <collision>
+          <geometry>
+            <mesh filename="file://$(find cr5_description)/meshes/collision/Link2_0.obj"/>
+          </geometry>
+        </collision>
+        <collision>
+          <geometry>
+            <mesh filename="file://$(find cr5_description)/meshes/collision/Link2_1.obj"/>
+          </geometry>
+        </collision>
+        <collision>
+          <geometry>
+            <mesh filename="file://$(find cr5_description)/meshes/collision/Link2_2.obj"/>
+          </geometry>
+        </collision>
+      </xacro:if>
+      <xacro:if value="${collider == 'simple'}">
+        <collision>
+          <origin rpy="0 0 0" xyz="0 0 0.145"/>
+          <geometry>
+            <cylinder length="0.18" radius="0.07"/>
+          </geometry>
+        </collision>
+        <collision>
+          <origin rpy="0 1.5708 0" xyz="-0.2 0 0.15"/>
+          <geometry>
+            <cylinder length="0.43" radius="0.065"/>
+          </geometry>
+        </collision>
+        <collision>
+          <origin xyz="-0.43 0 0.145"/>
+          <geometry>
+            <cylinder length="0.18" radius="0.07"/>
+          </geometry>
+        </collision>
+      </xacro:if>
     </link>
     <joint name="joint2" type="revolute">
@@ -117,19 +164,41 @@
         </geometry>
       </visual>
-      <collision>
-        <geometry>
-          <mesh filename="file://$(find cr5_description)/meshes/collision/Link3_0.obj"/>
-        </geometry>
-      </collision>
-      <collision>
-        <geometry>
-          <mesh filename="file://$(find cr5_description)/meshes/collision/Link3_1.obj"/>
-        </geometry>
-      </collision>
-      <collision>
-        <geometry>
-          <mesh filename="file://$(find cr5_description)/meshes/collision/Link3_2.obj"/>
-        </geometry>
-      </collision>
+      <xacro:if value="${collider == 'convex'}">
+        <collision>
+          <geometry>
+            <mesh filename="file://$(find cr5_description)/meshes/collision/Link3_0.obj"/>
+          </geometry>
+        </collision>
+        <collision>
+          <geometry>
+            <mesh filename="file://$(find cr5_description)/meshes/collision/Link3_1.obj"/>
+          </geometry>
+        </collision>
+        <collision>
+          <geometry>
+            <mesh filename="file://$(find cr5_description)/meshes/collision/Link3_2.obj"/>
+          </geometry>
+        </collision>
+      </xacro:if>
+      <xacro:if value="${collider == 'simple'}">
+        <collision>
+          <origin xyz="0 0 0.02"/>
+          <geometry>
+            <cylinder length="0.15" radius="0.07"/>
+          </geometry>
+        </collision>
+        <collision>
+          <origin rpy="0 1.5708 0" xyz="-0.2 0 0.03"/>
+          <geometry>
+            <cylinder length="0.35" radius="0.05"/>
+          </geometry>
+        </collision>
+        <collision>
+          <origin xyz="-0.355 0 0.02"/>
+          <geometry>
+            <cylinder length="0.15" radius="0.05"/>
+          </geometry>
+        </collision>
+      </xacro:if>
     </link>
     <joint name="joint3" type="revolute">
@@ -157,14 +226,24 @@
         </geometry>
       </visual>
-      <collision>
-        <geometry>
-          <mesh filename="file://$(find cr5_description)/meshes/collision/Link4_0.obj"/>
-        </geometry>
-      </collision>
-      <collision>
-        <geometry>
-          <mesh filename="file://$(find cr5_description)/meshes/collision/Link4_1.obj"/>
-        </geometry>
-      </collision>
+      <xacro:if value="${collider == 'convex'}">
+        <collision>
+          <geometry>
+            <mesh filename="file://$(find cr5_description)/meshes/collision/Link4_0.obj"/>
+          </geometry>
+        </collision>
+        <collision>
+          <geometry>
+            <mesh filename="file://$(find cr5_description)/meshes/collision/Link4_1.obj"/>
+          </geometry>
+        </collision>
+      </xacro:if>
+      <xacro:if value="${collider == 'simple'}">
+        <collision>
+          <origin rpy="1.5708 0 0" />
+          <geometry>
+            <cylinder length="0.155" radius="0.055"/>
+          </geometry>
+        </collision>
+      </xacro:if>
     </link>
     <joint name="joint4" type="revolute">
@@ -192,9 +271,19 @@
         </geometry>
       </visual>
-      <collision>
-        <geometry>
-          <mesh filename="file://$(find cr5_description)/meshes/collision/Link5.obj"/>
-        </geometry>
-      </collision>
+      <xacro:if value="${collider == 'convex'}">
+        <collision>
+          <geometry>
+            <mesh filename="file://$(find cr5_description)/meshes/collision/Link5.obj"/>
+          </geometry>
+        </collision>
+      </xacro:if>
+      <xacro:if value="${collider == 'simple'}">
+        <collision>
+          <origin rpy="1.5708 0 0" />
+          <geometry>
+            <cylinder length="0.18" radius="0.055"/>
+          </geometry>
+        </collision>
+      </xacro:if>
     </link>
     <joint name="joint5" type="revolute">
@@ -222,9 +311,19 @@
         </geometry>
       </visual>
-      <collision>
-        <geometry>
-          <mesh filename="file://$(find cr5_description)/meshes/collision/Link6.obj"/>
-        </geometry>
-      </collision>
+      <xacro:if value="${collider == 'convex'}">
+        <collision>
+          <geometry>
+            <mesh filename="file://$(find cr5_description)/meshes/collision/Link6.obj"/>
+          </geometry>
+        </collision>
+      </xacro:if>
+      <xacro:if value="${collider == 'simple'}">
+        <collision>
+          <origin xyz="0 0 0.1" />
+          <geometry>
+            <box size="0.05 0.15 0.2"/>
+          </geometry>
+        </collision>
+      </xacro:if>
     </link>
     <joint name="joint6" type="revolute">

File: manipulator/Dobot/cr5_description/xacro/robot.xacro (robot description, xacro)
@@ -2,6 +2,7 @@
 <robot name="DobotCR5" xmlns:xacro="http://www.ros.org/wiki/xacro">
   <xacro:arg name="type" default="empty"/>
+  <xacro:arg name="collider" default="convex"/>
   <xacro:include filename="$(find cr5_description)/xacro/arm.xacro"/>
-  <xacro:CR5 name=""/>
+  <xacro:CR5 name="" collider="$(arg collider)"/>
   <!-- 根据type参数决定使用哪种夹爪 -->
   <xacro:if value="${'$(arg type)' == 'robotiq85'}">

File: manipulator/Dobot/cr5_description/xacro/ros2_control/cr5.ros2_control.xacro (robot description, xacro)
@@ -12,5 +12,5 @@
         <xacro:if value="${ros2_control_hardware_type == 'isaac'}">
           <plugin>topic_based_ros2_control/TopicBasedSystem</plugin>
-          <param name="joint_commands_topic">/isaac/joint_commands</param>
+          <param name="joint_commands_topic">/isaac/joint_command</param>
           <param name="joint_states_topic">/isaac/joint_states</param>
         </xacro:if>
