Commit message: convex decompose for panthera robot

File: manipulator/Ragtime-Lab/panthera_description/xacro/panthera.xacro (robot description, xacro)
@@ -17,10 +17,15 @@
       <visual>
         <geometry>
-          <mesh filename="file://$(find panthera_description)/meshes/base_link.obj"/>
-        </geometry>
-      </visual>
-      <collision>
-        <geometry>
-          <mesh filename="file://$(find panthera_description)/meshes/base_link.obj"/>
+          <mesh filename="file://$(find panthera_description)/meshes/visual/base_link.obj"/>
+        </geometry>
+      </visual>
+      <collision>
+        <geometry>
+          <mesh filename="file://$(find panthera_description)/meshes/collision/base_link_0.obj"/>
+        </geometry>
+      </collision>
+      <collision>
+        <geometry>
+          <mesh filename="file://$(find panthera_description)/meshes/collision/base_link_1.obj"/>
         </geometry>
       </collision>
@@ -40,10 +45,20 @@
       <visual>
         <geometry>
-          <mesh filename="file://$(find panthera_description)/meshes/link1.obj"/>
-        </geometry>
-      </visual>
-      <collision>
-        <geometry>
-          <mesh filename="file://$(find panthera_description)/meshes/link1.obj"/>
+          <mesh filename="file://$(find panthera_description)/meshes/visual/link1.obj"/>
+        </geometry>
+      </visual>
+      <collision>
+        <geometry>
+          <mesh filename="file://$(find panthera_description)/meshes/collision/link1_0.obj"/>
+        </geometry>
+      </collision>
+      <collision>
+        <geometry>
+          <mesh filename="file://$(find panthera_description)/meshes/collision/link1_1.obj"/>
+        </geometry>
+      </collision>
+      <collision>
+        <geometry>
+          <mesh filename="file://$(find panthera_description)/meshes/collision/link1_2.obj"/>
         </geometry>
       </collision>
@@ -70,10 +85,15 @@
       <visual>
         <geometry>
-          <mesh filename="file://$(find panthera_description)/meshes/link2.obj"/>
-        </geometry>
-      </visual>
-      <collision>
-        <geometry>
-          <mesh filename="file://$(find panthera_description)/meshes/link2.obj"/>
+          <mesh filename="file://$(find panthera_description)/meshes/visual/link2.obj"/>
+        </geometry>
+      </visual>
+      <collision>
+        <geometry>
+          <mesh filename="file://$(find panthera_description)/meshes/collision/link2_0.obj"/>
+        </geometry>
+      </collision>
+      <collision>
+        <geometry>
+          <mesh filename="file://$(find panthera_description)/meshes/collision/link2_1.obj"/>
         </geometry>
       </collision>
@@ -100,10 +120,20 @@
       <visual>
         <geometry>
-          <mesh filename="file://$(find panthera_description)/meshes/link3.obj"/>
-        </geometry>
-      </visual>
-      <collision>
-        <geometry>
-          <mesh filename="file://$(find panthera_description)/meshes/link3.obj"/>
+          <mesh filename="file://$(find panthera_description)/meshes/visual/link3.obj"/>
+        </geometry>
+      </visual>
+      <collision>
+        <geometry>
+          <mesh filename="file://$(find panthera_description)/meshes/collision/link3_0.obj"/>
+        </geometry>
+      </collision>
+      <collision>
+        <geometry>
+          <mesh filename="file://$(find panthera_description)/meshes/collision/link3_1.obj"/>
+        </geometry>
+      </collision>
+      <collision>
+        <geometry>
+          <mesh filename="file://$(find panthera_description)/meshes/collision/link3_2.obj"/>
         </geometry>
       </collision>
@@ -130,10 +160,25 @@
       <visual>
         <geometry>
-          <mesh filename="file://$(find panthera_description)/meshes/link4.obj"/>
-        </geometry>
-      </visual>
-      <collision>
-        <geometry>
-          <mesh filename="file://$(find panthera_description)/meshes/link4.obj"/>
+          <mesh filename="file://$(find panthera_description)/meshes/visual/link4.obj"/>
+        </geometry>
+      </visual>
+      <collision>
+        <geometry>
+          <mesh filename="file://$(find panthera_description)/meshes/collision/link4_0.obj"/>
+        </geometry>
+      </collision>
+      <collision>
+        <geometry>
+          <mesh filename="file://$(find panthera_description)/meshes/collision/link4_1.obj"/>
+        </geometry>
+      </collision>
+      <collision>
+        <geometry>
+          <mesh filename="file://$(find panthera_description)/meshes/collision/link4_2.obj"/>
+        </geometry>
+      </collision>
+      <collision>
+        <geometry>
+          <mesh filename="file://$(find panthera_description)/meshes/collision/link4_3.obj"/>
         </geometry>
       </collision>
@@ -160,10 +205,20 @@
       <visual>
         <geometry>
-          <mesh filename="file://$(find panthera_description)/meshes/link5.obj"/>
-        </geometry>
-      </visual>
-      <collision>
-        <geometry>
-          <mesh filename="file://$(find panthera_description)/meshes/link5.obj"/>
+          <mesh filename="file://$(find panthera_description)/meshes/visual/link5.obj"/>
+        </geometry>
+      </visual>
+      <collision>
+        <geometry>
+          <mesh filename="file://$(find panthera_description)/meshes/collision/link5_0.obj"/>
+        </geometry>
+      </collision>
+      <collision>
+        <geometry>
+          <mesh filename="file://$(find panthera_description)/meshes/collision/link5_1.obj"/>
+        </geometry>
+      </collision>
+      <collision>
+        <geometry>
+          <mesh filename="file://$(find panthera_description)/meshes/collision/link5_2.obj"/>
         </geometry>
       </collision>
@@ -190,12 +245,7 @@
       <visual>
         <geometry>
-          <mesh filename="file://$(find panthera_description)/meshes/link6.obj"/>
-        </geometry>
-      </visual>
-      <collision>
-        <geometry>
-          <mesh filename="file://$(find panthera_description)/meshes/link6.obj"/>
-        </geometry>
-      </collision>
+          <mesh filename="file://$(find panthera_description)/meshes/visual/link6.obj"/>
+        </geometry>
+      </visual>
     </link>
     <joint name="${prefix}joint6" type="revolute">
@@ -220,10 +270,20 @@
       <visual>
         <geometry>
-          <mesh filename="file://$(find panthera_description)/meshes/gripper_center_link.obj"/>
-        </geometry>
-      </visual>
-      <collision>
-        <geometry>
-          <mesh filename="file://$(find panthera_description)/meshes/gripper_center_link.obj"/>
+          <mesh filename="file://$(find panthera_description)/meshes/visual/gripper_center_link.obj"/>
+        </geometry>
+      </visual>
+      <collision>
+        <geometry>
+          <mesh filename="file://$(find panthera_description)/meshes/collision/gripper_center_0.obj"/>
+        </geometry>
+      </collision>
+      <collision>
+        <geometry>
+          <mesh filename="file://$(find panthera_description)/meshes/collision/gripper_center_1.obj"/>
+        </geometry>
+      </collision>
+      <collision>
+        <geometry>
+          <mesh filename="file://$(find panthera_description)/meshes/collision/gripper_center_2.obj"/>
         </geometry>
       </collision>
@@ -249,10 +309,10 @@
       <visual>
         <geometry>
-          <mesh filename="file://$(find panthera_description)/meshes/gripper_pad.obj"/>
-        </geometry>
-      </visual>
-      <collision>
-        <geometry>
-          <mesh filename="file://$(find panthera_description)/meshes/gripper_pad.obj"/>
+          <mesh filename="file://$(find panthera_description)/meshes/visual/gripper_pad.obj"/>
+        </geometry>
+      </visual>
+      <collision>
+        <geometry>
+          <mesh filename="file://$(find panthera_description)/meshes/collision/gripper_pad.obj"/>
         </geometry>
       </collision>
@@ -278,10 +338,10 @@
       <visual>
         <geometry>
-          <mesh filename="file://$(find panthera_description)/meshes/gripper_pad.obj" scale="1 -1 1"/>
-        </geometry>
-      </visual>
-      <collision>
-        <geometry>
-          <mesh filename="file://$(find panthera_description)/meshes/gripper_pad.obj" scale="1 -1 1"/>
+          <mesh filename="file://$(find panthera_description)/meshes/visual/gripper_pad.obj" scale="1 -1 1"/>
+        </geometry>
+      </visual>
+      <collision>
+        <geometry>
+          <mesh filename="file://$(find panthera_description)/meshes/collision/gripper_pad.obj" scale="1 -1 1"/>
         </geometry>
       </collision>

File: manipulator/Ragtime-Lab/panthera_description/xacro/ros2_control/panthera.ros2_control.xacro (robot description, xacro)
@@ -12,6 +12,6 @@
         <xacro:if value="${ros2_control_hardware_type == 'isaac'}">
           <plugin>topic_based_ros2_control/TopicBasedSystem</plugin>
-          <param name="joint_commands_topic">/isaac_joint_commands</param>
-          <param name="joint_states_topic">/isaac_joint_states</param>
+          <param name="joint_commands_topic">/isaac/joint_command</param>
+          <param name="joint_states_topic">/isaac/joint_states</param>
         </xacro:if>
       </hardware>
