Commit message: add airbot mmk2

File: humanoid/Airbot/airbot_mmk2_description/urdf/airbot_mmk2.urdf (robot description, URDF)
Before this commit: robot mmk2, 28 links, 27 joints
Links:
- added link lft_behind_wheel_link, mass 0.15002; collision mesh filename=package://airbot_mmk2_description/meshes/support_wheel.obj; visual mesh filename=package://airbot_mmk2_description/meshes/support_wheel.obj
- added link lft_front_wheel_link, mass 0.15002; collision mesh filename=package://airbot_mmk2_description/meshes/support_wheel.obj; visual mesh filename=package://airbot_mmk2_description/meshes/support_wheel.obj
- added link rgt_behind_wheel_link, mass 0.15002; collision mesh filename=package://airbot_mmk2_description/meshes/support_wheel.obj; visual mesh filename=package://airbot_mmk2_description/meshes/support_wheel.obj
- added link rgt_front_wheel_link, mass 0.15002; collision mesh filename=package://airbot_mmk2_description/meshes/support_wheel.obj; visual mesh filename=package://airbot_mmk2_description/meshes/support_wheel.obj
- link lft_wheel_link: mass 1.15656808621832 -> 1.1566; geometry collision mesh filename=package://airbot_mmk2_description/meshes/drive_wheel.obj; visual mesh filename=package://airbot_mmk2_description/meshes/drive_wheel.obj
- link rgt_wheel_link: mass 1.15656808640541 -> 1.1566; geometry collision mesh filename=package://airbot_mmk2_description/meshes/drive_wheel.obj scale=1 1 -1; visual mesh filename=package://airbot_mmk2_description/meshes/drive_wheel.obj scale=1 1 -1
Joints:
- added joint lft_behind_wheel_joint: type fixed, parent base_link, child lft_behind_wheel_link, origin xyz=-0.1315 -0.1 0.097
- added joint lft_front_wheel_joint: type fixed, parent base_link, child lft_front_wheel_link, origin xyz=0.15482 0.0895 0.097
- added joint rgt_behind_wheel_joint: type fixed, parent base_link, child rgt_behind_wheel_link, origin xyz=-0.1315 0.1 0.097
- added joint rgt_front_wheel_joint: type fixed, parent base_link, child rgt_front_wheel_link, origin xyz=0.15482 -0.0895 0.097
- joint lft_wheel_joint: axis 0 0 1 -> 0 0 -1; limit lower=-3.1416 upper=3.1416 effort=6.5 velocity=0.7 -> (none); type revolute -> continuous

File: humanoid/Airbot/airbot_mmk2_description/xacro/mmk2_base.xacro (robot description, xacro)
@@ -19,23 +19,41 @@
     </collision>
   </link>
+  <link name="lft_wheel_link">
+    <inertial>
+      <origin xyz="2.9309E-07 5.2077E-06 -0.029871"/>
+      <mass value="1.1566"/>
+      <inertia ixx="0.0021045" ixy="6.963E-10" ixz="-1.9831E-08" iyy="0.0021045" iyz="-3.5159E-07" izz="0.0035528"/>
+    </inertial>
+    <visual>
+      <geometry>
+        <mesh filename="file://$(find airbot_mmk2_description)/meshes/drive_wheel.obj"/>
+      </geometry>
+    </visual>
+    <collision>
+      <geometry>
+        <mesh filename="file://$(find airbot_mmk2_description)/meshes/drive_wheel.obj"/>
+      </geometry>
+    </collision>
+  </link>
+  <joint name="lft_wheel_joint" type="continuous">
+    <origin xyz="0 0.16325 0.08401" rpy="1.5708 1.5708 0"/>
+    <parent link="base_link"/>
+    <child link="lft_wheel_link"/>
+    <axis xyz="0 0 -1"/>
+  </joint>
   <link name="rgt_wheel_link">
     <inertial>
-      <origin xyz="5.20143266670436E-06 5.37603125005695E-07 -0.0018711144360713"/>
-      <mass value="1.15656808640541"/>
-      <inertia ixx="0.0021044922532766" ixy="1.88606601059021E-10" ixz="-3.50324127667933E-07" iyy="0.00210448664280546"
-               iyz="-3.619495141978E-08" izz="0.00355284737378788"/>
-    </inertial>
-    <visual>
-      <geometry>
-        <mesh filename="file://$(find airbot_mmk2_description)/meshes/rgt_wheel_link.STL"/>
-      </geometry>
-      <material name="">
-        <color rgba="0.752941176470588 0.752941176470588 0.752941176470588 1"/>
-      </material>
-    </visual>
-    <collision>
-      <geometry>
-        <mesh
-            filename="file://$(find airbot_mmk2_description)/meshes/rgt_wheel_link.STL"/>
+      <origin xyz="2.9312E-07 5.2196E-06 0.029871"/>
+      <mass value="1.1566"/>
+      <inertia ixx="0.0021045" ixy="-8.6762E-11" ixz="1.9824E-08" iyy="0.0021045" iyz="3.5159E-07" izz="0.0035528"/>
+    </inertial>
+    <visual>
+      <geometry>
+        <mesh filename="file://$(find airbot_mmk2_description)/meshes/drive_wheel.obj" scale="1 1 -1"/>
+      </geometry>
+    </visual>
+    <collision>
+      <geometry>
+        <mesh filename="file://$(find airbot_mmk2_description)/meshes/drive_wheel.obj" scale="1 1 -1"/>
       </geometry>
     </collision>
@@ -48,31 +66,91 @@
     <limit lower="-3.1416" upper="3.1416" effort="6.5" velocity="0.7"/>
   </joint>
-  <link name="lft_wheel_link">
-    <inertial>
-      <origin xyz="1.28756699316335E-06 -5.0575586944921E-06 0.00187111444199509"/>
-      <mass value="1.15656808621832"/>
-      <inertia ixx="0.00210448719172768" ixy="-1.67788115008943E-09" ixz="8.7251015028674E-08" iyy="0.00210449170378954"
-               iyz="-3.41206350459015E-07" izz="0.00355284737380655"/>
-    </inertial>
-    <visual>
-      <geometry>
-        <mesh filename="file://$(find airbot_mmk2_description)/meshes/lft_wheel_link.STL"/>
-      </geometry>
-      <material name="">
-        <color rgba="0.752941176470588 0.752941176470588 0.752941176470588 1"/>
-      </material>
-    </visual>
-    <collision>
-      <geometry>
-        <mesh filename="file://$(find airbot_mmk2_description)/meshes/lft_wheel_link.STL"/>
-      </geometry>
-    </collision>
-  </link>
-  <joint name="lft_wheel_joint" type="revolute">
-    <origin xyz="0 0.16325 0.08401" rpy="1.5708 1.5708 0"/>
-    <parent link="base_link"/>
-    <child link="lft_wheel_link"/>
-    <axis xyz="0 0 1"/>
-    <limit lower="-3.1416" upper="3.1416" effort="6.5" velocity="0.7"/>
+  <link name="rgt_behind_wheel_link">
+    <inertial>
+      <origin xyz="0.0098797 -0.26998 -0.044087"/>
+      <mass value="0.15002"/>
+      <inertia ixx="0.00016534" ixy="1.4827E-07" ixz="-2.9264E-07" iyy="0.00014609" iyz="4.0633E-05" izz="9.3638E-05"/>
+    </inertial>
+    <visual>
+      <geometry>
+        <mesh filename="file://$(find airbot_mmk2_description)/meshes/support_wheel.obj"/>
+      </geometry>
+    </visual>
+    <collision>
+      <geometry>
+        <mesh filename="file://$(find airbot_mmk2_description)/meshes/support_wheel.obj"/>
+      </geometry>
+    </collision>
+  </link>
+  <joint name="rgt_behind_wheel_joint" type="fixed">
+    <origin xyz="-0.1315 0.1 0.097"/>
+    <parent link="base_link"/>
+    <child link="rgt_behind_wheel_link"/>
+  </joint>
+  <link name="lft_behind_wheel_link">
+    <inertial>
+      <origin xyz="-0.01012 -0.26998 -0.044087"/>
+      <mass value="0.15002"/>
+      <inertia ixx="0.00016534" ixy="1.4827E-07" ixz="-2.9264E-07" iyy="0.00014609" iyz="4.0633E-05" izz="9.3638E-05"/>
+    </inertial>
+    <visual>
+      <geometry>
+        <mesh filename="file://$(find airbot_mmk2_description)/meshes/support_wheel.obj"/>
+      </geometry>
+    </visual>
+    <collision>
+      <geometry>
+        <mesh filename="file://$(find airbot_mmk2_description)/meshes/support_wheel.obj"/>
+      </geometry>
+    </collision>
+  </link>
+  <joint name="lft_behind_wheel_joint" type="fixed">
+    <origin xyz="-0.1315 -0.1 0.097"/>
+    <parent link="base_link"/>
+    <child link="lft_behind_wheel_link"/>
+  </joint>
+  <link name="rgt_front_wheel_link">
+    <inertial>
+      <origin xyz="-0.01012 0.30602 -0.044087"/>
+      <mass value="0.15002"/>
+      <inertia ixx="0.00016534" ixy="1.4827E-07" ixz="-2.9264E-07" iyy="0.00014609" iyz="4.0633E-05" izz="9.3637E-05"/>
+    </inertial>
+    <visual>
+      <geometry>
+        <mesh filename="file://$(find airbot_mmk2_description)/meshes/support_wheel.obj"/>
+      </geometry>
+    </visual>
+    <collision>
+      <geometry>
+        <mesh filename="file://$(find airbot_mmk2_description)/meshes/support_wheel.obj"/>
+      </geometry>
+    </collision>
+  </link>
+  <joint name="rgt_front_wheel_joint" type="fixed">
+    <origin xyz="0.15482 -0.0895 0.097"/>
+    <parent link="base_link"/>
+    <child link="rgt_front_wheel_link"/>
+  </joint>
+  <link name="lft_front_wheel_link">
+    <inertial>
+      <origin xyz="0.0098797 0.30602 -0.044087"/>
+      <mass value="0.15002"/>
+      <inertia ixx="0.00016534" ixy="1.4827E-07" ixz="-2.9264E-07" iyy="0.00014609" iyz="4.0633E-05" izz="9.3637E-05"/>
+    </inertial>
+    <visual>
+      <geometry>
+        <mesh filename="file://$(find airbot_mmk2_description)/meshes/support_wheel.obj"/>
+      </geometry>
+    </visual>
+    <collision>
+      <geometry>
+        <mesh filename="file://$(find airbot_mmk2_description)/meshes/support_wheel.obj"/>
+      </geometry>
+    </collision>
+  </link>
+  <joint name="lft_front_wheel_joint" type="fixed">
+    <origin xyz="0.15482 0.0895 0.097"/>
+    <parent link="base_link"/>
+    <child link="lft_front_wheel_link"/>
   </joint>
   <link name="slide_link">
@@ -87,7 +165,4 @@
         <mesh filename="file://$(find airbot_mmk2_description)/meshes/slide.obj"/>
       </geometry>
-      <material name="">
-        <color rgba="0.752941176470588 0.752941176470588 0.752941176470588 1"/>
-      </material>
     </visual>
     <collision>
@@ -102,5 +177,5 @@
     <child link="slide_link"/>
     <axis xyz="0 0 1"/>
-    <limit lower="-0.04" upper="0.87" effort="5" velocity="0.3"/>
+    <limit lower="-0.04" upper="0.87" effort="500" velocity="0.3"/>
   </joint>
   <link name="head_yaw_link">
@@ -115,7 +190,4 @@
         <mesh filename="file://$(find airbot_mmk2_description)/meshes/head_yaw.obj"/>
       </geometry>
-      <material name="">
-        <color rgba="0.752941176470588 0.752941176470588 0.752941176470588 1"/>
-      </material>
     </visual>
     <collision>
@@ -143,7 +215,4 @@
         <mesh filename="file://$(find airbot_mmk2_description)/meshes/head_pitch.obj"/>
       </geometry>
-      <material name="">
-        <color rgba="0.752941176470588 0.752941176470588 0.752941176470588 1"/>
-      </material>
     </visual>
     <collision>
