Commit message: modified g1 interfaces

File: humanoid/Agibot/agibot_g1_description/xacro/robot.xacro (robot description, xacro)
@@ -4,5 +4,6 @@
 <!-- |    This file includes the base robot structure and both arms                    | -->
 <!-- =================================================================================== -->
-<robot name="genie" xmlns:xacro="http://www.ros.org/wiki/xacro">
+<robot name="Agibot G1" xmlns:xacro="http://www.ros.org/wiki/xacro">
+	<xacro:arg name="type" default="AG2F120S"/>
 	<!-- Include the base robot structure -->
 	<xacro:include filename="$(find agibot_g1_description)/xacro/g1_base.xacro"/>
@@ -12,9 +13,4 @@
 	<xacro:G1Arm name="left"/>
 	<xacro:G1Arm name="right" direction="-1"/>
-	<xacro:arg name="type" default="AG2F120S"/>
-	<!-- Include gripper -->
-	<xacro:include filename="$(find changingtek_description)/xacro/AG2F120S.xacro"/>
-	<xacro:AG2F120S name="left"/>
-	<xacro:AG2F120S name="right"/>
 	<!-- Arm base links -->
 	<link name="arm_base"/>
@@ -35,17 +31,23 @@
 		<origin rpy="-1.5707963267948966 0.0 3.141592653589793" xyz="0.0 -0.025 0.0"/>
 	</joint>
-	<!-- Gripper joints -->
-	<joint name="ee_left_joint" type="fixed">
-		<origin xyz="0 0 0.027727" rpy="0 0 3.1415"/>
-		<parent link="left_end_link"/>
-		<child link="left_gripper_base"/>
-	</joint>
-	<joint name="ee_right_joint" type="fixed">
-		<origin xyz="0 0 0.027727" rpy="0 0 3.1415"/>
-		<parent link="right_end_link"/>
-		<child link="right_gripper_base"/>
-	</joint>
-	<xacro:include filename="$(find agibot_g1_description)/xacro/120s_camera_stand.xacro"/>
-	<xacro:Camera name="left"/>
-	<xacro:Camera name="right"/>
+	<xacro:if value="${'$(arg type)' == 'AG2F120S'}">
+		<!-- Include gripper -->
+		<xacro:include filename="$(find changingtek_description)/xacro/AG2F120S.xacro"/>
+		<xacro:AG2F120S name="left"/>
+		<xacro:AG2F120S name="right"/>
+		<!-- Gripper joints -->
+		<joint name="ee_left_joint" type="fixed">
+			<origin xyz="0 0 0.027727" rpy="0 0 3.1415"/>
+			<parent link="left_end_link"/>
+			<child link="left_gripper_base"/>
+		</joint>
+		<joint name="ee_right_joint" type="fixed">
+			<origin xyz="0 0 0.027727" rpy="0 0 3.1415"/>
+			<parent link="right_end_link"/>
+			<child link="right_gripper_base"/>
+		</joint>
+		<xacro:include filename="$(find agibot_g1_description)/xacro/120s_camera_stand.xacro"/>
+		<xacro:Camera name="left"/>
+		<xacro:Camera name="right"/>
+	</xacro:if>
 </robot>

File: humanoid/Agibot/agibot_g1_description/xacro/ros2_control/g1_base_interfaces.xacro (robot description, xacro)
@@ -1,41 +1,44 @@
 <?xml version="1.0"?>
 <robot xmlns:xacro="http://www.ros.org/wiki/xacro">
-  <!-- G1基座关节接口宏定义 -->
-  <xacro:macro name="g1_base_interfaces">
-    <joint name="left_wheel_joint">
-      <command_interface name="velocity">
-        <param name="min">-1.0</param>
-        <param name="max">1.0</param>
-      </command_interface>
-      <state_interface name="position"/>
-      <state_interface name="velocity"/>
-      <state_interface name="effort"/>
-    </joint>
-    <joint name="right_wheel_joint">
-      <command_interface name="velocity">
-        <param name="min">-1.0</param>
-        <param name="max">1.0</param>
-      </command_interface>
-      <state_interface name="position"/>
-      <state_interface name="velocity"/>
-      <state_interface name="effort"/>
-    </joint>
-    <!-- 基座关节接口定义 -->
-    <joint name="body_joint1">
-      <command_interface name="position"/>
-      <state_interface name="position">
-        <param name="initial_value">0.1</param>
-      </state_interface>
-      <state_interface name="velocity"/>
-      <state_interface name="effort"/>
-    </joint>
-    <joint name="body_joint2">
-      <command_interface name="position"/>
-      <state_interface name="position">
-        <param name="initial_value">0.0</param>
-      </state_interface>
-      <state_interface name="velocity"/>
-      <state_interface name="effort"/>
-    </joint>
-  </xacro:macro>
+	<!-- G1基座关节接口宏定义 -->
+	<xacro:macro name="g1_base_interfaces">
+		<xacro:arg name="gazebo" default="false"/>
+		<xacro:if value="$(arg gazebo)">
+			<joint name="left_wheel_joint">
+				<command_interface name="velocity">
+					<param name="min">-1.0</param>
+					<param name="max">1.0</param>
+				</command_interface>
+				<state_interface name="position"/>
+				<state_interface name="velocity"/>
+				<state_interface name="effort"/>
+			</joint>
+			<joint name="right_wheel_joint">
+				<command_interface name="velocity">
+					<param name="min">-1.0</param>
+					<param name="max">1.0</param>
+				</command_interface>
+				<state_interface name="position"/>
+				<state_interface name="velocity"/>
+				<state_interface name="effort"/>
+			</joint>
+		</xacro:if>
+		<!-- 基座关节接口定义 -->
+		<joint name="body_joint1">
+			<command_interface name="position"/>
+			<state_interface name="position">
+				<param name="initial_value">0.1</param>
+			</state_interface>
+			<state_interface name="velocity"/>
+			<state_interface name="effort"/>
+		</joint>
+		<joint name="body_joint2">
+			<command_interface name="position"/>
+			<state_interface name="position">
+				<param name="initial_value">0.0</param>
+			</state_interface>
+			<state_interface name="velocity"/>
+			<state_interface name="effort"/>
+		</joint>
+	</xacro:macro>
 </robot>

Commit message: add omni picker

File: humanoid/Agibot/agibot_g1_description/xacro/robot.xacro (robot description, xacro)
@@ -51,3 +51,22 @@
 		<xacro:Camera name="right"/>
 	</xacro:if>
+	<xacro:if value="${'$(arg type)' == 'omni-picker'}">
+		<xacro:include filename="$(find agibot_omni_description)/xacro/omni_picker.xacro"/>
+		<xacro:omni-picker name="left"/>
+		<xacro:omni-picker name="right"/>
+		<!-- Gripper joints -->
+		<joint name="ee_left_joint" type="fixed">
+			<origin xyz="0 0 0.0052" rpy="0 0 1.5708"/>
+			<parent link="left_end_link"/>
+			<child link="left_gripper_base"/>
+		</joint>
+		<joint name="ee_right_joint" type="fixed">
+			<origin xyz="0 0 0.0052" rpy="0 0 -1.5708"/>
+			<parent link="right_end_link"/>
+			<child link="right_gripper_base"/>
+		</joint>
+		<xacro:include filename="$(find agibot_g1_description)/xacro/omnipicker_camera_stand.xacro"/>
+		<xacro:Camera name="left"/>
+		<xacro:Camera name="right"/>
+	</xacro:if>
 </robot>
