Commit message: add omni picker ros2 configuration

File: humanoid/Agibot/agibot_g1_description/xacro/ros2_control/robot.xacro (robot description, xacro)
@@ -40,4 +40,9 @@
 			<xacro:ag2f120s_interfaces name="right"/>
 		</xacro:if>
+		<xacro:if value="${'$(arg type)' == 'omni-picker'}">
+			<xacro:include filename="$(find agibot_omni_description)/xacro/ros2_control/omni_picker.xacro"/>
+			<xacro:omni_picker_interfaces name="left"/>
+			<xacro:omni_picker_interfaces name="right"/>
+		</xacro:if>
 	</ros2_control>
 	<xacro:arg name="gazebo" default="false" />

File: humanoid/Agibot/agibot_omni_description/xacro/omni_picker.xacro (robot description, xacro)
@@ -4,4 +4,5 @@
 		<xacro:property name="mesh_path" value="file://$(find agibot_omni_description)/meshes/omni_picker"/>
 		<xacro:property name="prefix" value="${name + '_' if name else ''}"/>
+		<xacro:property name="PI" value="3.1415926535897931"/>
 		<link name="${prefix}gripper_base">
 			<inertial>
@@ -40,9 +41,9 @@
 		</link>
 		<joint name="${prefix}gripper_joint" type="revolute">
-			<origin xyz="0 -0.0195 0.0565" rpy="-2.9951 -1.5708 -0.15964"/>
+			<origin xyz="0 -0.0195 0.0565" rpy="-2.9951 -${PI/2} -0.15964"/>
 			<parent link="${prefix}gripper_base"/>
 			<child link="${prefix}narrow1_Link"/>
 			<axis xyz="0 0 1"/>
-			<limit lower="0" upper="1" effort="0" velocity="0"/>
+			<limit lower="0" upper="1" effort="50" velocity="${PI}"/>
 		</joint>
 		<link name="${prefix}narrow2_Link">
@@ -74,5 +75,5 @@
 			<child link="${prefix}narrow2_Link"/>
 			<axis xyz="0 0 -1"/>
-			<limit lower="-3.14" upper="3.14" effort="0" velocity="0"/>
+			<limit lower="-${PI}" upper="${PI}" effort="50" velocity="${PI}"/>
 			<mimic joint="${prefix}gripper_joint" multiplier="0.02" offset="0"/>
 		</joint>
@@ -105,5 +106,5 @@
 			<child link="${prefix}narrow3_Link"/>
 			<axis xyz="0 0 -1"/>
-			<limit lower="-3.14" upper="3.14" effort="0" velocity="0"/>
+			<limit lower="-${PI}" upper="${PI}" effort="50" velocity="${PI}"/>
 			<mimic joint="${prefix}gripper_joint" multiplier="0.4" offset="0"/>
 		</joint>
@@ -114,5 +115,5 @@
 			<child link="${prefix}narrow4_Link"/>
 			<axis xyz="0 0 1"/>
-			<limit lower="-3.14" upper="3.14" effort="0" velocity="0"/>
+			<limit lower="-${PI}" upper="${PI}" effort="50" velocity="${PI}"/>
 		</joint>
 		<link name="${prefix}narrow_loop_Link">
@@ -140,9 +141,9 @@
 		</link>
 		<joint name="${prefix}narrow_loop_joint" type="revolute">
-			<origin xyz="0 -0.021633 0.07387" rpy="-2.9951 -1.5708 -0.15964"/>
+			<origin xyz="0 -0.021633 0.07387" rpy="-2.9951 -${PI/2} -0.15964"/>
 			<parent link="${prefix}gripper_base"/>
 			<child link="${prefix}narrow_loop_Link"/>
 			<axis xyz="0 0 1"/>
-			<limit lower="-3.14" upper="3.14" effort="0" velocity="0"/>
+			<limit lower="-${PI}" upper="${PI}" effort="50" velocity="${PI}"/>
 			<mimic joint="${prefix}gripper_joint" multiplier="1.5" offset="0"/>
 		</joint>
@@ -171,9 +172,9 @@
 		</link>
 		<joint name="${prefix}wide1_joint" type="revolute">
-			<origin xyz="0 0.0195 0.0565" rpy="-2.9951 -1.5708 -0.15964"/>
+			<origin xyz="0 0.0195 0.0565" rpy="-2.9951 -${PI/2} -0.15964"/>
 			<parent link="${prefix}gripper_base"/>
 			<child link="${prefix}wide1_Link"/>
 			<axis xyz="0 0 -1"/>
-			<limit lower="-3.14" upper="3.14" effort="0" velocity="0"/>
+			<limit lower="-${PI}" upper="${PI}" effort="50" velocity="${PI}"/>
 			<mimic joint="${prefix}gripper_joint" multiplier="1" offset="0"/>
 		</joint>
@@ -206,5 +207,5 @@
 			<child link="${prefix}wide2_Link"/>
 			<axis xyz="0 0 1"/>
-			<limit lower="-3.14" upper="3.14" effort="0" velocity="0"/>
+			<limit lower="-${PI}" upper="${PI}" effort="50" velocity="${PI}"/>
 			<mimic joint="${prefix}gripper_joint" multiplier="0.02" offset="0"/>
 		</joint>
@@ -237,5 +238,5 @@
 			<child link="${prefix}wide3_Link"/>
 			<axis xyz="0 0 1"/>
-			<limit lower="-3.14" upper="3.14" effort="0" velocity="0"/>
+			<limit lower="-${PI}" upper="${PI}" effort="50" velocity="${PI}"/>
 			<mimic joint="${prefix}gripper_joint" multiplier="0.4" offset="0"/>
 		</joint>
@@ -270,9 +271,9 @@
 		</link>
 		<joint name="${prefix}wide_loop_joint" type="revolute">
-			<origin xyz="0 0.021633 0.07387" rpy="-2.9951 -1.5708 -0.15964"/>
+			<origin xyz="0 0.021633 0.07387" rpy="-2.9951 -${PI/2} -0.15964"/>
 			<parent link="${prefix}gripper_base"/>
 			<child link="${prefix}wide_loop_Link"/>
 			<axis xyz="0 0 -1"/>
-			<limit lower="-3.14" upper="3.14" effort="0" velocity="0"/>
+			<limit lower="-${PI}" upper="${PI}" effort="50" velocity="${PI}"/>
 			<mimic joint="${prefix}gripper_joint" multiplier="1.5" offset="0"/>
 		</joint>
