Commit message: g1 omni picker ocs2 urdf

File: humanoid/Agibot/agibot_g1_description/urdf/agibot_g1_omni-picker.urdf (robot description, URDF)
Before this commit: robot Agibot G1, 30 links, 29 joints
Joints:
- joint left_eef_joint: origin xyz=0.0 0.0 0.25 -> xyz=0.0 0.0 0.15
- joint right_eef_joint: origin xyz=0.0 0.0 0.25 -> xyz=0.0 0.0 0.15
