Commit message: add agilex aloha v1

File: manipulator/AgileX/agilex_aloha_description/xacro/aloha_v2.xacro (robot description, xacro)
@@ -1,315 +1,68 @@
 <?xml version="1.0" encoding="utf-8" ?>
-<robot name="arx5_description" xmlns:xacro="http://www.ros.org/wiki/xacro">
-  <!-- <link name="footprint"/> -->
-  <xacro:include filename="$(find piper_description)/xacro/Piper.xacro"/>
-  <link name="footprint">
-  </link>
-  <!-- tracer base -->
-  <link name="base_link">
-    <visual>
-      <origin xyz="0 0 0" rpy="1.57 0 0"/>
-      <geometry>
-        <mesh filename="file://$(find agilex_aloha_description)/meshes/aloha_v2/tracer_base_link.obj"/>
-      </geometry>
-    </visual>
-    <collision>
-      <origin xyz="0 0 0" rpy="1.57 0 0"/>
-      <geometry>
-        <mesh filename="file://$(find agilex_aloha_description)/meshes/aloha_v2/tracer_base_link.obj"/>
-      </geometry>
-    </collision>
-  </link>
-  <link name="inertial_link">
-    <inertial>
-      <!--mass value="44.3898489950015" /-->
-      <mass value="132.3898489950015"/>
-      <!-- <mass value="50" /> -->
-      <!-- <origin xyz="-0.00065 -0.085 0.062" />
-      <inertia ixx="0.6022" ixy="-0.02364" ixz="-0.1197" iyy="1.7386" iyz="-0.001544" izz="2.0296" /> -->
-      <origin xyz="0.015 0.0231316650320557 0"/>
-      <!--<origin
-        xyz="-0.0145261552504705 0.0231316650320557 0.00586280190939592"
-        />-->
-      <inertia ixx="0.185196122711036"
-               ixy="4.30144213829512E-08"
-               ixz="5.81037523686401E-08"
-               iyy="0.364893736238929"
-               iyz="-0.000386720198091934"
-               izz="0.223868521722778"/>
-      <!--<inertia ixx="2.288641" ixy="0" ixz="0" iyy="5.103976" iyz="0" izz="3.431465" />-->
-    </inertial>
-  </link>
-  <joint name="inertial_joint" type="fixed">
-    <origin xyz="0 0 0"/>
-    <parent link="base_link"/>
-    <child link="inertial_link"/>
-  </joint>
-  <link name="right_wheel_link">
-    <inertial>
-      <mass value="6"/>
-      <inertia ixx="0.7171" ixy="0" ixz="0" iyy="0.1361" iyz="0" izz="0.7171"/>
-    </inertial>
-    <visual>
-      <geometry>
-        <mesh filename="file://$(find agilex_aloha_description)/meshes/aloha_v2/tracer_wheel.obj"/>
-      </geometry>
-    </visual>
-    <collision>
-      <geometry>
-        <mesh filename="file://$(find agilex_aloha_description)/meshes/aloha_v2/tracer_wheel.obj"/>
-      </geometry>
-    </collision>
-  </link>
-  <joint name="right_wheel" type="continuous">
-    <parent link="base_link"/>
-    <child link="right_wheel_link"/>
-    <origin xyz="0 -0.17 -0.082"/>
-    <axis xyz="0 1 0"/>
-  </joint>
-  <link name="left_wheel_link">
-    <inertial>
-      <mass value="6"/>
-      <inertia ixx="0.7171" ixy="0" ixz="0" iyy="0.1361" iyz="0" izz="0.7171"/>
-    </inertial>
-    <visual>
-      <geometry>
-        <mesh filename="file://$(find agilex_aloha_description)/meshes/aloha_v2/tracer_wheel.obj"/>
-      </geometry>
-    </visual>
-    <collision>
-      <geometry>
-        <mesh filename="file://$(find agilex_aloha_description)/meshes/aloha_v2/tracer_wheel.obj"/>
-      </geometry>
-    </collision>
-  </link>
-  <joint name="left_wheel" type="continuous">
-    <parent link="base_link"/>
-    <child link="left_wheel_link"/>
-    <origin xyz="0 0.17 -0.082"/>
-    <axis xyz="0 1 0"/>
-  </joint>
-  <link name="fl_castor_link">
-    <inertial>
-      <mass value="1"/>
-      <inertia ixx="0.7171" ixy="0" ixz="0" iyy="0.1361" iyz="0" izz="0.7171"/>
-    </inertial>
-    <visual>
-      <geometry>
-        <mesh filename="file://$(find agilex_aloha_description)/meshes/aloha_v2/castor_joint.obj"/>
-      </geometry>
-    </visual>
-  </link>
-  <joint name="fl_castor_wheel" type="continuous">
-    <parent link="base_link"/>
-    <child link="fl_castor_link"/>
-    <origin xyz="0.19 0.17 -0.038" rpy="-1.57 0 0"/>
-    <axis xyz="0 1 0"/>
-  </joint>
-  <link name="fr_castor_link">
-    <inertial>
-      <mass value="1"/>
-      <inertia ixx="0.7171" ixy="0" ixz="0" iyy="0.1361" iyz="0" izz="0.7171"/>
-    </inertial>
-    <visual>
-      <geometry>
-        <mesh filename="file://$(find agilex_aloha_description)/meshes/aloha_v2/castor_joint.obj"/>
-      </geometry>
-    </visual>
-  </link>
-  <joint name="fr_castor_wheel" type="continuous">
-    <origin xyz="0.18955 -0.17 -0.0380886" rpy="-1.57 0 0"/>
-    <parent link="base_link"/>
-    <child link="fr_castor_link"/>
-    <axis xyz="0 1 0"/>
-  </joint>
-  <link name="rr_castor_link">
-    <inertial>
-      <mass value="1"/>
-      <inertia ixx="0.7171" ixy="0" ixz="0" iyy="0.1361" iyz="0" izz="0.7171"/>
-    </inertial>
-    <visual>
-      <geometry>
-        <mesh filename="file://$(find agilex_aloha_description)/meshes/aloha_v2/castor_joint.obj"/>
-      </geometry>
-    </visual>
-  </link>
-  <joint name="rr_castor_wheel" type="continuous">
-    <origin xyz="-0.18955 -0.17 -0.0380886" rpy="-1.57 0 0"/>
-    <parent link="base_link"/>
-    <child link="rr_castor_link"/>
-    <axis xyz="0 1 0"/>
-  </joint>
-  <link name="rl_castor_link">
-    <inertial>
-      <mass value="1"/>
-      <inertia ixx="0.7171" ixy="0" ixz="0" iyy="0.1361" iyz="0" izz="0.7171"/>
-    </inertial>
-    <visual>
-      <geometry>
-        <mesh filename="file://$(find agilex_aloha_description)/meshes/aloha_v2/castor_joint.obj"/>
-      </geometry>
-    </visual>
-  </link>
-  <joint name="rl_castor_wheel" type="continuous">
-    <origin xyz="-0.18955 0.17 -0.0380886" rpy="-1.57 0 0"/>
-    <parent link="base_link"/>
-    <child link="rl_castor_link"/>
-    <axis xyz="0 1 0"/>
-  </joint>
-  <link name="fl_wheel_link">
-    <inertial>
-      <mass value="1"/>
-      <inertia ixx="0.3131" ixy="0" ixz="0" iyy="0.3131" iyz="0" izz="0.1361"/>
-    </inertial>
-    <visual>
-      <geometry>
-        <mesh filename="file://$(find agilex_aloha_description)/meshes/aloha_v2/castor.obj"/>
-      </geometry>
-    </visual>
-    <collision>
-      <geometry>-->
-        <mesh filename="file://$(find agilex_aloha_description)/meshes/aloha_v2/castor.obj"/>
-      </geometry>
-    </collision>
-  </link>
-  <joint name="fl_wheel" type="continuous">
-    <parent link="fl_castor_link"/>
-    <child link="fl_wheel_link"/>
-    <dynamics damping="0.0" friction="0.0"/>
-    <origin xyz="-0.0218084 0.077 0"/>
-    <axis xyz="0 0 1"/>
-  </joint>
-  <link name="fr_wheel_link">
-    <inertial>
-      <mass value="1"/>
-      <inertia ixx="0.3131" ixy="0" ixz="0" iyy="0.3131" iyz="0" izz="0.1361"/>
-    </inertial>
-    <visual>
-      <geometry>
-        <mesh filename="file://$(find agilex_aloha_description)/meshes/aloha_v2/castor.obj"/>
-      </geometry>
-    </visual>
-    <collision>
-      <geometry>-->
-        <mesh filename="file://$(find agilex_aloha_description)/meshes/aloha_v2/castor.obj"/>
-      </geometry>
-    </collision>
-  </link>
-  <joint name="fr_wheel" type="continuous">
-    <parent link="fr_castor_link"/>
-    <child link="fr_wheel_link"/>
-    <dynamics damping="0.0" friction="0.0"/>
-    <origin xyz="-0.0218084 0.077 0"/>
-    <axis xyz="0 0 1"/>
-  </joint>
-  <link name="rr_wheel_link">
-    <inertial>
-      <mass value="1"/>
-      <inertia ixx="0.3131" ixy="0" ixz="0" iyy="0.3131" iyz="0" izz="0.1361"/>
-    </inertial>
-    <visual>
-      <geometry>
-        <mesh filename="file://$(find agilex_aloha_description)/meshes/aloha_v2/castor.obj"/>
-      </geometry>
-    </visual>
-    <collision>
-      <geometry>
-        <mesh filename="file://$(find agilex_aloha_description)/meshes/aloha_v2/castor.obj"/>
-      </geometry>
-    </collision>
-  </link>
-  <joint name="rr_wheel" type="continuous">
-    <parent link="rr_castor_link"/>
-    <child link="rr_wheel_link"/>
-    <dynamics damping="0.0" friction="0.0"/>
-    <origin xyz="-0.0218084 0.077 0"/>
-    <axis xyz="0 0 1"/>
-  </joint>
-  <link name="rl_wheel_link">
-    <inertial>
-      <mass value="1"/>
-      <inertia ixx="0.3131" ixy="0" ixz="0" iyy="0.3131" iyz="0" izz="0.1361"/>
-    </inertial>
-    <visual>
-      <geometry>
-        <mesh filename="file://$(find agilex_aloha_description)/meshes/aloha_v2/castor.obj"/>
-      </geometry>
-    </visual>
-    <collision>
-      <geometry>
-        <mesh filename="file://$(find agilex_aloha_description)/meshes/aloha_v2/castor.obj"/>
-      </geometry>
-    </collision>
-  </link>
-  <joint name="rl_wheel" type="continuous">
-    <parent link="rl_castor_link"/>
-    <child link="rl_wheel_link"/>
-    <dynamics damping="0.0" friction="0.0"/>
-    <origin xyz="-0.0218084 0.077 0"/>
-    <axis xyz="0 0 1"/>
-  </joint>
-  <!-- aloha base -->
-  <joint name="base_joint" type="fixed">
-    <origin xyz="0 0 0.15"/>
-    <parent link="footprint"/>
-    <child link="base_link"/>
-    <axis xyz="0 0 0"/>
-  </joint>
-  <link name="body_Link">
-    <inertial>
-      <origin xyz="0.015107 -0.027922 0.00013672"/>
-      <mass value="3.736"/>
-      <inertia ixx="0.097545" ixy="-9.2609E-06" ixz="0.00015366" iyy="0.045841" iyz="-0.0020459" izz="0.084773"/>
-    </inertial>
-    <visual>
-      <origin xyz="0 0 0.168" rpy="0 0 3.14"/>
-      <geometry>
-        <mesh filename="file://$(find agilex_aloha_description)/meshes/aloha_v2/body.obj"/>
-      </geometry>
-    </visual>
-    <collision>
-      <origin xyz="0 0 0.168" rpy="0 0 3.14"/>
-      <geometry>
-        <mesh filename="file://$(find agilex_aloha_description)/meshes/aloha_v2/body.obj"/>
-      </geometry>
-    </collision>
-  </link>
-  <joint name="body_joint" type="fixed">
-    <origin xyz="0 0 0"/>
-    <parent link="footprint"/>
-    <child link="body_Link"/>
-    <axis xyz="0 0 0"/>
-  </joint>
-  <!--***************************** front-left ****************************** -->
-  <xacro:Piper name="fl"/>
-  <joint name="fl_base_joint" type="fixed">
-    <origin xyz="0.23875 0.3 0.775"/>
-    <parent link="body_Link"/>
-    <child link="fl_base_link"/>
-    <axis xyz="0.0 0.0 1.0"/>
-  </joint>
-  <!--***************************** front-right ****************************** -->
-  <xacro:Piper name="fr"/>
-  <joint name="fr_base_joint" type="fixed">
-    <origin xyz="0.23875 -0.3 0.775"/>
-    <parent link="body_Link"/>
-    <child link="fr_base_link"/>
-    <axis xyz="0.0 0.0 1.0"/>
-  </joint>
-  <!--***************************** back-left ****************************** -->
-  <xacro:Piper name="bl" is_master="true"/>
-  <joint name="bl_base_joint" type="fixed">
-    <origin xyz="-0.379 0.3075 0.901"/>
-    <parent link="body_Link"/>
-    <child link="bl_base_link"/>
-    <axis xyz="0.0 0.0 1.0"/>
-  </joint>
-  <!--***************************** back-right ****************************** -->
-  <xacro:Piper name="br" is_master="true"/>
-  <joint name="br_base_joint" type="fixed">
-    <origin xyz="-0.379 -0.3075 0.901"/>
-    <parent link="body_Link"/>
-    <child link="br_base_link"/>
-    <axis xyz="0.0 0.0 1.0"/>
-  </joint>
+<robot name="aloha v2" xmlns:xacro="http://www.ros.org/wiki/xacro">
+	<xacro:macro name="aloha_v2" params="chassis:=tracer">
+		<xacro:include filename="$(find piper_description)/xacro/Piper.xacro"/>
+		<xacro:if value="${chassis == 'tracer'}">
+			<xacro:include filename="$(find agilex_aloha_description)/xacro/base/tracer.xacro"/>
+		</xacro:if>
+		<xacro:if value="${chassis == 'tracer_v2'}">
+			<xacro:include filename="$(find agilex_aloha_description)/xacro/base/tracer_v2.xacro"/>
+		</xacro:if>
+		<!-- aloha base -->
+		<link name="body_Link">
+			<inertial>
+				<origin xyz="0.015107 -0.027922 0.00013672"/>
+				<mass value="3.736"/>
+				<inertia ixx="0.097545" ixy="-9.2609E-06" ixz="0.00015366" iyy="0.045841" iyz="-0.0020459" izz="0.084773"/>
+			</inertial>
+			<visual>
+				<geometry>
+					<mesh filename="file://$(find agilex_aloha_description)/meshes/aloha_v2/body.obj"/>
+				</geometry>
+			</visual>
+			<collision>
+				<geometry>
+					<mesh filename="file://$(find agilex_aloha_description)/meshes/aloha_v2/body.obj"/>
+				</geometry>
+			</collision>
+		</link>
+		<joint name="body_joint" type="fixed">
+			<origin xyz="0 0 0.168"/>
+			<parent link="base_footprint"/>
+			<child link="body_Link"/>
+			<axis/>
+		</joint>
+		<!--***************************** front-left ****************************** -->
+		<xacro:Piper name="fl"/>
+		<joint name="fl_base_joint" type="fixed">
+			<origin xyz="0.23875 0.3 0.607"/>
+			<parent link="body_Link"/>
+			<child link="fl_base_link"/>
+			<axis xyz="0 0 1"/>
+		</joint>
+		<!--***************************** front-right ****************************** -->
+		<xacro:Piper name="fr"/>
+		<joint name="fr_base_joint" type="fixed">
+			<origin xyz="0.23875 -0.3 0.607"/>
+			<parent link="body_Link"/>
+			<child link="fr_base_link"/>
+			<axis xyz="0 0 1"/>
+		</joint>
+		<!--***************************** back-left ****************************** -->
+		<xacro:Piper name="bl" is_master="true"/>
+		<joint name="bl_base_joint" type="fixed">
+			<origin xyz="-0.379 0.3075 0.733"/>
+			<parent link="body_Link"/>
+			<child link="bl_base_link"/>
+			<axis xyz="0 0 1"/>
+		</joint>
+		<!--***************************** back-right ****************************** -->
+		<xacro:Piper name="br" is_master="true"/>
+		<joint name="br_base_joint" type="fixed">
+			<origin xyz="-0.379 -0.3075 0.733"/>
+			<parent link="body_Link"/>
+			<child link="br_base_link"/>
+			<axis xyz="0 0 1"/>
+		</joint>
+	</xacro:macro>
 </robot>

File: manipulator/AgileX/agilex_aloha_description/xacro/robot.xacro (robot description, xacro)
@@ -6,6 +6,19 @@
     <xacro:include filename="$(find agilex_aloha_description)/xacro/aloha_split.xacro"/>
   </xacro:if>
+  <xacro:if value="${'$(arg type)' == 'v1'}">
+    <xacro:include filename="$(find agilex_aloha_description)/xacro/aloha_v1.xacro"/>
+    <xacro:aloha_v1/>
+  </xacro:if>
+  <xacro:if value="${'$(arg type)' == 'v1_x5'}">
+    <xacro:include filename="$(find agilex_aloha_description)/xacro/aloha_v1.xacro"/>
+    <xacro:aloha_v1 arm="x5"/>
+  </xacro:if>
   <xacro:if value="${'$(arg type)' == 'v2'}">
     <xacro:include filename="$(find agilex_aloha_description)/xacro/aloha_v2.xacro"/>
+    <xacro:aloha_v2/>
+  </xacro:if>
+  <xacro:if value="${'$(arg type)' == 'v2.1'}">
+    <xacro:include filename="$(find agilex_aloha_description)/xacro/aloha_v2.xacro"/>
+    <xacro:aloha_v2 chassis="tracer_v2"/>
   </xacro:if>
 </robot>
