Commit message: update camera models for galaxea

File: humanoid/Galaxea/galaxea_r1_description/xacro/realsense.xacro (robot description, xacro)
@@ -13,10 +13,16 @@
       <visual>
         <geometry>
-          <mesh filename="file://$(find galaxea_r1_description)/meshes/camera_link.obj"/>
+          <mesh filename="file://$(find galaxea_r1_description)/meshes/camera_stand.obj"/>
+        </geometry>
+      </visual>
+      <visual>
+        <origin rpy="${PI/2} ${-PI/2} 0" xyz="0.0325 0 0"/>
+        <geometry>
+          <mesh filename="file://$(find camera_models)/meshes/d435/d435.obj"/>
         </geometry>
       </visual>
       <collision>
         <geometry>
-          <mesh filename="file://$(find galaxea_r1_description)/meshes/camera_link.obj"/>
+          <mesh filename="file://$(find galaxea_r1_description)/meshes/camera_stand.obj"/>
         </geometry>
       </collision>

File: humanoid/Galaxea/galaxea_r1pro_description/xacro/realsense.xacro (robot description, xacro)
@@ -13,10 +13,16 @@
       <visual>
         <geometry>
-          <mesh filename="file://$(find galaxea_r1_description)/meshes/camera_link.obj"/>
+          <mesh filename="file://$(find galaxea_r1_description)/meshes/camera_stand.obj"/>
+        </geometry>
+      </visual>
+      <visual>
+        <origin rpy="${PI/2} ${-PI/2} 0" xyz="0.0325 0 0"/>
+        <geometry>
+          <mesh filename="file://$(find camera_models)/meshes/d435/d435.obj"/>
         </geometry>
       </visual>
       <collision>
         <geometry>
-          <mesh filename="file://$(find galaxea_r1_description)/meshes/camera_link.obj"/>
+          <mesh filename="file://$(find galaxea_r1_description)/meshes/camera_stand.obj"/>
         </geometry>
       </collision>

File: manipulator/Galaxea/galaxea_r1lite_description/urdf/galaxea_r1lite.urdf (robot description, URDF)
Before this commit: robot A1Lite, 36 links, 35 joints
Links:
- removed link left_D405_link
- removed link right_D405_link
Joints:
- removed joint left_D405_joint
- removed joint right_D405_joint

File: manipulator/Galaxea/galaxea_r1lite_description/xacro/robot.xacro (robot description, xacro)
@@ -6,4 +6,5 @@
 	<xacro:property name="PI" value="3.1415926535897931"/>
 	<xacro:include filename="$(find galaxea_r1lite_description)/xacro/chassis.xacro"/>
+	<xacro:include filename="$(find galaxea_r1lite_description)/xacro/camera.xacro"/>
 	<xacro:arg name="type" default="x"/>
 	<xacro:if value="${'$(arg type)' == 'x'}">
@@ -14,48 +15,6 @@
 	</xacro:if>
 	<xacro:Arm name="left"/>
-	<link name="left_D405_link">
-		<inertial>
-			<origin xyz="0.00904707172595565 0.0155186578135894 -0.00819594831599657"/>
-			<mass value="0.1"/>
-			<inertia ixx="2.7808294491585E-05" ixy="-4.06196123763752E-10" ixz="1.50543456146707E-08" iyy="2.1895142505718E-05" iyz="-3.73269688232892E-06" izz="2.07706210421564E-05"/>
-		</inertial>
-		<visual>
-			<geometry>
-				<mesh filename="file://$(find galaxea_r1lite_description)/meshes/visual/camera.obj"/>
-			</geometry>
-		</visual>
-		<collision>
-			<geometry>
-				<mesh filename="file://$(find galaxea_r1lite_description)/meshes/collision/camera.stl"/>
-			</geometry>
-		</collision>
-	</link>
-	<joint name="left_D405_joint" type="fixed">
-		<origin xyz="-0.019206 0.009 0.074757" rpy="-2.268 0 ${-PI/2}"/>
-		<parent link="left_gripper_base"/>
-		<child link="left_D405_link"/>
-	</joint>
+	<xacro:camera name="left"/>
 	<xacro:Arm name="right"/>
-	<link name="right_D405_link">
-		<inertial>
-			<origin xyz="0.00904707172594749 0.0155186578138565 -0.00819594831521042"/>
-			<mass value="0.1"/>
-			<inertia ixx="2.78082944930657E-05" ixy="-4.06196131154851E-10" ixz="1.50543456329152E-08" iyy="2.18951425070333E-05" iyz="-3.73269688187078E-06" izz="2.07706210423581E-05"/>
-		</inertial>
-		<visual>
-			<geometry>
-				<mesh filename="file://$(find galaxea_r1lite_description)/meshes/visual/camera.obj"/>
-			</geometry>
-		</visual>
-		<collision>
-			<geometry>
-				<mesh filename="file://$(find galaxea_r1lite_description)/meshes/collision/camera.stl"/>
-			</geometry>
-		</collision>
-	</link>
-	<joint name="right_D405_joint" type="fixed">
-		<origin xyz="-0.019206 0.009 0.074757" rpy="-2.268 0 ${-PI/2}"/>
-		<parent link="right_gripper_base"/>
-		<child link="right_D405_link"/>
-	</joint>
+	<xacro:camera name="right"/>
 </robot>
