Commit message: add airbot play demo for discoverse

File: manipulator/Airbot/airbot_play_description/xacro/ros2_control/interfaces.xacro (robot description, xacro)
@@ -1,56 +1,59 @@
 <?xml version="1.0"?>
 <robot xmlns:xacro="http://www.ros.org/wiki/xacro">
-  <xacro:macro name="airbot_play_interfaces" params="name">
-    <xacro:property name="prefix" value="${name + '_' if name else ''}"/>
-    <!-- 关节接口定义 -->
-    <joint name="${prefix}joint1">
-      <command_interface name="position"/>
-      <state_interface name="position"/>
-      <state_interface name="velocity"/>
-      <state_interface name="effort"/>
-    </joint>
-    <joint name="${prefix}joint2">
-      <command_interface name="position"/>
-      <state_interface name="position"/>
-      <state_interface name="velocity"/>
-      <state_interface name="effort"/>
-    </joint>
-    <joint name="${prefix}joint3">
-      <command_interface name="position"/>
-      <state_interface name="position"/>
-      <state_interface name="velocity"/>
-      <state_interface name="effort"/>
-    </joint>
-    <joint name="${prefix}joint4">
-      <command_interface name="position"/>
-      <state_interface name="position"/>
-      <state_interface name="velocity"/>
-      <state_interface name="effort"/>
-    </joint>
-    <joint name="${prefix}joint5">
-      <command_interface name="position"/>
-      <state_interface name="position"/>
-      <state_interface name="velocity"/>
-      <state_interface name="effort"/>
-    </joint>
-    <joint name="${prefix}joint6">
-      <command_interface name="position"/>
-      <state_interface name="position"/>
-      <state_interface name="velocity"/>
-      <state_interface name="effort"/>
-    </joint>
-    <joint name="${prefix}gripper_joint">
-      <command_interface name="position"/>
-      <state_interface name="position">
-        <param name="initial_value">0.01</param>
-      </state_interface>
-      <state_interface name="velocity"/>
-      <state_interface name="effort"/>
-    </joint>
-    <joint name="${prefix}gripper_joint1">
-      <state_interface name="position"/>
-      <state_interface name="velocity"/>
-      <state_interface name="effort"/>
-    </joint>
-  </xacro:macro>
+	<xacro:macro name="airbot_play_interfaces" params="name">
+		<xacro:arg name="gazebo" default="false"/>
+		<xacro:property name="prefix" value="${name + '_' if name else ''}"/>
+		<!-- 关节接口定义 -->
+		<joint name="${prefix}joint1">
+			<command_interface name="position"/>
+			<state_interface name="position"/>
+			<state_interface name="velocity"/>
+			<state_interface name="effort"/>
+		</joint>
+		<joint name="${prefix}joint2">
+			<command_interface name="position"/>
+			<state_interface name="position"/>
+			<state_interface name="velocity"/>
+			<state_interface name="effort"/>
+		</joint>
+		<joint name="${prefix}joint3">
+			<command_interface name="position"/>
+			<state_interface name="position"/>
+			<state_interface name="velocity"/>
+			<state_interface name="effort"/>
+		</joint>
+		<joint name="${prefix}joint4">
+			<command_interface name="position"/>
+			<state_interface name="position"/>
+			<state_interface name="velocity"/>
+			<state_interface name="effort"/>
+		</joint>
+		<joint name="${prefix}joint5">
+			<command_interface name="position"/>
+			<state_interface name="position"/>
+			<state_interface name="velocity"/>
+			<state_interface name="effort"/>
+		</joint>
+		<joint name="${prefix}joint6">
+			<command_interface name="position"/>
+			<state_interface name="position"/>
+			<state_interface name="velocity"/>
+			<state_interface name="effort"/>
+		</joint>
+		<joint name="${prefix}gripper_joint">
+			<command_interface name="position"/>
+			<state_interface name="position">
+				<param name="initial_value">0.01</param>
+			</state_interface>
+			<state_interface name="velocity"/>
+			<state_interface name="effort"/>
+		</joint>
+		<xacro:if value="$(arg gazebo)">
+			<joint name="${prefix}gripper_joint1">
+				<state_interface name="position"/>
+				<state_interface name="velocity"/>
+				<state_interface name="effort"/>
+			</joint>
+		</xacro:if>
+	</xacro:macro>
 </robot>

File: manipulator/Airbot/airbot_play_description/xacro/ros2_control/robot.xacro (robot description, xacro)
@@ -20,4 +20,9 @@
 				<param name="joint_states_topic">/isaac/joint_states</param>
 			</xacro:if>
+			<xacro:if value="${'$(arg ros2_control_hardware_type)' == 'discoverse'}">
+				<plugin>topic_based_ros2_control/TopicBasedSystem</plugin>
+				<param name="joint_commands_topic">/airbot_play/joint_command</param>
+				<param name="joint_states_topic">/airbot_play/joint_states</param>
+			</xacro:if>
 		</hardware>
 		<xacro:airbot_play_interfaces name=""/>
