Commit message: agilex mesh refactor

File: humanoid/Galaxea/galaxea_r1_description/urdf/galaxea_r1.urdf (robot description, URDF)
Before this commit: robot R1, 36 links, 35 joints
Links:
- link left_realsense_link: geometry collision mesh filename=package://galaxea_r1_description/meshes/camera_stand.obj; visual mesh filename=package://camera_models/meshes/d435/d435.obj
- link right_realsense_link: geometry collision mesh filename=package://galaxea_r1_description/meshes/camera_stand.obj; visual mesh filename=package://camera_models/meshes/d435/d435.obj
Joints:
- joint left_gripper_joint: limit lower=0 upper=0.05 effort=100 velocity=0.25 -> lower=0 upper=0.05 effort=10 velocity=0.25
- joint left_gripper_joint2: limit lower=0 upper=0.05 effort=100 velocity=0.25 -> lower=0 upper=0.05 effort=10 velocity=0.25
- joint right_gripper_joint: limit lower=0 upper=0.05 effort=100 velocity=0.25 -> lower=0 upper=0.05 effort=10 velocity=0.25
- joint right_gripper_joint2: limit lower=0 upper=0.05 effort=100 velocity=0.25 -> lower=0 upper=0.05 effort=10 velocity=0.25

File: humanoid/Galaxea/galaxea_r1pro_description/urdf/galaxea_r1pro.urdf (robot description, URDF)
Before this commit: robot R1Pro, 38 links, 37 joints
Links:
- link left_realsense_link: geometry collision mesh filename=package://galaxea_r1_description/meshes/camera_stand.obj; visual mesh filename=package://camera_models/meshes/d435/d435.obj
- link right_realsense_link: geometry collision mesh filename=package://galaxea_r1_description/meshes/camera_stand.obj; visual mesh filename=package://camera_models/meshes/d435/d435.obj
Joints:
- joint left_gripper_base_joint: origin xyz=-0.0295 0 -0.16065 rpy=0 1.5708 0 -> xyz=-0.0295 0 -0.16065 rpy=0 1.5707963267948966 0
- joint left_gripper_joint: limit lower=0 upper=0.05 effort=100 velocity=0.25 -> lower=0 upper=0.05 effort=10 velocity=0.25
- joint left_gripper_joint2: limit lower=0 upper=0.05 effort=100 velocity=0.25 -> lower=0 upper=0.05 effort=10 velocity=0.25
- joint left_joint2: limit lower=-0.1745 upper=3.1416 effort=55 velocity=7.1209 -> lower=-0.1745 upper=3.141592653589793 effort=55 velocity=7.1209
- joint left_joint7: limit lower=-1.5708 upper=1.5708 effort=18 velocity=10.4720 -> lower=-1.5707963267948966 upper=1.5707963267948966 effort=18 velocity=10.4720
- joint left_realsense_joint: origin xyz=0.02101 0.0028934 -0.1555183 rpy=2.70516 -0.0077831 -1.5708 -> xyz=0.02101 0.0028934 -0.1555183 rpy=2.70516 -0.0077831 -1.5707963267948966
- joint right_gripper_base_joint: origin xyz=-0.0295 0 -0.16065 rpy=0 1.5708 0 -> xyz=-0.0295 0 -0.16065 rpy=0 1.5707963267948966 0
- joint right_gripper_joint: limit lower=0 upper=0.05 effort=100 velocity=0.25 -> lower=0 upper=0.05 effort=10 velocity=0.25
- joint right_gripper_joint2: limit lower=0 upper=0.05 effort=100 velocity=0.25 -> lower=0 upper=0.05 effort=10 velocity=0.25
- joint right_joint2: limit lower=-0.1745 upper=3.1416 effort=55 velocity=7.1209 -> lower=-0.1745 upper=3.141592653589793 effort=55 velocity=7.1209
- joint right_joint7: limit lower=-1.5708 upper=1.5708 effort=18 velocity=10.4720 -> lower=-1.5707963267948966 upper=1.5707963267948966 effort=18 velocity=10.4720
- joint right_realsense_joint: origin xyz=0.02101 0.0028934 -0.1555183 rpy=2.70516 -0.0077831 -1.5708 -> xyz=0.02101 0.0028934 -0.1555183 rpy=2.70516 -0.0077831 -1.5707963267948966
- joint steer_motor_joint1: limit lower=-1.5708 upper=1.5708 effort=44 velocity=3.1416 -> lower=-1.5707963267948966 upper=1.5707963267948966 effort=44 velocity=3.141592653589793
- joint steer_motor_joint2: limit lower=-1.5708 upper=1.5708 effort=44 velocity=3.1416 -> lower=-1.5707963267948966 upper=1.5707963267948966 effort=44 velocity=3.141592653589793
- joint steer_motor_joint3: limit lower=-1.5708 upper=1.5708 effort=44 velocity=3.1416 -> lower=-1.5707963267948966 upper=1.5707963267948966 effort=44 velocity=3.141592653589793
- joint torso_joint3: limit lower=-1.8326 upper=1.5708 effort=500 velocity=2.5 -> lower=-1.8326 upper=1.5707963267948966 effort=500 velocity=2.5
- joint wheel_motor_joint1: origin xyz=0 0 -0.09525 rpy=0 0 3.14159 -> xyz=0 0 -0.09525 rpy=0 0 3.141592653589793
- joint wheel_motor_joint3: origin xyz=0 0 -0.09525 rpy=0 0 3.14159 -> xyz=0 0 -0.09525 rpy=0 0 3.141592653589793
- joint zed_joint: origin xyz=0.065512 0.060005 0.47598 rpy=-1.9199 0 -1.5708 -> xyz=0.065512 0.060005 0.47598 rpy=-1.9199 0 -1.5707963267948966

File: manipulator/ARX/arx5_description/urdf/arx5_agilex.urdf (robot description, URDF)
Before this commit: robot ARX 5, 14 links, 13 joints
Links:
- link base_link: mass 0.43995 -> 0.42272; geometry collision mesh filename=package://arx5_description/meshes/r5/base_link.obj; visual mesh filename=package://arx5_description/meshes/r5/base_link.obj
- link camera: geometry visual mesh filename=package://camera_models/meshes/d405/d405.obj
- link link1: mass 0.066982 -> 0.096804; geometry collision mesh filename=package://arx5_description/meshes/r5/link1.obj; visual mesh filename=package://arx5_description/meshes/r5/link1.obj
- link link2: mass 1.0795 -> 1.1988; geometry collision mesh filename=package://arx5_description/meshes/r5/link2.obj; visual mesh filename=package://arx5_description/meshes/r5/link2_agilex.obj
- link link3: mass 0.54534 -> 0.84082; geometry collision mesh filename=package://arx5_description/meshes/r5/link3.obj; visual mesh filename=package://arx5_description/meshes/r5/link3_agilex.obj
- link link4: mass 0.11714 -> 0.12432; geometry collision mesh filename=package://arx5_description/meshes/r5/link4.obj; visual mesh filename=package://arx5_description/meshes/r5/link4.obj
- link link5: mass 0.63488 -> 0.63601; geometry collision mesh filename=package://arx5_description/meshes/r5/link5.obj; visual mesh filename=package://arx5_description/meshes/r5/link5.obj
- link link6: geometry collision mesh filename=package://arx5_description/meshes/r5/link6.obj; visual mesh filename=package://arx5_description/meshes/r5/link6.obj
- link link7: geometry collision mesh filename=package://arx5_description/meshes/r5/link7.obj; visual mesh filename=package://arx5_description/meshes/r5/link7.obj
- link link8: mass 0.064798 -> 0.0647981725781684; geometry collision mesh filename=package://arx5_description/meshes/r5/link8.obj; visual mesh filename=package://arx5_description/meshes/r5/link8.obj
Joints:
- joint gripper_center_fixed: origin xyz=0.145 0 0 -> xyz=0.08657 0 0
- joint joint1: limit lower=-2.87 upper=3.14 effort=100 velocity=5 -> lower=-2.618 upper=2.168 effort=100 velocity=5; origin xyz=0 0 0.0605 -> xyz=0 0 0.0565
- joint joint2: origin xyz=0.02 0 0.04 -> xyz=0.02 0 0.047
- joint joint3: origin xyz=-0.264 0 0 rpy=3.1416 0 0 -> xyz=-0.264 0 0 rpy=-3.1416 0 0
- joint joint4: origin xyz=0.245 0 -0.056 -> xyz=0.245 -5E-05 -0.06
- joint joint5: origin xyz=0.06775 0.0005 -0.0865 -> xyz=0.0702 5E-05 -0.083391
- joint joint6: origin xyz=0.02895 0 0.0865 rpy=-3.1416 0 0 -> xyz=0.025286 0 0.083391 rpy=3.1416 0 0

File: manipulator/ARX/arx5_description/urdf/arx5_r5.urdf (robot description, URDF)
Before this commit: robot ARX 5, 12 links, 11 joints
Links:
- added link camera; visual mesh filename=package://camera_models/meshes/d405/d405.obj
- added link camera_support; visual mesh filename=package://arx5_description/meshes/camera_stand/stand_d405.o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
Joints:
- added joint camera_fixed: type fixed, parent camera_support, child camera, origin xyz=0.0385 0 0.0475 rpy=0 0.523 0
- added joint camera_support_fixed: type fixed, parent link6, child camera_support, origin xyz=0.045 0 0.021

File: manipulator/ARX/arx5_description/xacro/robot.xacro (robot description, xacro)
@@ -10,3 +10,7 @@
     <xacro:X5 name=""/>
   </xacro:if>
+  <xacro:if value="${'$(arg type)' == 'agilex'}">
+    <xacro:include filename="$(find arx5_description)/xacro/R5.xacro"/>
+    <xacro:R5 name="" style="agilex"/>
+  </xacro:if>
 </robot>

File: manipulator/AgileX/agilex_aloha_description/xacro/aloha_split.xacro (robot description, xacro)
@@ -44,12 +44,7 @@
     <visual>
       <geometry>
-        <mesh filename="file://$(find agilex_aloha_description)/meshes/aloha_split/camera.obj"/>
+        <mesh filename="file://$(find camera_models)/meshes/dabai/dabai.obj"/>
       </geometry>
     </visual>
-    <collision>
-      <geometry>
-        <mesh filename="file://$(find agilex_aloha_description)/meshes/aloha_split/camera.obj"/>
-      </geometry>
-    </collision>
   </link>
   <joint name="front_camera_joint" type="fixed">
@@ -75,9 +70,4 @@
       </geometry>
     </visual>
-    <collision>
-      <geometry>
-        <mesh filename="file://$(find camera_models)/meshes/mid360/mid360.obj"/>
-      </geometry>
-    </collision>
   </link>
   <joint name="lidar_joint" type="fixed">
@@ -130,12 +120,7 @@
     <visual>
       <geometry>
-        <mesh filename="file://$(find agilex_aloha_description)/meshes/aloha_split/camera.obj"/>
+        <mesh filename="file://$(find camera_models)/meshes/dabai/dabai.obj"/>
       </geometry>
     </visual>
-    <collision>
-      <geometry>
-        <mesh filename="file://$(find agilex_aloha_description)/meshes/aloha_split/camera.obj"/>
-      </geometry>
-    </collision>
   </link>
   <joint name="top_camera_joint" type="fixed">

File: manipulator/AgileX/agilex_aloha_description/xacro/aloha_v1.xacro (robot description, xacro)
@@ -110,4 +110,27 @@
 			<child link="camera_link2"/>
 		</joint>
+		<link name="lidar_link">
+			<inertial>
+				<origin xyz="-0.0022133 -0.00090659 0.025996"/>
+				<mass value="0.048617"/>
+				<inertia
+						ixx="1.0358E-05"
+						ixy="9.2377E-09"
+						ixz="-2.6386E-07"
+						iyy="1.0387E-05"
+						iyz="-2.6377E-07"
+						izz="1.7919E-05"/>
+			</inertial>
+			<visual>
+				<geometry>
+					<mesh filename="file://$(find camera_models)/meshes/mid360/mid360.obj"/>
+				</geometry>
+			</visual>
+		</link>
+		<joint name="lidar_joint" type="fixed">
+			<origin xyz="0.22937 0 0.040672"/>
+			<parent link="body_link"/>
+			<child link="lidar_link"/>
+		</joint>
 		<joint name="fl_base_joint" type="fixed">
 			<origin xyz="0.233 0.3 0.7775"/>

File: manipulator/AgileX/agilex_aloha_description/xacro/aloha_v2.xacro (robot description, xacro)
@@ -1,5 +1,5 @@
 <?xml version="1.0" encoding="utf-8" ?>
 <robot name="aloha v2" xmlns:xacro="http://www.ros.org/wiki/xacro">
-	<xacro:macro name="aloha_v2" params="chassis:=tracer">
+	<xacro:macro name="aloha_v2" params="chassis:=tracer enable_master:=false">
 		<xacro:include filename="$(find piper_description)/xacro/Piper.xacro"/>
 		<xacro:if value="${chassis == 'tracer'}">
@@ -33,36 +33,86 @@
 			<axis/>
 		</joint>
+		<link name="camera_link">
+			<inertial>
+				<origin xyz="-0.011443 2.4833E-05 -0.0012615"/>
+				<mass value="0.020053"/>
+				<inertia
+						ixx="1.1181E-05"
+						ixy="1.204E-07"
+						ixz="4.9068E-08"
+						iyy="2.2587E-06"
+						iyz="5.7637E-07"
+						izz="1.0097E-05"/>
+			</inertial>
+			<visual>
+				<geometry>
+					<mesh filename="file://$(find camera_models)/meshes/dabai/dabai.obj"/>
+				</geometry>
+			</visual>
+		</link>
+		<joint name="camera_joint" type="fixed">
+			<origin xyz="0.24007 0 0.91661" rpy="0 0.825 0"/>
+			<parent link="body_Link"/>
+			<child link="camera_link"/>
+		</joint>
+		<link name="lidar_link">
+			<inertial>
+				<origin xyz="-0.0022133 -0.00090659 0.025996"/>
+				<mass value="0.048617"/>
+				<inertia
+						ixx="1.0358E-05"
+						ixy="9.2377E-09"
+						ixz="-2.6386E-07"
+						iyy="1.0387E-05"
+						iyz="-2.6377E-07"
+						izz="1.7919E-05"/>
+			</inertial>
+			<visual>
+				<geometry>
+					<mesh filename="file://$(find camera_models)/meshes/mid360/mid360.obj"/>
+				</geometry>
+			</visual>
+		</link>
+		<joint name="lidar_joint" type="fixed">
+			<origin xyz="0.27289 0 0.01488"/>
+			<parent link="body_Link"/>
+			<child link="lidar_link"/>
+		</joint>
 		<!--***************************** front-left ****************************** -->
-		<xacro:Piper name="fl"/>
-		<joint name="fl_base_joint" type="fixed">
+		<xacro:Piper name="left"/>
+		<joint name="left_base_joint" type="fixed">
 			<origin xyz="0.23875 0.3 0.607"/>
 			<parent link="body_Link"/>
-			<child link="fl_base_link"/>
+			<child link="left_base_link"/>
 			<axis xyz="0 0 1"/>
 		</joint>
 		<!--***************************** front-right ****************************** -->
-		<xacro:Piper name="fr"/>
-		<joint name="fr_base_joint" type="fixed">
+		<xacro:Piper name="right"/>
+		<joint name="right_base_joint" type="fixed">
 			<origin xyz="0.23875 -0.3 0.607"/>
 			<parent link="body_Link"/>
-			<child link="fr_base_link"/>
+			<child link="right_base_link"/>
 			<axis xyz="0 0 1"/>
 		</joint>
 		<!--***************************** back-left ****************************** -->
-		<xacro:Piper name="bl" is_master="true"/>
-		<joint name="bl_base_joint" type="fixed">
-			<origin xyz="-0.379 0.3075 0.733"/>
-			<parent link="body_Link"/>
-			<child link="bl_base_link"/>
-			<axis xyz="0 0 1"/>
-		</joint>
+		<xacro:if value="${enable_master}">
+			<xacro:Piper name="bl" is_master="true"/>
+			<joint name="bl_base_joint" type="fixed">
+				<origin xyz="-0.379 0.3075 0.733"/>
+				<parent link="body_Link"/>
+				<child link="bl_base_link"/>
+				<axis xyz="0 0 1"/>
+			</joint>
+		</xacro:if>
 		<!--***************************** back-right ****************************** -->
-		<xacro:Piper name="br" is_master="true"/>
-		<joint name="br_base_joint" type="fixed">
-			<origin xyz="-0.379 -0.3075 0.733"/>
-			<parent link="body_Link"/>
-			<child link="br_base_link"/>
-			<axis xyz="0 0 1"/>
-		</joint>
+		<xacro:if value="${enable_master}">
+			<xacro:Piper name="br" is_master="true"/>
+			<joint name="br_base_joint" type="fixed">
+				<origin xyz="-0.379 -0.3075 0.733"/>
+				<parent link="body_Link"/>
+				<child link="br_base_link"/>
+				<axis xyz="0 0 1"/>
+			</joint>
+		</xacro:if>
 	</xacro:macro>
 </robot>

File: manipulator/AgileX/agilex_aloha_description/xacro/base/tracer.xacro (robot description, xacro)
@@ -3,5 +3,5 @@
 	<link name="base_footprint"/>
 	<joint name="base_joint" type="fixed">
-		<origin xyz="0 0 0.15"/>
+		<origin xyz="0 0 0.143"/>
 		<parent link="base_footprint"/>
 		<child link="base_link"/>
@@ -10,5 +10,4 @@
 	<link name="base_link">
 		<visual>
-			<origin rpy="1.57 0 0"/>
 			<geometry>
 				<mesh filename="file://$(find agilex_aloha_description)/meshes/tracer/tracer_base_link.obj"/>
@@ -16,5 +15,4 @@
 		</visual>
 		<collision>
-			<origin rpy="1.57 0 0"/>
 			<geometry>
 				<mesh filename="file://$(find agilex_aloha_description)/meshes/tracer/tracer_base_link.obj"/>
@@ -171,5 +169,5 @@
 		<child link="fl_wheel_link"/>
 		<dynamics damping="0.0" friction="0.0"/>
-		<origin xyz="-0.0218084 0.077 0"/>
+		<origin xyz="-0.022 0.06385 0"/>
 		<axis xyz="0 0 1"/>
 	</joint>
@@ -194,5 +192,5 @@
 		<child link="fr_wheel_link"/>
 		<dynamics damping="0.0" friction="0.0"/>
-		<origin xyz="-0.0218084 0.077 0"/>
+		<origin xyz="-0.022 0.06385 0"/>
 		<axis xyz="0 0 1"/>
 	</joint>
@@ -217,5 +215,5 @@
 		<child link="rr_wheel_link"/>
 		<dynamics damping="0.0" friction="0.0"/>
-		<origin xyz="-0.0218084 0.077 0"/>
+		<origin xyz="-0.022 0.06385 0"/>
 		<axis xyz="0 0 1"/>
 	</joint>
@@ -240,5 +238,5 @@
 		<child link="rl_wheel_link"/>
 		<dynamics damping="0.0" friction="0.0"/>
-		<origin xyz="-0.0218084 0.077 0"/>
+		<origin xyz="-0.022 0.06385 0"/>
 		<axis xyz="0 0 1"/>
 	</joint>
