Commit message: agilex mesh refactor

File: manipulator/AgileX/agilex_aloha_description/xacro/base/tracer_v2.xacro (robot description, xacro)
@@ -22,13 +22,10 @@
 		<visual>
 			<geometry>
-				<mesh filename="file://$(find agilex_aloha_description)/meshes/tracer_v2/base_link.STL"/>
-			</geometry>
-			<material name="">
-				<color rgba="1 1 1 1"/>
-			</material>
-		</visual>
-		<collision>
-			<geometry>
-				<mesh filename="file://$(find agilex_aloha_description)/meshes/tracer_v2/base_link.STL"/>
+				<mesh filename="file://$(find agilex_aloha_description)/meshes/tracer_v2/base.obj"/>
+			</geometry>
+		</visual>
+		<collision>
+			<geometry>
+				<mesh filename="file://$(find agilex_aloha_description)/meshes/tracer_v2/base.obj"/>
 			</geometry>
 		</collision>
@@ -48,41 +45,23 @@
 		<visual>
 			<geometry>
-				<mesh
-						filename="file://$(find agilex_aloha_description)/meshes/tracer_v2/right_link.STL"/>
-			</geometry>
-			<material
-					name="">
-				<color
-						rgba="1 1 1 1"/>
-			</material>
-		</visual>
-		<collision>
-			<geometry>
-				<mesh
-						filename="file://$(find agilex_aloha_description)/meshes/tracer_v2/right_link.STL"/>
-			</geometry>
-		</collision>
-	</link>
-	<joint
-			name="right_joint"
-			type="continuous">
-		<origin
-				xyz="-0.018818 -0.2537 -0.0905"
-				rpy="-1.5708 0 0"/>
-		<parent
-				link="base_link"/>
-		<child
-				link="right_link"/>
-		<axis
-				xyz="0 0 1"/>
-	</joint>
-	<link
-			name="left_Link">
-		<inertial>
-			<origin
-					xyz="-8.2507E-18 0 -0.005"
-			/>
-			<mass
-					value="0.14836"/>
+				<mesh filename="file://$(find agilex_aloha_description)/meshes/tracer_v2/drive_wheel.obj"/>
+			</geometry>
+		</visual>
+		<collision>
+			<geometry>
+				<mesh filename="file://$(find agilex_aloha_description)/meshes/tracer_v2/drive_wheel.obj"/>
+			</geometry>
+		</collision>
+	</link>
+	<joint name="right_joint" type="continuous">
+		<origin xyz="-0.018818 -0.2537 -0.0905" rpy="-1.5708 0 0"/>
+		<parent link="base_link"/>
+		<child link="right_link"/>
+		<axis xyz="0 0 1"/>
+	</joint>
+	<link name="left_Link">
+		<inertial>
+			<origin xyz="-8.2507E-18 0 -0.005"/>
+			<mass value="0.14836"/>
 			<inertia
 					ixx="0.00013099"
@@ -95,41 +74,23 @@
 		<visual>
 			<geometry>
-				<mesh
-						filename="file://$(find agilex_aloha_description)/meshes/tracer_v2/left_Link.STL"/>
-			</geometry>
-			<material
-					name="">
-				<color
-						rgba="1 1 1 1"/>
-			</material>
-		</visual>
-		<collision>
-			<geometry>
-				<mesh
-						filename="file://$(find agilex_aloha_description)/meshes/tracer_v2/left_Link.STL"/>
-			</geometry>
-		</collision>
-	</link>
-	<joint
-			name="left_joint"
-			type="continuous">
-		<origin
-				xyz="-0.018818 0.2537 -0.0905"
-				rpy="1.5708 0 0"/>
-		<parent
-				link="base_link"/>
-		<child
-				link="left_Link"/>
-		<axis
-				xyz="0 0 1"/>
-	</joint>
-	<link
-			name="right_front_link">
-		<inertial>
-			<origin
-					xyz="-0.013166 2.7397E-05 0.04181"
-			/>
-			<mass
-					value="0.2864"/>
+				<mesh filename="file://$(find agilex_aloha_description)/meshes/tracer_v2/drive_wheel.obj"/>
+			</geometry>
+		</visual>
+		<collision>
+			<geometry>
+				<mesh filename="file://$(find agilex_aloha_description)/meshes/tracer_v2/drive_wheel.obj"/>
+			</geometry>
+		</collision>
+	</link>
+	<joint name="left_joint" type="continuous">
+		<origin xyz="-0.018818 0.2537 -0.0905" rpy="1.5708 0 0"/>
+		<parent link="base_link"/>
+		<child link="left_Link"/>
+		<axis xyz="0 0 1"/>
+	</joint>
+	<link name="right_front_link">
+		<inertial>
+			<origin xyz="-0.013166 2.7397E-05 0.04181"/>
+			<mass value="0.2864"/>
 			<inertia
 					ixx="0.00029479"
@@ -142,41 +103,22 @@
 		<visual>
 			<geometry>
-				<mesh
-						filename="file://$(find agilex_aloha_description)/meshes/tracer_v2/right_front_link.STL"/>
-			</geometry>
-			<material
-					name="">
-				<color
-						rgba="1 1 1 1"/>
-			</material>
-		</visual>
-		<collision>
-			<geometry>
-				<mesh
-						filename="file://$(find agilex_aloha_description)/meshes/tracer_v2/right_front_link.STL"/>
-			</geometry>
-		</collision>
-	</link>
-	<joint
-			name="right_front_joint"
-			type="fixed">
-		<origin
-				xyz="0.23918 -0.1977 -0.058"
-				rpy="3.1416 0 0"/>
-		<parent
-				link="base_link"/>
-		<child
-				link="right_front_link"/>
-		<axis
-				xyz="0 0 0"/>
-	</joint>
-	<link
-			name="right_rear_link">
-		<inertial>
-			<origin
-					xyz="-0.013166 2.7397E-05 0.04181"
-			/>
-			<mass
-					value="0.2864"/>
+				<mesh filename="file://$(find agilex_aloha_description)/meshes/tracer_v2/support_wheel.obj"/>
+			</geometry>
+		</visual>
+		<collision>
+			<geometry>
+				<mesh filename="file://$(find agilex_aloha_description)/meshes/tracer_v2/support_wheel.obj"/>
+			</geometry>
+		</collision>
+	</link>
+	<joint name="right_front_joint" type="fixed">
+		<origin xyz="0.23918 -0.1977 -0.058" rpy="3.1416 0 0"/>
+		<parent link="base_link"/>
+		<child link="right_front_link"/>
+	</joint>
+	<link name="right_rear_link">
+		<inertial>
+			<origin xyz="-0.013166 2.7397E-05 0.04181"/>
+			<mass value="0.2864"/>
 			<inertia
 					ixx="0.00029479"
@@ -189,41 +131,22 @@
 		<visual>
 			<geometry>
-				<mesh
-						filename="file://$(find agilex_aloha_description)/meshes/tracer_v2/right_rear_link.STL"/>
-			</geometry>
-			<material
-					name="">
-				<color
-						rgba="1 1 1 1"/>
-			</material>
-		</visual>
-		<collision>
-			<geometry>
-				<mesh
-						filename="file://$(find agilex_aloha_description)/meshes/tracer_v2/right_rear_link.STL"/>
-			</geometry>
-		</collision>
-	</link>
-	<joint
-			name="right_rea_joint"
-			type="fixed">
-		<origin
-				xyz="-0.27082 -0.183 -0.058"
-				rpy="3.1416 0 0"/>
-		<parent
-				link="base_link"/>
-		<child
-				link="right_rear_link"/>
-		<axis
-				xyz="0 0 0"/>
-	</joint>
-	<link
-			name="left_front_link">
-		<inertial>
-			<origin
-					xyz="-0.013166 -2.7397E-05 -0.04181"
-			/>
-			<mass
-					value="0.2864"/>
+				<mesh filename="file://$(find agilex_aloha_description)/meshes/tracer_v2/support_wheel.obj"/>
+			</geometry>
+		</visual>
+		<collision>
+			<geometry>
+				<mesh filename="file://$(find agilex_aloha_description)/meshes/tracer_v2/support_wheel.obj"/>
+			</geometry>
+		</collision>
+	</link>
+	<joint name="right_rea_joint" type="fixed">
+		<origin xyz="-0.27082 -0.183 -0.058" rpy="3.1416 0 0"/>
+		<parent link="base_link"/>
+		<child link="right_rear_link"/>
+	</joint>
+	<link name="left_front_link">
+		<inertial>
+			<origin xyz="-0.013166 -2.7397E-05 -0.04181"/>
+			<mass value="0.2864"/>
 			<inertia
 					ixx="0.00029479"
@@ -236,76 +159,44 @@
 		<visual>
 			<geometry>
-				<mesh
-						filename="file://$(find agilex_aloha_description)/meshes/tracer_v2/left_front_link.STL"/>
-			</geometry>
-			<material
-					name="">
-				<color
-						rgba="1 1 1 1"/>
-			</material>
-		</visual>
-		<collision>
-			<geometry>
-				<mesh
-						filename="file://$(find agilex_aloha_description)/meshes/tracer_v2/left_front_link.STL"/>
-			</geometry>
-		</collision>
-	</link>
-	<joint
-			name="left_front_joint"
-			type="fixed">
-		<origin
-				xyz="0.23918 0.1977 -0.058"
-		/>
-		<parent
-				link="base_link"/>
-		<child
-				link="left_front_link"/>
-		<axis
-				xyz="0 0 0"/>
-	</joint>
-	<link
-			name="left_rear_link">
-		<inertial>
-			<mass
-					value="0"/>
-			<inertia
-					ixx="0"
-					ixy="0"
-					ixz="0"
-					iyy="0"
-					iyz="0"
-					izz="0"/>
-		</inertial>
-		<visual>
-			<geometry>
-				<mesh
-						filename="file://$(find agilex_aloha_description)/meshes/tracer_v2/left_rear_link.STL"/>
-			</geometry>
-			<material
-					name="">
-				<color
-						rgba="1 1 1 1"/>
-			</material>
-		</visual>
-		<collision>
-			<geometry>
-				<mesh
-						filename="file://$(find agilex_aloha_description)/meshes/tracer_v2/left_rear_link.STL"/>
-			</geometry>
-		</collision>
-	</link>
-	<joint
-			name="left_rear_joint"
-			type="fixed">
-		<origin
-				xyz="-0.27077 0.18305 -0.058"
-		/>
-		<parent
-				link="base_link"/>
-		<child
-				link="left_rear_link"/>
-		<axis
-				xyz="0 0 0"/>
+				<mesh filename="file://$(find agilex_aloha_description)/meshes/tracer_v2/support_wheel.obj"/>
+			</geometry>
+		</visual>
+		<collision>
+			<geometry>
+				<mesh filename="file://$(find agilex_aloha_description)/meshes/tracer_v2/support_wheel.obj"/>
+			</geometry>
+		</collision>
+	</link>
+	<joint name="left_front_joint" type="fixed">
+		<origin xyz="0.23918 0.1977 -0.058"/>
+		<parent link="base_link"/>
+		<child link="left_front_link"/>
+	</joint>
+	<link name="left_rear_link">
+		<inertial>
+			<mass value="0.2864"/>
+			<inertia
+					ixx="0.00029479"
+					ixy="-5.5901E-08"
+					ixz="-5.9543E-05"
+					iyy="0.00032696"
+					iyz="-1.5316E-07"
+					izz="0.00020885"/>
+		</inertial>
+		<visual>
+			<geometry>
+				<mesh filename="file://$(find agilex_aloha_description)/meshes/tracer_v2/support_wheel.obj"/>
+			</geometry>
+		</visual>
+		<collision>
+			<geometry>
+				<mesh filename="file://$(find agilex_aloha_description)/meshes/tracer_v2/support_wheel.obj"/>
+			</geometry>
+		</collision>
+	</link>
+	<joint name="left_rear_joint" type="fixed">
+		<origin xyz="-0.27077 0.18305 -0.058"/>
+		<parent link="base_link"/>
+		<child link="left_rear_link"/>
 	</joint>
 </robot>

File: manipulator/AgileX/agilex_aloha_description/xacro/robot.xacro (robot description, xacro)
@@ -18,7 +18,11 @@
     <xacro:aloha_v2/>
   </xacro:if>
-  <xacro:if value="${'$(arg type)' == 'v2.1'}">
+  <xacro:if value="${'$(arg type)' == 'v2-1'}">
     <xacro:include filename="$(find agilex_aloha_description)/xacro/aloha_v2.xacro"/>
     <xacro:aloha_v2 chassis="tracer_v2"/>
   </xacro:if>
+  <xacro:if value="${'$(arg type)' == 'v2-master'}">
+    <xacro:include filename="$(find agilex_aloha_description)/xacro/aloha_v2.xacro"/>
+    <xacro:aloha_v2 chassis="tracer_v2" enable_master="true"/>
+  </xacro:if>
 </robot>

File: manipulator/Galaxea/galaxea_r1lite_description/urdf/galaxea_r1lite_y.urdf (robot description, URDF)
Before this commit: robot A1Lite, 36 links, 35 joints
Links:
- link left_camera_stand: geometry collision mesh filename=package://galaxea_r1lite_description/meshes/collision/camer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; visual mesh filename=package://galaxea_r1lite_description/meshes/visual/camera_s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
- link left_link3: mass 0.739 -> 0.762; geometry collision mesh filename=package://galaxea_a1_description/meshes/a1_xy/a1_y/link3.obj; visual mesh filename=package://galaxea_a1_description/meshes/a1_xy/a1_y/link3.obj
- link left_link4: mass 0.419 -> 0.353; geometry collision mesh filename=package://galaxea_a1_description/meshes/a1_xy/a1_y/link4.obj; visual mesh filename=package://galaxea_a1_description/meshes/a1_xy/a1_y/link4.obj
- link left_link5: mass 0.054 -> 0.366; geometry collision mesh filename=package://galaxea_a1_description/meshes/a1_xy/a1_y/link5.obj; visual mesh filename=package://galaxea_a1_description/meshes/a1_xy/a1_y/link5.obj
- link right_camera_stand: geometry collision mesh filename=package://galaxea_r1lite_description/meshes/collision/camer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; visual mesh filename=package://galaxea_r1lite_description/meshes/visual/camera_s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
- link right_link3: mass 0.739 -> 0.762; geometry collision mesh filename=package://galaxea_a1_description/meshes/a1_xy/a1_y/link3.obj; visual mesh filename=package://galaxea_a1_description/meshes/a1_xy/a1_y/link3.obj
- link right_link4: mass 0.419 -> 0.353; geometry collision mesh filename=package://galaxea_a1_description/meshes/a1_xy/a1_y/link4.obj; visual mesh filename=package://galaxea_a1_description/meshes/a1_xy/a1_y/link4.obj
- link right_link5: mass 0.054 -> 0.366; geometry collision mesh filename=package://galaxea_a1_description/meshes/a1_xy/a1_y/link5.obj; visual mesh filename=package://galaxea_a1_description/meshes/a1_xy/a1_y/link5.obj
Joints:
- joint left_joint3: limit lower=-3.3161 upper=0 effort=27 velocity=10.472 -> lower=-3.316127 upper=0 effort=27 velocity=10.4720; origin xyz=-0.3 0.00025004 0 -> xyz=-0.3 0.00024449 0
- joint left_joint4: axis 0 1 0 -> 1 0 0; limit lower=-3.141592653589793 upper=3.141592653589793 effort=14 velocity=32.9867 -> lower=-2.879795 upper=2.879795 effort=14 velocity=32.9867; origin xyz=0.1747 0.00049739 0.075485 -> xyz=0.1544 -0.030998 0.075485
- joint left_joint5: axis 0 0 1 -> 0 1 0; limit lower=-3.141592653589793 upper=3.141592653589793 effort=14 velocity=32.9867 -> lower=-1.832597 upper=1.832597 effort=14 velocity=32.9867; origin xyz=0.08 -0.031498 0.0405 -> xyz=0.0418 0.023501 0
- joint left_joint6: limit lower=-2.8798 upper=2.8798 effort=14 velocity=32.9867 -> lower=-2.879795 upper=2.879795 effort=14 velocity=32.9867; origin xyz=0.022503 0 -0.0405 -> xyz=0.081 -0.023499 0
- joint right_joint3: limit lower=-3.3161 upper=0 effort=27 velocity=10.472 -> lower=-3.316127 upper=0 effort=27 velocity=10.4720; origin xyz=-0.3 0.00025004 0 -> xyz=-0.3 0.00024449 0
- joint right_joint4: axis 0 1 0 -> 1 0 0; limit lower=-3.141592653589793 upper=3.141592653589793 effort=14 velocity=32.9867 -> lower=-2.879795 upper=2.879795 effort=14 velocity=32.9867; origin xyz=0.1747 0.00049739 0.075485 -> xyz=0.1544 -0.030998 0.075485
- joint right_joint5: axis 0 0 1 -> 0 1 0; limit lower=-3.141592653589793 upper=3.141592653589793 effort=14 velocity=32.9867 -> lower=-1.832597 upper=1.832597 effort=14 velocity=32.9867; origin xyz=0.08 -0.031498 0.0405 -> xyz=0.0418 0.023501 0
- joint right_joint6: limit lower=-2.8798 upper=2.8798 effort=14 velocity=32.9867 -> lower=-2.879795 upper=2.879795 effort=14 velocity=32.9867; origin xyz=0.022503 0 -0.0405 -> xyz=0.081 -0.023499 0
