Commit message: update mid model path

File: manipulator/AgileX/agilex_aloha_description/urdf/agilex_aloha.urdf (robot description, URDF)
Before this commit: robot AgileX Aloha, 38 links, 37 joints
Links:
- link lidar_link: geometry collision mesh filename=package://camera_models/meshes/mid360/mid360.obj; visual mesh filename=package://camera_models/meshes/mid360/mid360.obj
